File: Pallas/Pallas.sch (KiCad schematic (older format))
At the start: 237 parts, among them J1 OLED, J2 RGB_LED, Q1 IRLML6344TRPbF, SW00 SW_PUSH, SW01 SW_PUSH, SW010 SW_PUSH, SW011 SW_PUSH, SW012 SW_PUSH, SW013 SW_PUSH, SW014 SW_PUSH, SW02 SW_PUSH, SW03 SW_PUSH, SW04 SW_PUSH, SW05 SW_PUSH, SW06 SW_PUSH, SW07 SW_PUSH, SW08 SW_PUSH, SW09 SW_PUSH, SW10 SW_PUSH, SW11 SW_PUSH, SW110 SW_PUSH, SW111 SW_PUSH, SW112 SW_PUSH, SW113 SW_PUSH, SW114 SW_PUSH, SW12 SW_PUSH, SW13 SW_PUSH, SW14 SW_PUSH, SW15 SW_PUSH, SW16 SW_PUSH, SW17 SW_PUSH, SW18 SW_PUSH, SW19 SW_PUSH, SW20 SW_PUSH, SW21 SW_PUSH, SW210 SW_PUSH, SW211 SW_PUSH, SW212 SW_PUSH, SW213 SW_PUSH, SW214 SW_PUSH, SW22 SW_PUSH, SW23 SW_PUSH, SW24 SW_PUSH, SW25 SW_PUSH, SW26 SW_PUSH, SW27 SW_PUSH, SW28 SW_PUSH, SW29 SW_PUSH, SW30 SW_PUSH, SW31 SW_PUSH, SW310 SW_PUSH, SW311 SW_PUSH, SW312 SW_PUSH, SW313 SW_PUSH, SW314 SW_PUSH, SW32 SW_PUSH, SW33 SW_PUSH, SW34 SW_PUSH, SW35 SW_PUSH, SW36 SW_PUSH, SW37 SW_PUSH, SW38 SW_PUSH, SW39 SW_PUSH, SW40 SW_PUSH, SW41 SW_PUSH, SW410 SW_PUSH, SW411 SW_PUSH, SW412 SW_PUSH, SW413 SW_PUSH, SW414 SW_PUSH, SW42 SW_PUSH, SW43 SW_PUSH, SW44 SW_PUSH, SW45 SW_PUSH, SW46 SW_PUSH, SW47 SW_PUSH, SW48 SW_PUSH, SW49 SW_PUSH, U1 Elite-C

Commit message: Consolidate symbol and fp libraries
Parts:
- D00, D01, D010, D011, D012, D013, D014, D02, D03, D04, D05, D06, D07, D08, D09, D10, D11, D110, D111, D112, D113, D114, D12, D13, D14, D15, D16, D17, D18, D19, D20, D21, D210, D211, D212, D213, D214, D22, D23, D24, D25, D26, D27, D28, D29, D30, D31, D310, D311, D312, D313, D314, D32, D33, D34, D35, D36, D37, D38, D39, D40, D41, D410, D411, D412, D413, D414, D42, D43, D44, D45, D46, D47, D48, D49: footprint keyboard:Diode_SMD_THT -> Pallas:Diode_SMD_THT; symbol keyboard:D -> Pallas:D
- J1: footprint keyboard:OLED_128x64_I2C -> Pallas:OLED_128x64_I2C; symbol keyboard:Conn_01x04 -> Pallas:Conn_01x04
- J2: footprint keyboard:conn_3pins -> Pallas:conn_3pins; symbol keyboard:Conn_01x03 -> Pallas:Conn_01x03
- Q1: footprint keyboard:SOT23-3_HSOL_Back -> Pallas:SOT23-3_HSOL_Back; symbol keyboard:MOSFET -> Pallas:MOSFET
- R00, R01, R010, R011, R012, R013, R014, R02, R03, R04, R05, R06, R07, R08, R09, R1, R10, R11, R110, R111, R112, R113, R114, R12, R13, R14, R15, R16, R17, R18, R19, R2, R20, R21, R210, R211, R212, R213, R214, R22, R23, R24, R25, R26, R27, R28, R29, R3, R30, R31, R310, R311, R312, R313, R314, R32, R33, R34, R35, R36, R37, R38, R39, R40, R41, R410, R411, R412, R413, R414, R42, R43, R44, R45, R46, R47, R48, R49: footprint keyboard:Resistors_SMD_THT -> Pallas:Resistors_SMD_THT; symbol keyboard:R -> Pallas:R
- RGB1, RGB2, RGB3, RGB4: footprint keyboard:WS2812B_Front -> Pallas:WS2812B_Front; symbol keyboard:WS2812B -> Pallas:WS2812B
- RSW0: footprint keyboard:SW_RST -> Pallas:SW_RST; symbol keyboard:SW_RST -> Pallas:SW_RST
- SW00, SW01, SW010, SW011, SW012, SW013, SW014, SW02, SW03, SW04, SW05, SW06, SW07, SW08, SW09, SW11, SW110, SW111, SW112, SW113, SW114, SW12, SW13, SW14, SW15, SW16, SW17, SW18, SW19, SW21, SW210, SW211, SW212, SW213, SW22, SW23, SW24, SW25, SW26, SW27, SW28, SW29, SW31, SW310, SW311, SW312, SW313, SW32, SW33, SW34, SW35, SW36, SW37, SW38, SW39, SW410, SW43, SW46, SW47, SW48, SW49: footprint keyboard:SW_Cherry_MX_1.00u_PCB -> Pallas:SW_Cherry_MX_1.00u_PCB; symbol keyboard:KEY_SW_LED -> Pallas:KEY_SW_LED
- SW10: footprint keyboard:SW_Cherry_MX_1.50u_PCB -> Pallas:SW_Cherry_MX_1.50u_PCB; symbol keyboard:KEY_SW_LED -> Pallas:KEY_SW_LED
- SW20, SW314: footprint keyboard:SW_Cherry_MX_1.75u_PCB -> Pallas:SW_Cherry_MX_1.75u_PCB; symbol keyboard:KEY_SW_LED -> Pallas:KEY_SW_LED
- SW214: footprint keyboard:SW_Cherry_MX_2.25u_ISO_PCB -> Pallas:SW_Cherry_MX_2.25u_ISO_PCB; symbol keyboard:KEY_SW_LED -> Pallas:KEY_SW_LED
- SW30: footprint keyboard:SW_Cherry_MX_2.25u_PCB -> Pallas:SW_Cherry_MX_2.25u_PCB; symbol keyboard:KEY_SW_LED -> Pallas:KEY_SW_LED
- SW40, SW41, SW411, SW413, SW414, SW42, SW45: footprint keyboard:SW_Cherry_MX_1.25u_PCB -> Pallas:SW_Cherry_MX_1.25u_PCB; symbol keyboard:KEY_SW_LED -> Pallas:KEY_SW_LED
- SW412: footprint keyboard:SW_Cherry_MX_2.75u_PCB -> Pallas:SW_Cherry_MX_2.75u_PCB; symbol keyboard:KEY_SW_LED -> Pallas:KEY_SW_LED
- SW44: footprint keyboard:SW_Cherry_MX_2.00u_PCB -> Pallas:SW_Cherry_MX_2.00u_PCB; symbol keyboard:KEY_SW_LED -> Pallas:KEY_SW_LED
- U1: footprint keyboard:Elite-C-castellated-29pin-holes -> Pallas:Elite-C-castellated-29pin-holes; symbol keyboard:Elite-C -> Pallas:Elite-C
Connections:
- wire segments 410 -> 350
