File: Pallas/Pallas.kicad_pcb (KiCad board)
At the start: 2 copper layers, 467.5 x 140 mm, 263 parts, among them J1 OLED, J2 RGB_LED, Q1 IRLML6344TRPbF, SW00 SW_PUSH, SW01 SW_PUSH, SW010 SW_PUSH, SW011 SW_PUSH, SW012 SW_PUSH, SW013 SW_PUSH, SW014 SW_PUSH, SW02 SW_PUSH, SW03 SW_PUSH, SW04 SW_PUSH, SW05 SW_PUSH, SW06 SW_PUSH, SW07 SW_PUSH, SW08 SW_PUSH, SW09 SW_PUSH, SW10 SW_PUSH, SW11 SW_PUSH, SW110 SW_PUSH, SW111 SW_PUSH, SW112 SW_PUSH, SW113 SW_PUSH, SW114 SW_PUSH, SW12 SW_PUSH, SW13 SW_PUSH, SW14 SW_PUSH, SW15 SW_PUSH, SW16 SW_PUSH, SW17 SW_PUSH, SW18 SW_PUSH, SW19 SW_PUSH, SW20 SW_PUSH, SW21 SW_PUSH, SW210 SW_PUSH, SW211 SW_PUSH, SW212 SW_PUSH, SW213 SW_PUSH, SW214 SW_PUSH, SW22 SW_PUSH, SW23 SW_PUSH, SW24 SW_PUSH, SW25 SW_PUSH, SW26 SW_PUSH, SW27 SW_PUSH, SW28 SW_PUSH, SW29 SW_PUSH, SW30 SW_PUSH, SW31 SW_PUSH, SW310 SW_PUSH, SW311 SW_PUSH, SW312 SW_PUSH, SW313 SW_PUSH, SW314 SW_PUSH, SW32 SW_PUSH, SW33 SW_PUSH, SW34 SW_PUSH, SW35 SW_PUSH, SW36 SW_PUSH, SW37 SW_PUSH, SW38 SW_PUSH, SW39 SW_PUSH, SW40 SW_PUSH, SW41 SW_PUSH, SW410 SW_PUSH, SW411 SW_PUSH, SW412 SW_PUSH, SW413 SW_PUSH, SW414 SW_PUSH, SW42 SW_PUSH, SW43 SW_PUSH, SW44 SW_PUSH, SW45 SW_PUSH, SW46 SW_PUSH, SW47 SW_PUSH, SW48 SW_PUSH, SW49 SW_PUSH, U1 Elite-C

Commit message: clean routes
Parts:
- moved DecorationHoleTop1 116.4 mm to (232.6, 230.4)
- moved DecorationHoleTop2 116.4 mm to (332.6, 230.4)
- moved J2 51.3 mm to (306.5, 43.9), turned to 270 degrees
- moved Q1 28.4 mm to (236.7, 59.0), turned to 90 degrees
- moved R3 26.8 mm to (241.8, 59.0)
- moved R1 22.9 mm to (240.8, 63.3), turned to 270 degrees
- moved R2 20.1 mm to (243.6, 63.3), turned to 270 degrees
- moved R214 8.01 mm to (493.3, 111.8), turned to 90 degrees
Routing:
- net VCC: track 2309.2 -> 41.4 mm, vias 8 -> 0
- net LED: track 2383.0 -> 305.2 mm, vias 1 -> 0
- net row2: track 687.7 -> 64.7 mm, vias 26 -> 0
- net row3: track 624.8 -> 55.4 mm, vias 26 -> 0
- net row4: track 623.7 -> 56.2 mm, vias 2 -> 0
- net row0: track 606.5 -> 55.4 mm, vias 27 -> 0
- net row1: track 602.7 -> 57.6 mm, vias 30 -> 0
- net col14: track 359.3 -> 0.71 mm
- net col10: track 352.3 -> 2.45 mm
- net col11: track 359.6 -> 15.6 mm
- net col12: track 343.2 -> 11.0 mm
- net col9: track 328.8 -> 2.60 mm
- net col13: track 318.8 -> 0.00 mm
- net col8: track 320.6 -> 3.38 mm
- net col0: track 283.7 -> 1.13 mm, vias 2 -> 0
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
Commit message: New routes
Parts:
- moved RGB3 100.2 mm to (238.7, 129.4), turned to 270 degrees
- moved RGB4 100.2 mm to (238.7, 100.8), turned to 270 degrees
- moved RGB1 100.0 mm to (338.9, 100.8), turned to 90 degrees
- moved RGB2 100.0 mm to (338.9, 129.4), turned to 90 degrees
- moved DecorationHoleTop1 20.2 mm to (236.5, 210.6)
- moved DecorationHoleTop2 20.2 mm to (336.5, 210.6)
- moved D214 1.46 mm to (492.7, 94.3)
- moved D412 1.38 mm to (372.8, 148.7)
- moved R3 1.19 mm to (242.4, 58.1)
- moved Q1 1.19 mm to (237.4, 58.1)
- moved R07 1.08 mm to (375.8, 59.0)
- moved D08 1.03 mm to (380.3, 68.5)
- moved R013 1.00 mm to (492.5, 45.9)
- moved R214 0.98 mm to (492.9, 110.9)
- moved R19 0.97 mm to (408.7, 71.6)
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Routing:
- net row4: track 56.2 -> 500.2 mm
- net row0: track 55.4 -> 398.8 mm
- net row3: track 55.4 -> 374.3 mm
- net row2: track 64.7 -> 378.9 mm
- net row1: track 57.6 -> 360.2 mm
- net (no net): track 0.00 -> 112.0 mm
- net Net-(R30-Pad2): track 0.71 -> 21.0 mm
- net Net-(R412-Pad2): track 4.11 -> 20.1 mm
- net Net-(R44-Pad2): track 4.11 -> 20.1 mm
- net col11: track 15.6 -> 2.45 mm
- net VCC: track 41.4 -> 29.1 mm
- net LED: track 305.2 -> 295.4 mm
- net col12: track 11.0 -> 2.65 mm
- net Net-(R011-Pad2): track 3.86 -> 11.2 mm
- net Net-(R411-Pad2): track 3.86 -> 11.1 mm
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
Commit message: Pallas rev 0.3
Parts:
- removed LogoMiddle1: LOGO, Pallas:athena
- RSW0: value SW_Push -> SW_RST
- moved DecorationHoleTop1 96.3 mm to (238.9, 114.3)
- moved DecorationHoleTop2 96.3 mm to (338.9, 114.3)
- turned RGB1 to 0 degrees
- turned RGB2 to 0 degrees
- turned RGB3 to 180 degrees
- turned RGB4 to 180 degrees
Connections:
- RGB1 pad 2: RGB -> Net-(RGB1-Pad2)
- RGB1 pad 4: Net-(RGB1-Pad4) -> RGB
- RGB2 pad 2: Net-(RGB1-Pad4) -> Net-(RGB2-Pad2)
- RGB2 pad 4: Net-(RGB2-Pad4) -> Net-(RGB1-Pad2)
- RGB3 pad 2: Net-(RGB2-Pad4) -> Net-(RGB3-Pad2)
- RGB3 pad 4: Net-(RGB3-Pad4) -> Net-(RGB2-Pad2)
- RGB4 pad 2: Net-(RGB3-Pad4) -> Net-(RGB4-Pad2)
- RGB4 pad 4: Net-(RGB4-Pad4) -> Net-(RGB3-Pad2)
Routing:
- net VCC: track 29.1 -> 2265.9 mm, vias 0 -> 5
- net LED: track 295.4 -> 2180.5 mm, vias 0 -> 1
- net col14: track 0.71 -> 357.2 mm
- net col11: track 2.45 -> 357.9 mm
- net col10: track 2.45 -> 340.2 mm
- net col12: track 2.65 -> 332.1 mm, vias 0 -> 1
- net col13: track 0.00 -> 311.4 mm
- net col9: track 2.60 -> 287.0 mm
- net col0: track 1.13 -> 278.4 mm
- net col1: track 2.76 -> 265.0 mm
- net col2: track 0.32 -> 248.7 mm
- net col3: track 0.80 -> 221.0 mm
- net row3: track 374.3 -> 591.9 mm, vias 0 -> 4
- net col5: track 0.65 -> 217.9 mm
- net col4: track 2.52 -> 211.6 mm
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
Commit message: review
Routing:
- net GND: vias 3 -> 99
