File: Kanagawa/Link/Link.kicad_pcb (KiCad board)
At the start: 2 copper layers, 23 x 24 mm, 2 parts, among them J0 Conn_02x10_Counter_Clockwise, J1 Conn_02x10_Counter_Clockwise

Commit message: link bridge
Parts:
- removed J1: Conn_02x10_Counter_Clockwise, link:conn_2x10_P2.00mm_Vertical
- J0: footprint link:conn_2x10_P2.00mm_Vertical -> link:bridge_2x10_P2.00mm
Other:
- board outline removed

Commit message: improve link
Parts:
- J0: value Conn_02x10_Counter_Clockwise -> Conn_02x15; footprint link:bridge_2x10_P2.00mm -> link:bridge_2x15_P2.54mm
Connections:
- net col0 renamed rotA
- net col1 renamed rotB
- net col2 renamed col00
- net col3 renamed col01
- net col4 renamed col02
- net col5 renamed col03
- net col6 renamed col04
- net col7 renamed col05
- J0 pad 11: row0 -> col06
- J0 pad 12: row1 -> col07
- J0 pad 13: row2 -> col08
- J0 pad 14: row3 -> col10
- J0 pad 15: row4 -> col12
- J0 pad 16: row5 -> col13
- J0 pad 17: SCL -> col11
- J0 pad 18: SDA -> col09
- J0 pad 19: RGB -> row7
- J0 pad 20: GND -> row6
Routing:
- net VCC: track 0.00 -> 11.8 mm
- net RGB: track 0.00 -> 11.1 mm
- net GND: track 0.00 -> 10.8 mm
- net col04: track 0.00 -> 10.6 mm
- net col02: track 0.00 -> 10.6 mm
- net col01: track 0.00 -> 10.6 mm
- net col09: track 0.00 -> 10.6 mm
- net LED: track 0.00 -> 10.6 mm
- net SCL: track 0.00 -> 10.6 mm
- net SDA: track 0.00 -> 10.6 mm
- net row7: track 0.00 -> 10.6 mm
- net col06: track 0.00 -> 10.6 mm
- net col03: track 0.00 -> 10.6 mm
- net row3: track 0.00 -> 10.6 mm
- net col08: track 0.00 -> 10.6 mm
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- added copper zone on B.Cu, net GND
- added copper zone on F.Cu, net GND
Other:
- board outline added: 24 x 48 mm
