File: Kanagawa/Kanagawa/Kanagawa.kicad_pcb (KiCad board)
At the start: 2 copper layers, 90 parts, among them J0 Conn_01x03, J1 Conn_01x04, SW99 Rotary_Encoder_Switch

Commit message: Begin placing footprints
Parts:
- added KA0: KEY_SW, keyboard:SW_Cherry_MX_1.00u_SK6812MINI, F.Cu at (167.5, 348.0)
- added KA1: KEY_SW, keyboard:SW_Cherry_MX_1.00u_SK6812MINI, F.Cu at (146.3, 347.7)
- added KA10: KEY_SW, keyboard:SW_Cherry_MX_1.00u_SK6812MINI, F.Cu at (-49.0, 347.5)
- added KA11: KEY_SW, keyboard:SW_Cherry_MX_1.00u_SK6812MINI, F.Cu at (65.0, 347.5)
- added KA12: KEY_SW, keyboard:SW_Cherry_MX_1.00u_SK6812MINI, F.Cu at (45.0, 347.5)
- added KA2: KEY_SW, keyboard:SW_Cherry_MX_1.00u_SK6812MINI, F.Cu at (-70.0, 347.5)
- added KA3: KEY_SW, keyboard:SW_Cherry_MX_1.00u_SK6812MINI, F.Cu at (-0.50, 348.0)
- added KA4: KEY_SW, keyboard:SW_Cherry_MX_1.00u_SK6812MINI, F.Cu at (86.1, 347.5)
- added KA5: KEY_SW, keyboard:SW_Cherry_MX_1.00u_SK6812MINI, F.Cu at (-92.0, 347.5)
- added KA6: KEY_SW, keyboard:SW_Cherry_MX_1.00u_SK6812MINI, F.Cu at (21.5, 348.0)
- added KA7: KEY_SW, keyboard:SW_Cherry_MX_1.00u_SK6812MINI, F.Cu at (126.1, 347.7)
- added KA8: KEY_SW, keyboard:SW_Cherry_MX_1.00u_SK6812MINI, F.Cu at (106.3, 347.5)
- added KA9: KEY_SW, keyboard:SW_Cherry_MX_1.00u_SK6812MINI, F.Cu at (-25.0, 348.0)
- added KB0: KEY_SW, keyboard:SW_Cherry_MX_1.00u_SK6812MINI, F.Cu at (92.5, 372.0)
- added KB1: KEY_SW, keyboard:SW_Cherry_MX_1.00u_SK6812MINI, F.Cu at (31.7, 371.3)
- added KB10: KEY_SW, keyboard:SW_Cherry_MX_1.00u_SK6812MINI, F.Cu at (-29.5, 370.4)
- added KB11: KEY_SW, keyboard:SW_Cherry_MX_1.00u_SK6812MINI, F.Cu at (172.7, 372.2)
- added KB12: KEY_SW, keyboard:SW_Cherry_MX_1.00u_SK6812MINI, F.Cu at (132.9, 372.0)
- added KB13: KEY_SW, keyboard:SW_Cherry_MX_1.00u_SK6812MINI, F.Cu at (72.1, 371.3)
- added KB14: KEY_SW, keyboard:SW_Cherry_MX_1.00u_SK6812MINI, F.Cu at (53.8, 233.6)
- added KB2: KEY_SW, keyboard:SW_Cherry_MX_1.00u_SK6812MINI, F.Cu at (11.4, 370.6)
- added KB3: KEY_SW, keyboard:SW_Cherry_MX_1.00u_SK6812MINI, F.Cu at (-91.4, 370.6)
- added KB4: KEY_SW, keyboard:SW_Cherry_MX_1.00u_SK6812MINI, F.Cu at (-49.7, 370.4)
- added KB5: KEY_SW, keyboard:SW_Cherry_MX_1.00u_SK6812MINI, F.Cu at (152.5, 372.2)
- added KB6: KEY_SW, keyboard:SW_Cherry_MX_1.00u_SK6812MINI, F.Cu at (112.7, 372.0)
- added KB7: KEY_SW, keyboard:SW_Cherry_MX_1.00u_SK6812MINI, F.Cu at (51.9, 371.3)
- added KB8: KEY_SW, keyboard:SW_Cherry_MX_1.00u_SK6812MINI, F.Cu at (-8.80, 370.6)
- added KB9: KEY_SW, keyboard:SW_Cherry_MX_1.00u_SK6812MINI, F.Cu at (-71.2, 370.6)
- added KC0: KEY_SW, keyboard:SW_Cherry_MX_1.00u_SK6812MINI, F.Cu at (-71.7, 392.3)
- added KC1: KEY_SW, keyboard:SW_Cherry_MX_1.00u_SK6812MINI, F.Cu at (-30.5, 392.1)
- added KC10: KEY_SW, keyboard:SW_Cherry_MX_1.00u_SK6812MINI, F.Cu at (33.6, 294.2)
- added KC11: KEY_SW, keyboard:SW_Cherry_MX_1.00u_SK6812MINI, F.Cu at (53.8, 274.0)
- added KC12: KEY_SW, keyboard:SW_Cherry_MX_1.00u_SK6812MINI, F.Cu at (74.0, 253.8)
- added KC13: KEY_SW, keyboard:SW_Cherry_MX_1.00u_SK6812MINI, F.Cu at (71.0, 391.5)
- added KC14: KEY_SW, keyboard:SW_Cherry_MX_1.00u_SK6812MINI, F.Cu at (9.90, 392.1)
- added KC2: KEY_SW, keyboard:SW_Cherry_MX_1.00u_SK6812MINI, F.Cu at (30.7, 391.9)
- added KC3: KEY_SW, keyboard:SW_Cherry_MX_1.00u_SK6812MINI, F.Cu at (94.2, 233.6)
- added KC4: KEY_SW, keyboard:SW_Cherry_MX_1.00u_SK6812MINI, F.Cu at (-91.9, 392.3)
- added KC5: KEY_SW, keyboard:SW_Cherry_MX_1.00u_SK6812MINI, F.Cu at (53.8, 253.8)
- added KC6: KEY_SW, keyboard:SW_Cherry_MX_1.00u_SK6812MINI, F.Cu at (74.0, 233.6)
- added KC7: KEY_SW, keyboard:SW_Cherry_MX_1.00u_SK6812MINI, F.Cu at (-51.5, 392.3)
- added KC8: KEY_SW, keyboard:SW_Cherry_MX_1.00u_SK6812MINI, F.Cu at (-10.3, 392.1)
- added KC9: KEY_SW, keyboard:SW_Cherry_MX_1.00u_SK6812MINI, F.Cu at (50.9, 391.9)
- added KD0: KEY_SW, keyboard:SW_Cherry_MX_1.00u_SK6812MINI, F.Cu at (10.6, 415.4)
- added KD1: KEY_SW, keyboard:SW_Cherry_MX_1.00u_SK6812MINI, F.Cu at (53.8, 294.2)
- added KD10: KEY_SW, keyboard:SW_Cherry_MX_1.00u_SK6812MINI, F.Cu at (114.4, 253.8)
- added KD11: KEY_SW, keyboard:SW_Cherry_MX_1.00u_SK6812MINI, F.Cu at (134.6, 233.6)
- added KD12: KEY_SW, keyboard:SW_Cherry_MX_1.00u_SK6812MINI, F.Cu at (-51.9, 415.8)
- added KD13: KEY_SW, keyboard:SW_Cherry_MX_1.00u_SK6812MINI, F.Cu at (-10.2, 415.6)
- added KD2: KEY_SW, keyboard:SW_Cherry_MX_1.00u_SK6812MINI, F.Cu at (74.0, 274.0)
- added KD3: KEY_SW, keyboard:SW_Cherry_MX_1.00u_SK6812MINI, F.Cu at (94.2, 253.8)
- added KD4: KEY_SW, keyboard:SW_Cherry_MX_1.00u_SK6812MINI, F.Cu at (114.4, 233.6)
- added KD5: KEY_SW, keyboard:SW_Cherry_MX_1.00u_SK6812MINI, F.Cu at (-72.1, 415.8)
- added KD6: KEY_SW, keyboard:SW_Cherry_MX_1.00u_SK6812MINI, F.Cu at (-30.4, 415.6)
- added KD7: KEY_SW, keyboard:SW_Cherry_MX_1.00u_SK6812MINI, F.Cu at (30.8, 415.4)
- added KD8: KEY_SW, keyboard:SW_Cherry_MX_1.00u_SK6812MINI, F.Cu at (134.6, 294.2)
- added KD9: KEY_SW, keyboard:SW_Cherry_MX_1.00u_SK6812MINI, F.Cu at (-92.3, 415.8)
- added KE0: KEY_SW, keyboard:SW_Cherry_MX_1.00u_SK6812MINI, F.Cu at (-71.5, 436.4)
- added KE1: KEY_SW, keyboard:SW_Cherry_MX_1.00u_SK6812MINI, F.Cu at (94.2, 294.2)
- added KE10: KEY_SW, keyboard:SW_Cherry_MX_1.00u_SK6812MINI, F.Cu at (134.6, 274.0)
- added KE11: KEY_SW, keyboard:SW_Cherry_MX_1.00u_SK6812MINI, F.Cu at (154.8, 253.8)
- added KE12: KEY_SW, keyboard:SW_Cherry_MX_1.00u_SK6812MINI, F.Cu at (175.0, 233.6)
- added KE2: KEY_SW, keyboard:SW_Cherry_MX_1.00u_SK6812MINI, F.Cu at (114.4, 274.0)
- added KE3: KEY_SW, keyboard:SW_Cherry_MX_1.00u_SK6812MINI, F.Cu at (134.6, 253.8)
- added KE4: KEY_SW, keyboard:SW_Cherry_MX_1.00u_SK6812MINI, F.Cu at (154.8, 233.6)
- added KE5: KEY_SW, keyboard:SW_Cherry_MX_1.00u_SK6812MINI, F.Cu at (74.0, 294.2)
- added KE6: KEY_SW, keyboard:SW_Cherry_MX_1.00u_SK6812MINI, F.Cu at (33.6, 274.0)
- added KE7: KEY_SW, keyboard:SW_Cherry_MX_1.00u_SK6812MINI, F.Cu at (-91.5, 436.5)
- added KE8: KEY_SW, keyboard:SW_Cherry_MX_1.00u_SK6812MINI, F.Cu at (-51.3, 436.4)
- added KE9: KEY_SW, keyboard:SW_Cherry_MX_1.00u_SK6812MINI, F.Cu at (114.4, 294.2)
- added KF0: KEY_SW, keyboard:SW_Cherry_MX_1.00u_SK6812MINI, F.Cu at (-72.0, 458.8)
- added KF1: KEY_SW, keyboard:SW_Cherry_MX_1.00u_SK6812MINI, F.Cu at (-9.80, 458.6)
- added KF10: KEY_SW, keyboard:SW_Cherry_MX_1.00u_SK6812MINI, F.Cu at (175.0, 274.0)
- added KF11: KEY_SW, keyboard:SW_Cherry_MX_1.00u_SK6812MINI, F.Cu at (-31.6, 458.8)
- added KF12: KEY_SW, keyboard:SW_Cherry_MX_1.00u_SK6812MINI, F.Cu at (30.6, 458.6)
- added KF2: KEY_SW, keyboard:SW_Cherry_MX_1.00u_SK6812MINI, F.Cu at (94.2, 274.0)
- added KF3: KEY_SW, keyboard:SW_Cherry_MX_1.00u_SK6812MINI, F.Cu at (-92.2, 458.8)
- added KF4: KEY_SW, keyboard:SW_Cherry_MX_1.00u_SK6812MINI, F.Cu at (154.8, 274.0)
- added KF5: KEY_SW, keyboard:SW_Cherry_MX_1.00u_SK6812MINI, F.Cu at (175.0, 253.8)
- added KF6: KEY_SW, keyboard:SW_Cherry_MX_1.00u_SK6812MINI, F.Cu at (-51.8, 458.8)
- added KF7: KEY_SW, keyboard:SW_Cherry_MX_1.00u_SK6812MINI, F.Cu at (10.4, 458.6)
- added KF8: KEY_SW, keyboard:SW_Cherry_MX_1.00u_SK6812MINI, F.Cu at (52.5, 458.5)
- added KF9: KEY_SW, keyboard:SW_Cherry_MX_1.00u_SK6812MINI, F.Cu at (154.8, 294.2)
- moved SW99 405.4 mm to (379.5, 87.0)

Commit message: update footprint
Parts:
- removed DA14, DB14, DC14: D, keyboard:Diode_SMD_THT
- removed the G*** at (216.2, 140.5)
- removed KB14, KC14: KEY_SW, keyboard:SW_Cherry_MX_1.00u_SK6812MINI
- added DA13: D, keyboard:Diode_SMD_THT, F.Cu at (-1.84, 95.6)
- added DE13: D, keyboard:Diode_SMD_THT, F.Cu at (-1.84, 99.3)
- added DF13: D, keyboard:Diode_SMD_THT, F.Cu at (-1.84, 103.1)
- added G***: LOGO, layout-for-export:Dwgs.User_g222, F.Cu at (217.0, 152.0)
- added KE13: KEY_SW, keyboard:SW_Cherry_MX_1.25u_SK6812MINI, F.Cu at (119.6, 410.1)
- added KF13: KEY_SW, keyboard:SW_Cherry_MX_1.25u_SK6812MINI, F.Cu at (223.5, 432.5)
- added U0: Pico, RP-Pico:RPi_Pico_SMD_TH, F.Cu at (371.0, 59.5)
- KB13, KD12, KF4, KF5: footprint keyboard:SW_Cherry_MX_1.00u_SK6812MINI -> keyboard:SW_Cherry_MX_2.00u_SK6812MINI
- KC0, KC12: footprint keyboard:SW_Cherry_MX_1.00u_SK6812MINI -> keyboard:SW_Cherry_MX_1.50u_SK6812MINI
- KD0: footprint keyboard:SW_Cherry_MX_1.00u_SK6812MINI -> keyboard:SW_Cherry_MX_1.75u_SK6812MINI
- KD13, KF0, KF2, KF7, KF9: footprint keyboard:SW_Cherry_MX_1.00u_SK6812MINI -> keyboard:SW_Cherry_MX_1.25u_SK6812MINI
- KE0, KE11: footprint keyboard:SW_Cherry_MX_1.00u_SK6812MINI -> keyboard:SW_Cherry_MX_2.25u_SK6812MINI
- moved KC5 346.9 mm to (381.8, 366.8)
- moved KC11 321.3 mm to (361.5, 366.5)
- moved KF2 320.1 mm to (371.5, 434.0)
- moved KC0 316.8 mm to (244.0, 366.0)
- moved KE6 306.9 mm to (308.5, 410.5)
- moved KD2 305.2 mm to (356.5, 389.5)
- moved KC10 286.8 mm to (311.0, 367.0)
- moved KC12 285.7 mm to (336.5, 366.5)
- moved KB13 281.5 mm to (352.5, 346.0)
- moved KD11 254.0 mm to (335.1, 389.6)
- moved KD4 254.0 mm to (314.9, 389.6)
- moved KE12 247.8 mm to (349.0, 410.1)
- moved KE4 247.8 mm to (328.8, 410.1)
- moved KD3 242.1 mm to (295.0, 389.0)
- moved KF10 235.3 mm to (348.5, 433.0)
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Connections:
- KB13 pad 3: Net-(KB13-Pad3) -> LEDR0
- KB13 pad 5: col13 -> SW99A
- KC13 pad 3: Net-(KC13-Pad3) -> LEDR1
- KC13 pad 5: col13 -> SW99A
- KD13 pad 5: col13 -> SW99A
- KE12 pad 3: LEDR3 -> Net-(KE12-Pad3)
- KF12 pad 3: LEDR4 -> Net-(KF12-Pad3)

Commit message: prepare pcb layout
Parts:
- added J1: OLED, keyboard:OLED_128x64_I2C, F.Cu at (351.0, 106.0)
- KC12: footprint keyboard:SW_Cherry_MX_1.50u_SK6812MINI -> keyboard:SW_Cherry_MX_1.00u_SK6812MINI
- KC13: footprint keyboard:SW_Cherry_MX_1.00u_SK6812MINI -> keyboard:SW_Cherry_MX_1.50u_SK6812MINI
- moved KE13 363.2 mm to (359.5, 137.5)
- moved KF2 353.1 mm to (112.0, 194.5)
- moved J0 349.3 mm to (325.5, 32.0)
- moved KD13 338.6 mm to (359.5, 118.5)
- moved KA0 336.9 mm to (66.5, 94.5)
- moved R2 334.4 mm to (362.0, 31.0)
- moved KD2 332.7 mm to (119.0, 156.5)
- moved KF11 328.0 mm to (347.5, 199.5)
- moved KD12 319.4 mm to (323.5, 156.5)
- moved KC5 311.5 mm to (171.0, 137.5)
- moved KF13 307.7 mm to (359.5, 156.5)
- moved R1 307.3 mm to (362.0, 25.5)
- moved KD9 304.8 mm to (252.5, 156.5)
- moved KA1 301.8 mm to (95.0, 94.5)
- moved KF12 299.0 mm to (366.5, 199.5)
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Routing:
- added copper zone on B.Cu, net GND
- added copper zone on F.Cu, net GND
Other:
- board outline added: 349.5 x 165 mm

Commit message: test footprint
Parts:
- moved U0 32.2 mm to (110.7, 94.7)
- moved J1 2.08 mm to (349.5, 107.4)
Changed lines of the file:
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@@
-(kicad_pcb (version 20171130) (host pcbnew "(5.1.6)-1")
+(kicad_pcb (version 20171130) (host pcbnew "(5.1.9)-1")
   (general
     (thickness 1.6)
@@
   )
   (module keyboard:OLED_128x64_I2C (layer F.Cu)
-    (at 351 106 180)
+    (at 349.504 107.442 180)
     (tags "OLED 0.96 inch 128x64 I2C")
     (fp_text reference J1 (at 0 0 180) (layer F.SilkS)
@@
       (effects (font (size 1 1) (thickness 0.15)))
     )
-    (fp_text user SDA (at 16.2 3.5 180) (layer B.SilkS)
-      (effects (font (size 0.5 0.5) (thickness 0.1)) (justify mirror))
-    )
-    (fp_text user SCL (at 13.5 3.5 180) (layer B.SilkS)
-      (effects (font (size 0.5 0.5) (thickness 0.1)) (justify mirror))
-    )
-    (fp_text user VCC (at 11.1 3.5 180) (layer B.SilkS)
-      (effects (font (size 0.5 0.5) (thickness 0.1)) (justify mirror))
-    )
-    (fp_text user GND (at 8.5 3.5 180) (layer B.SilkS)
-      (effects (font (size 0.5 0.5) (thickness 0.1)) (justify mirror))
-    )
-    (fp_text user OLED (at 3 6 180) (layer F.SilkS) hide
-      (effects (font (size 0.8128 0.8128) (thickness 0.15)))
-    )
-    (fp_text user O3 (at 20 6) (layer F.SilkS) hide
-      (effects (font (size 0.8128 0.8128) (thickness 0.15)))
-    )
-    (fp_text user %R (at 12 12 180) (layer F.SilkS)
-      (effects (font (size 1 1) (thickness 0.15)))
-    )
-    (fp_text user %R (at 12 12 180) (layer B.SilkS)
-      (effects (font (size 1 1) (thickness 0.15)) (justify mirror))
-    )
-    (fp_text user GND (at 8.5 3.5 180) (layer F.SilkS)
-      (effects (font (size 0.5 0.5) (thickness 0.1)))
-    )
-    (fp_text user VCC (at 11.1 3.5 180) (layer F.SilkS)
-      (effects (font (size 0.5 0.5) (thickness 0.1)))
-    )
-    (fp_text user SCL (at 13.5 3.5 180) (layer F.SilkS)
-      (effects (font (size 0.5 0.5) (thickness 0.1)))
-    )
-    (fp_text user SDA (at 16.2 3.5 180) (layer F.SilkS)
-      (effects (font (size 0.5 0.5) (thickness 0.1)))
-    )
     (fp_line (start 23.22 6.58) (end 23.22 17.44) (layer F.SilkS) (width 0.12))
     (fp_line (start 1.48 6.58) (end 23.22 6.58) (layer B.SilkS) (width 0.12))
@@
     (fp_line (start 17.35 0.254) (end 17.35 2.794) (layer B.SilkS) (width 0.15))
     (fp_line (start 7.35 2.794) (end 17.35 2.794) (layer F.SilkS) (width 0.15))
+    (fp_text user SDA (at 16.2 3.5 180) (layer B.SilkS)
+      (effects (font (size 0.5 0.5) (thickness 0.1)) (justify mirror))
+    )
+    (fp_text user SCL (at 13.5 3.5 180) (layer B.SilkS)
+      (effects (font (size 0.5 0.5) (thickness 0.1)) (justify mirror))
+    )
+    (fp_text user VCC (at 11.1 3.5 180) (layer B.SilkS)
+      (effects (font (size 0.5 0.5) (thickness 0.1)) (justify mirror))
+    )
+    (fp_text user GND (at 8.5 3.5 180) (layer B.SilkS)
+      (effects (font (size 0.5 0.5) (thickness 0.1)) (justify mirror))
+    )
+    (fp_text user OLED (at 3 6 180) (layer F.SilkS) hide
+      (effects (font (size 0.8128 0.8128) (thickness 0.15)))
+    )
+    (fp_text user O3 (at 20 6) (layer F.SilkS) hide
+      (effects (font (size 0.8128 0.8128) (thickness 0.15)))
+    )
+    (fp_text user %R (at 12 12 180) (layer F.SilkS)
+      (effects (font (size 1 1) (thickness 0.15)))
+    )
+    (fp_text user %R (at 12 12 180) (layer B.SilkS)
+      (effects (font (size 1 1) (thickness 0.15)) (justify mirror))
+    )
+    (fp_text user GND (at 8.5 3.5 180) (layer F.SilkS)
+      (effects (font (size 0.5 0.5) (thickness 0.1)))
+    )
+    (fp_text user VCC (at 11.1 3.5 180) (layer F.SilkS)
+      (effects (font (size 0.5 0.5) (thickness 0.1)))
+    )
+    (fp_text user SCL (at 13.5 3.5 180) (layer F.SilkS)
+      (effects (font (size 0.5 0.5) (thickness 0.1)))
+    )
+    (fp_text user SDA (at 16.2 3.5 180) (layer F.SilkS)
+      (effects (font (size 0.5 0.5) (thickness 0.1)))
+    )
     (pad 2 thru_hole circle (at 11.08 1.5 180) (size 1.397 1.397) (drill 0.8128) (layers *.Cu *.Mask F.SilkS))
     (pad 3 thru_hole circle (at 13.62 1.5 180) (size 1.397 1.397) (drill 0.8128) (layers *.Cu *.Mask F.SilkS))
@@
   )
   (module RP-Pico:RPi_Pico_SMD_TH (layer F.Cu)
-    (at 78.5 95 90)
+    (at 110.744 94.742 90)
     (descr "Through hole straight pin header, 2x20, 2.54mm pitch, double rows")
     (tags "Through hole pin header THT 2x20 2.54mm double row")

Commit message: update pcb
Parts:
- removed the J1 at (349.5, 107.4)
- added REF**: Keebio_USB-C_breakout_shadow, keyboard:Keebio_USB-C_breakout_shadow, F.Cu at (219.8, 84.5)
- J1: footprint keyboard:conn_4pins -> keyboard:OLED_128x64_I2C
- KD13, KE13, KF13: footprint keyboard:SW_Cherry_MX_1.25u_SK6812MINI -> keyboard:SW_Cherry_MX_1.25u_SK6812MINI_Rotated
- U0: footprint RP-Pico:RPi_Pico_SMD_TH -> keyboard:RPi_Pico_TH
- moved DA13 470.8 mm to (381.9, 96.7), turned to 90 degrees
- moved DF12 419.7 mm to (375.6, 204.4), turned to 90 degrees
- moved DD13 414.3 mm to (364.3, 107.8), turned to 180 degrees
- moved DA12 412.2 mm to (322.9, 99.8), turned to 90 degrees
- moved DD12 411.4 mm to (341.7, 161.7), turned to 90 degrees
- moved DC13 408.0 mm to (338.5, 142.4), turned to 90 degrees
- moved DE12 407.9 mm to (356.7, 185.4), turned to 90 degrees
- moved DE13 406.0 mm to (364.5, 128.1), turned to 180 degrees
- moved DF11 403.1 mm to (356.1, 204.6), turned to 90 degrees
- moved DF10 395.8 mm to (337.1, 204.4), turned to 90 degrees
- moved DB13 394.5 mm to (319.2, 110.0)
- moved DA11 392.0 mm to (303.8, 99.7), turned to 90 degrees
- moved DF13 390.4 mm to (354.0, 147.2)
- moved DB12 385.3 mm to (303.7, 123.5), turned to 90 degrees
- moved DC12 382.2 mm to (313.6, 142.6), turned to 90 degrees
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Other:
- board size 349.5 x 165 mm -> 334.8 x 145.8 mm

Commit message: begin routes
Parts:
- moved DF3 12.5 mm to (141.1, 186.9), turned to 345 degrees
- moved DF13 10.5 mm to (364.5, 147.1), turned to 180 degrees
- moved DF5 3.88 mm to (204.9, 193.7), turned to 15 degrees
- moved SW99 2.25 mm to (370.0, 92.4)
- moved DA13 2.25 mm to (379.9, 97.5)
- moved DD0 1.87 mm to (82.2, 161.5)
- moved DF6 1.85 mm to (220.5, 189.5), turned to 15 degrees
- moved DC13 1.58 mm to (336.9, 142.6)
- moved DE11 1.56 mm to (329.9, 180.7)
- moved DD13 1.23 mm to (364.5, 109.1)
- moved DF4 1.09 mm to (161.3, 192.3), turned to 345 degrees
- moved DF2 0.91 mm to (120.3, 199.8)
- moved DE12 0.72 mm to (356.0, 185.4)
- moved DF9 0.69 mm to (310.8, 199.8)
- moved DF7 0.66 mm to (267.8, 199.8)
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Routing:
- net VCC: track 0.00 -> 343.2 mm, vias 0 -> 1
- net LED: track 0.00 -> 67.3 mm, vias 0 -> 2
- net row05: track 0.00 -> 49.3 mm
- net row03: track 0.00 -> 48.3 mm
- net row02: track 0.00 -> 48.3 mm
- net row00: track 0.00 -> 48.3 mm
- net row01: track 0.00 -> 48.3 mm
- net row04: track 0.00 -> 48.3 mm
- net SDA: track 0.00 -> 32.8 mm, vias 0 -> 1
- net SCL: track 0.00 -> 29.3 mm
- net Net-(KA0-Pad3): track 0.00 -> 24.5 mm
- net Net-(KA8-Pad3): track 0.00 -> 19.7 mm
- net Net-(KA4-Pad3): track 0.00 -> 19.7 mm
- net Net-(DE0-Pad2): track 0.00 -> 16.5 mm
- net Net-(DE11-Pad2): track 0.00 -> 16.4 mm
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Other:
- outline, holes or cut-outs redrawn

Commit message: wip pcb
Parts:
- KD13, KE13, KF13: footprint keyboard:SW_Cherry_MX_1.25u_SK6812MINI_Rotated -> keyboard:SW_Cherry_MX_1.25u_SK6812MINI
- moved U0 37.5 mm to (357.5, 93.2), turned to 90 degrees
- moved DF13 17.2 mm to (372.6, 162.3), turned to 90 degrees
- moved DE13 17.0 mm to (372.6, 143.0), turned to 90 degrees
- moved DD13 17.0 mm to (372.6, 124.0), turned to 90 degrees
- moved KF13 4.76 mm to (364.2, 157.1)
- moved KE13 4.76 mm to (364.2, 138.1)
- moved KD13 4.75 mm to (364.2, 119.0)
- moved DA13 1.72 mm to (381.5, 98.0)
- moved SW99 1.62 mm to (371.5, 93.0)
- moved R1 1.42 mm to (333.6, 98.7)
- moved R2 1.42 mm to (336.3, 98.7)
- moved J1 1.00 mm to (349.5, 107.0)
Connections:
- KB13 pad 1: Net-(KB12-Pad3) -> Net-(KB13-Pad1)
- KD12 pad 3: Net-(KD12-Pad3) -> LEDR2
- KD13 pad 1: Net-(KD12-Pad3) -> Net-(KD13-Pad1)
- KD13 pad 3: LEDR2 -> LEDR5
- KE12 pad 3: Net-(KE12-Pad3) -> LEDR3
- KE13 pad 1: Net-(KE12-Pad3) -> Net-(KE13-Pad1)
- KE13 pad 3: LEDR3 -> Net-(KD13-Pad1)
- KF0 pad 1: Net-(KF0-Pad1) -> LEDR5
- KF12 pad 3: Net-(KF12-Pad3) -> LEDR4
- KF13 pad 1: Net-(KF12-Pad3) -> Net-(KF13-Pad1)
- KF13 pad 3: LEDR4 -> Net-(KE13-Pad1)
Routing:
- net VCC: track 343.2 -> 1905.8 mm, vias 1 -> 10
- net row05: track 49.3 -> 408.2 mm, vias 0 -> 1
- net row03: track 48.3 -> 374.4 mm
- net row04: track 48.3 -> 369.5 mm
- net row00: track 48.3 -> 329.0 mm
- net row02: track 48.3 -> 316.0 mm
- net row01: track 48.3 -> 306.5 mm
- net col07: track 0.00 -> 163.4 mm, vias 0 -> 10
- net col06: track 0.00 -> 157.1 mm, vias 0 -> 10
- net col05: track 0.00 -> 152.4 mm, vias 0 -> 10
- net col01: track 0.00 -> 135.5 mm, vias 0 -> 10
- net col02: track 0.00 -> 135.0 mm, vias 0 -> 10
- net col04: track 0.00 -> 131.0 mm, vias 0 -> 10
- net col03: track 0.00 -> 126.4 mm, vias 0 -> 10
- net col00: track 0.00 -> 109.0 mm
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Other:
- outline, holes or cut-outs redrawn
- net class Default: trace_width 0.25 -> 0.254

Commit message: update pcb
Parts:
- removed G***: LOGO, layout-for-export:Dwgs.User_g222
- moved U0 45.5 mm to (355.1, 138.7), turned to 0 degrees
- moved DD13 12.7 mm to (385.3, 123.4)
- moved DE13 12.7 mm to (385.3, 142.5)
- moved DF13 12.7 mm to (385.3, 161.8)
- moved KD13 12.7 mm to (376.9, 118.5)
- moved KF13 12.7 mm to (376.9, 156.6)
- moved KE13 12.7 mm to (376.9, 137.6)
- moved R2 8.18 mm to (343.7, 102.2), turned to 0 degrees
- moved J1 7.91 mm to (357.4, 107.8)
- moved R1 7.61 mm to (341.2, 99.4), turned to 0 degrees
Routing:
- net col09: track 0.00 -> 174.4 mm, vias 0 -> 10
- net col08: track 0.00 -> 159.9 mm, vias 0 -> 10
- net VCC: track 1905.8 -> 2021.0 mm
- net row03: track 374.4 -> 322.0 mm
- net ENCA: track 30.1 -> 0.00 mm
- net row00: track 329.0 -> 305.8 mm
- net row04: track 369.5 -> 346.8 mm
- net row05: track 408.2 -> 385.9 mm
- net ENCB: track 22.0 -> 0.93 mm
- net LED: track 47.2 -> 63.6 mm
- net SCL: track 10.8 -> 21.3 mm
- net SDA: track 10.8 -> 21.1 mm
- net SW99B: track 0.00 -> 6.78 mm
- net col03: track 126.4 -> 130.1 mm
- net col05: track 152.4 -> 155.5 mm
Other:
- board size 334.8 x 145.8 mm -> 334 x 143.3 mm
