File: Kanagawa/Kanagawa/Kanagawa.kicad_pcb (KiCad board)
At the start: 2 copper layers, 334 x 143.3 mm, 174 parts, among them J0 Conn_01x03, J1 Conn_01x04, SW99 Rotary_Encoder_Switch, U0 Pico

Commit message: wip routing
Parts:
- moved J0 32.2 mm to (328.2, 88.2), turned to 90 degrees
- moved DA13 2.47 mm to (384.0, 97.9)
- moved SW99 2.47 mm to (374.0, 92.9)
Connections:
- net SW99A renamed col13
- net SW99B renamed /SW99B
- KB13 pad 1: Net-(KB13-Pad1) -> Net-(KB12-Pad3)
- U0 pad 21: col05 -> col12
- U0 pad 22: col06 -> col11
- U0 pad 24: col07 -> col10
- U0 pad 25: col08 -> col09
- U0 pad 26: col09 -> col08
- U0 pad 27: col10 -> col07
- U0 pad 29: col11 -> col06
- U0 pad 31: col12 -> col05
Routing:
- net LEDR5: track 0.00 -> 416.6 mm, vias 0 -> 2
- net col00: track 109.0 -> 437.9 mm
- net LEDR3: track 0.00 -> 325.2 mm, vias 0 -> 6
- net col01: track 135.5 -> 438.7 mm
- net LEDR1: track 0.00 -> 298.0 mm, vias 0 -> 2
- net LEDR4: track 0.00 -> 296.6 mm
- net col02: track 135.0 -> 429.8 mm
- net col03: track 130.1 -> 411.9 mm
- net col04: track 131.0 -> 396.1 mm
- net col10: track 0.00 -> 254.4 mm, vias 0 -> 10
- net col11: track 0.00 -> 236.6 mm, vias 0 -> 11
- net col05: track 155.5 -> 367.7 mm, vias 10 -> 11
- net col12: track 0.00 -> 194.9 mm, vias 0 -> 9
- net col13: track 0.00 -> 181.9 mm, vias 0 -> 6
- net col06: track 157.1 -> 335.1 mm
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
Commit message: rework routing
Connections:
- KB0 pad 1: LEDR1 -> /LEDKB0
- KB0 pad 3: Net-(KB0-Pad3) -> LEDR0
- KB1 pad 1: Net-(KB0-Pad3) -> /LEDKB1
- KB1 pad 3: Net-(KB1-Pad3) -> /LEDKB0
- KB10 pad 1: Net-(KB10-Pad1) -> /LEDKB10
- KB10 pad 3: Net-(KB10-Pad3) -> /LEDKB9
- KB11 pad 1: Net-(KB10-Pad3) -> /LEDKB11
- KB11 pad 3: Net-(KB11-Pad3) -> /LEDKB10
- KB12 pad 1: Net-(KB11-Pad3) -> /LEDKB12
- KB12 pad 3: Net-(KB12-Pad3) -> /LEDKB11
- KB13 pad 1: Net-(KB12-Pad3) -> LEDR1
- KB13 pad 3: LEDR0 -> /LEDKB12
- KB2 pad 1: Net-(KB1-Pad3) -> /LEDKB2
- KB2 pad 3: Net-(KB2-Pad3) -> /LEDKB1
- KB3 pad 1: Net-(KB2-Pad3) -> /LEDKB3
- KB3 pad 3: Net-(KB3-Pad3) -> /LEDKB2
- KB4 pad 1: Net-(KB3-Pad3) -> /LEDKB4
- KB4 pad 3: Net-(KB4-Pad3) -> /LEDKB3
- KB5 pad 1: Net-(KB4-Pad3) -> /LEDKB5
- KB5 pad 3: Net-(KB5-Pad3) -> /LEDKB4
- KB6 pad 1: Net-(KB5-Pad3) -> /LEDKB6
- KB6 pad 3: Net-(KB6-Pad3) -> /LEDKB5
- KB7 pad 1: Net-(KB6-Pad3) -> /LEDKB7
- KB7 pad 3: Net-(KB7-Pad3) -> /LEDKB6
- KB8 pad 1: Net-(KB7-Pad3) -> /LEDKB8
- KB8 pad 3: Net-(KB8-Pad3) -> /LEDKB7
- KB9 pad 1: Net-(KB8-Pad3) -> /LEDKB9
- KB9 pad 3: Net-(KB10-Pad1) -> /LEDKB8
- KD0 pad 1: LEDR3 -> /LEDKD0
- KD0 pad 3: Net-(KD0-Pad3) -> LEDR2
- KD1 pad 1: Net-(KD0-Pad3) -> /LEDKD1
- KD1 pad 3: Net-(KD1-Pad3) -> /LEDKD0
- KD10 pad 1: Net-(KD10-Pad1) -> /LEDKD10
- KD10 pad 3: Net-(KD10-Pad3) -> /LEDKD9
- KD11 pad 1: Net-(KD10-Pad3) -> /LEDKD11
- KD11 pad 3: Net-(KD11-Pad3) -> /LEDKD10
- KD12 pad 1: Net-(KD11-Pad3) -> LEDR3
- KD12 pad 3: LEDR2 -> /LEDKD11
- KD13 pad 3: LEDR5 -> Net-(KD13-Pad3)
- KD2 pad 1: Net-(KD1-Pad3) -> /LEDKD2
- KD2 pad 3: Net-(KD2-Pad3) -> /LEDKD1
- KD3 pad 1: Net-(KD2-Pad3) -> /LEDKD3
- KD3 pad 3: Net-(KD3-Pad3) -> /LEDKD2
- KD4 pad 1: Net-(KD3-Pad3) -> /LEDKD4
- KD4 pad 3: Net-(KD4-Pad3) -> /LEDKD3
- KD5 pad 1: Net-(KD4-Pad3) -> /LEDKD5
- KD5 pad 3: Net-(KD5-Pad3) -> /LEDKD4
- KD6 pad 1: Net-(KD5-Pad3) -> /LEDKD6
- KD6 pad 3: Net-(KD6-Pad3) -> /LEDKD5
- KD7 pad 1: Net-(KD6-Pad3) -> /LEDKD7
- KD7 pad 3: Net-(KD7-Pad3) -> /LEDKD6
- KD8 pad 1: Net-(KD7-Pad3) -> /LEDKD8
- KD8 pad 3: Net-(KD8-Pad3) -> /LEDKD7
- KD9 pad 1: Net-(KD8-Pad3) -> /LEDKD9
- KD9 pad 3: Net-(KD10-Pad1) -> /LEDKD8
- KE13 pad 1: Net-(KE13-Pad1) -> Net-(KD13-Pad3)
- KE13 pad 3: Net-(KD13-Pad1) -> Net-(KE13-Pad3)
- KF0 pad 1: LEDR5 -> /LEDKF0
- KF0 pad 3: Net-(KF0-Pad3) -> LEDR4
- KF1 pad 1: Net-(KF0-Pad3) -> /LEDKF1
- KF1 pad 3: Net-(KF1-Pad3) -> /LEDKF0
- KF10 pad 1: Net-(KF10-Pad1) -> /LEDKF10
- KF10 pad 3: Net-(KF10-Pad3) -> /LEDKF9
- KF11 pad 1: Net-(KF10-Pad3) -> /LEDKF11
- KF11 pad 3: Net-(KF11-Pad3) -> /LEDKF10
- KF12 pad 1: Net-(KF11-Pad3) -> /LEDKF12
- KF12 pad 3: LEDR4 -> /LEDKF11
- KF13 pad 1: Net-(KF13-Pad1) -> Net-(KE13-Pad3)
- KF13 pad 3: Net-(KE13-Pad1) -> /LEDKF12
- KF2 pad 1: Net-(KF1-Pad3) -> /LEDKF2
- KF2 pad 3: Net-(KF2-Pad3) -> /LEDKF1
- KF3 pad 1: Net-(KF2-Pad3) -> /LEDKF3
- KF3 pad 3: Net-(KF3-Pad3) -> /LEDKF2
- KF4 pad 1: Net-(KF3-Pad3) -> /LEDKF4
- KF4 pad 3: Net-(KF4-Pad3) -> /LEDKF3
- KF5 pad 1: Net-(KF4-Pad3) -> /LEDKF5
- KF5 pad 3: Net-(KF5-Pad3) -> /LEDKF4
- KF6 pad 1: Net-(KF5-Pad3) -> /LEDKF6
- KF6 pad 3: Net-(KF6-Pad3) -> /LEDKF5
- KF7 pad 1: Net-(KF6-Pad3) -> /LEDKF7
- KF7 pad 3: Net-(KF7-Pad3) -> /LEDKF6
- KF8 pad 1: Net-(KF7-Pad3) -> /LEDKF8
- KF8 pad 3: Net-(KF8-Pad3) -> /LEDKF7
- KF9 pad 1: Net-(KF8-Pad3) -> /LEDKF9
- KF9 pad 3: Net-(KF10-Pad1) -> /LEDKF8
Routing:
- net LEDR5: track 416.6 -> 0.00 mm, vias 2 -> 0
- net LEDR1: track 298.0 -> 0.00 mm, vias 2 -> 0
- net LEDR4: track 296.6 -> 0.33 mm
- net LEDR3: track 325.2 -> 267.1 mm, vias 6 -> 2
- net Net-(KF4-Pad3): track 42.1 -> 0.00 mm
- net Net-(KD13-Pad1): track 30.1 -> 0.00 mm
- net Net-(KE13-Pad1): track 30.1 -> 0.00 mm
- net Net-(KD11-Pad3): track 28.9 -> 0.00 mm
- net Net-(KF3-Pad3): track 25.8 -> 0.00 mm
- net Net-(KF5-Pad3): track 25.7 -> 0.00 mm
- net Net-(KB12-Pad3): track 24.5 -> 0.00 mm
- net Net-(KF10-Pad1): track 23.0 -> 0.00 mm
- net Net-(KD0-Pad3): track 22.0 -> 0.00 mm
- net Net-(KF6-Pad3): track 19.1 -> 0.00 mm
- net Net-(KF2-Pad3): track 18.8 -> 0.00 mm
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
Commit message: Kanagawa routing
Parts:
- removed J0: Conn_01x03, keyboard:conn_3pins
- removed REF**: Keebio_USB-C_breakout_shadow, keyboard:Keebio_USB-C_breakout_shadow
- added LogoMiddle: LOGO, Pallas:Ciaanh_signature, F.Cu at (382.9, 197.2)
- added MountBaseMiddleTop1: MountingHole, keyboard:MountingHole_2.2mm_M2_Pad_Via, F.Cu at (60.9, 83.2)
- added MountBaseMiddleTop2: MountingHole, keyboard:MountingHole_2.2mm_M2_Pad_Via, F.Cu at (60.9, 205.2)
- added MountBaseMiddleTop3: MountingHole, keyboard:MountingHole_2.2mm_M2_Pad_Via, F.Cu at (382.9, 83.2)
- added MountBaseMiddleTop4: MountingHole, keyboard:MountingHole_2.2mm_M2_Pad_Via, F.Cu at (382.9, 205.2)
- added MountBaseMiddleTop5: MountingHole, keyboard:MountingHole_2.2mm_M2_Pad_Via, F.Cu at (267.0, 146.0)
- added MountBaseMiddleTop6: MountingHole, keyboard:MountingHole_2.2mm_M2_Pad_Via, F.Cu at (153.0, 146.0)
- added MountBaseMiddleTop7: MountingHole, keyboard:MountingHole_2.2mm_M2_Pad_Via, F.Cu at (210.9, 109.2)
- added MountBaseMiddleTop8: MountingHole, keyboard:MountingHole_2.2mm_M2_Pad_Via, F.Cu at (185.7, 217.2)
- added MountMiddle0: MountingHole USB breakout, keyboard:Keebio_USB-C_breakout_shadow, F.Cu at (214.9, 85.2)
- added RSW0: SW_RST, keyboard:SW_RST, F.Cu at (324.2, 80.0)
- KA0, KA1, KA10, KA11, KA12, KA2, KA3, KA4, KA5, KA6, KA7, KA8, KA9, KB0, KB1, KB10, KB11, KB12, KB2, KB3, KB4, KB5, KB6, KB7, KB8, KB9, KC1, KC10, KC11, KC12, KC2, KC3, KC4, KC5, KC6, KC7, KC8, KC9, KD1, KD10, KD11, KD2, KD3, KD4, KD5, KD6, KD7, KD8, KD9, KE1, KE10, KE12, KE2, KE3, KE4, KE5, KE6, KE7, KE8, KE9, KF1, KF10, KF11, KF12, KF3, KF6, KF8: footprint keyboard:SW_Cherry_MX_1.00u_SK6812MINI -> keyboard:SW_Cherry_MX_1.00u_Hotswap
- KB13, KD12, KF4, KF5: footprint keyboard:SW_Cherry_MX_2.00u_SK6812MINI -> keyboard:SW_Cherry_MX_2.00u_Hotswap
- KC0, KC13: footprint keyboard:SW_Cherry_MX_1.50u_SK6812MINI -> keyboard:SW_Cherry_MX_1.50u_Hotswap
- KD0: footprint keyboard:SW_Cherry_MX_1.75u_SK6812MINI -> keyboard:SW_Cherry_MX_1.75u_Hotswap
- KD13, KE13, KF0, KF13, KF2, KF7, KF9: footprint keyboard:SW_Cherry_MX_1.25u_SK6812MINI -> keyboard:SW_Cherry_MX_1.25u_Hotswap
- KE0, KE11: footprint keyboard:SW_Cherry_MX_2.25u_SK6812MINI -> keyboard:SW_Cherry_MX_2.25u_Hotswap
- U0: value Pico -> Elite-C; footprint keyboard:RPi_Pico_TH -> keyboard:Elite-C-29pin-holes
- moved J1 36.4 mm to (332.7, 80.9), turned to 0 degrees
- moved DF4 28.7 mm to (179.9, 214.1), turned to 75 degrees
- moved DF6 26.0 mm to (244.4, 199.7), turned to 105 degrees
- moved DB13 25.8 mm to (341.3, 123.5), turned to 90 degrees
- moved DF5 23.5 mm to (225.5, 204.9), turned to 105 degrees
- moved DF3 17.4 mm to (143.4, 204.1), turned to 75 degrees
- moved R2 16.2 mm to (346.2, 86.1), turned to 270 degrees
- moved R1 15.4 mm to (349.0, 86.1), turned to 270 degrees
- moved U0 7.19 mm to (353.9, 131.6), turned to 270 degrees
- moved DA13 2.67 mm to (384.0, 100.6)
- moved DD13 2.00 mm to (383.3, 123.4)
- moved DE13 2.00 mm to (383.3, 142.5)
- moved DF13 2.00 mm to (383.3, 161.8)
- moved KD13 2.00 mm to (374.9, 118.5)
- moved KE13 2.00 mm to (374.9, 137.6)
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Connections:
- KA0 pad 1: LEDR0 -> col00
- KA0 pad 2: VCC -> Net-(DA0-Pad2)
- KA1 pad 1: Net-(KA0-Pad3) -> col01
- KA1 pad 2: VCC -> Net-(DA1-Pad2)
- KA10 pad 1: Net-(KA10-Pad1) -> col10
- KA10 pad 2: VCC -> Net-(DA10-Pad2)
- KA11 pad 1: Net-(KA10-Pad3) -> col11
- KA11 pad 2: VCC -> Net-(DA11-Pad2)
- KA12 pad 1: Net-(KA11-Pad3) -> col12
- KA12 pad 2: VCC -> Net-(DA12-Pad2)
- KA2 pad 1: Net-(KA1-Pad3) -> col02
- KA2 pad 2: VCC -> Net-(DA2-Pad2)
- KA3 pad 1: Net-(KA2-Pad3) -> col03
- KA3 pad 2: VCC -> Net-(DA3-Pad2)
- KA4 pad 1: Net-(KA3-Pad3) -> col04
- KA4 pad 2: VCC -> Net-(DA4-Pad2)
- KA5 pad 1: Net-(KA4-Pad3) -> col05
- KA5 pad 2: VCC -> Net-(DA5-Pad2)
- KA6 pad 1: Net-(KA5-Pad3) -> col06
- KA6 pad 2: VCC -> Net-(DA6-Pad2)
- KA7 pad 1: Net-(KA6-Pad3) -> col07
- KA7 pad 2: VCC -> Net-(DA7-Pad2)
- KA8 pad 1: Net-(KA7-Pad3) -> col08
- KA8 pad 2: VCC -> Net-(DA8-Pad2)
- KA9 pad 1: Net-(KA8-Pad3) -> col09
- KA9 pad 2: VCC -> Net-(DA9-Pad2)
- KB0 pad 1: /LEDKB0 -> col00
- KB0 pad 2: VCC -> Net-(DB0-Pad2)
- KB1 pad 1: /LEDKB1 -> col01
- KB1 pad 2: VCC -> Net-(DB1-Pad2)
- KB10 pad 1: /LEDKB10 -> col10
- KB10 pad 2: VCC -> Net-(DB10-Pad2)
- KB11 pad 1: /LEDKB11 -> col11
- KB11 pad 2: VCC -> Net-(DB11-Pad2)
- KB12 pad 1: /LEDKB12 -> col12
- KB12 pad 2: VCC -> Net-(DB12-Pad2)
- KB13 pad 1: LEDR1 -> col13
- KB13 pad 2: VCC -> Net-(DB13-Pad2)
- KB2 pad 1: /LEDKB2 -> col02
- KB2 pad 2: VCC -> Net-(DB2-Pad2)
- KB3 pad 1: /LEDKB3 -> col03
- KB3 pad 2: VCC -> Net-(DB3-Pad2)
- KB4 pad 1: /LEDKB4 -> col04
- KB4 pad 2: VCC -> Net-(DB4-Pad2)
- KB5 pad 1: /LEDKB5 -> col05
- KB5 pad 2: VCC -> Net-(DB5-Pad2)
- KB6 pad 1: /LEDKB6 -> col06
- KB6 pad 2: VCC -> Net-(DB6-Pad2)
- KB7 pad 1: /LEDKB7 -> col07
- KB7 pad 2: VCC -> Net-(DB7-Pad2)
- KB8 pad 1: /LEDKB8 -> col08
- KB8 pad 2: VCC -> Net-(DB8-Pad2)
- KB9 pad 1: /LEDKB9 -> col09
- KB9 pad 2: VCC -> Net-(DB9-Pad2)
- KC0 pad 1: LEDR2 -> col00
- KC0 pad 2: VCC -> Net-(DC0-Pad2)
- KC1 pad 1: Net-(KC0-Pad3) -> col01
- KC1 pad 2: VCC -> Net-(DC1-Pad2)
- KC10 pad 1: Net-(KC10-Pad1) -> col10
- KC10 pad 2: VCC -> Net-(DC10-Pad2)
- KC11 pad 1: Net-(KC10-Pad3) -> col11
- KC11 pad 2: VCC -> Net-(DC11-Pad2)
- KC12 pad 1: Net-(KC11-Pad3) -> col12
- KC12 pad 2: VCC -> Net-(DC12-Pad2)
- KC13 pad 1: Net-(KC12-Pad3) -> col13
- KC13 pad 2: VCC -> Net-(DC13-Pad2)
- KC2 pad 1: Net-(KC1-Pad3) -> col02
- KC2 pad 2: VCC -> Net-(DC2-Pad2)
- KC3 pad 1: Net-(KC2-Pad3) -> col03
- KC3 pad 2: VCC -> Net-(DC3-Pad2)
- KC4 pad 1: Net-(KC3-Pad3) -> col04
- KC4 pad 2: VCC -> Net-(DC4-Pad2)
- KC5 pad 1: Net-(KC4-Pad3) -> col05
- KC5 pad 2: VCC -> Net-(DC5-Pad2)
- KC6 pad 1: Net-(KC5-Pad3) -> col06
- KC6 pad 2: VCC -> Net-(DC6-Pad2)
- KC7 pad 1: Net-(KC6-Pad3) -> col07
- KC7 pad 2: VCC -> Net-(DC7-Pad2)
- KC8 pad 1: Net-(KC7-Pad3) -> col08
- KC8 pad 2: VCC -> Net-(DC8-Pad2)
- KC9 pad 1: Net-(KC8-Pad3) -> col09
- KC9 pad 2: VCC -> Net-(DC9-Pad2)
- KD0 pad 1: /LEDKD0 -> col00
- KD0 pad 2: VCC -> Net-(DD0-Pad2)
- KD1 pad 1: /LEDKD1 -> col01
- KD1 pad 2: VCC -> Net-(DD1-Pad2)
- KD10 pad 1: /LEDKD10 -> col10
- KD10 pad 2: VCC -> Net-(DD10-Pad2)
- KD11 pad 1: /LEDKD11 -> col11
- KD11 pad 2: VCC -> Net-(DD11-Pad2)
- KD12 pad 1: LEDR3 -> col12
- KD12 pad 2: VCC -> Net-(DD12-Pad2)
- KD13 pad 1: Net-(KD13-Pad1) -> col13
- KD13 pad 2: VCC -> Net-(DD13-Pad2)
- KD2 pad 1: /LEDKD2 -> col02
- KD2 pad 2: VCC -> Net-(DD2-Pad2)
- KD3 pad 1: /LEDKD3 -> col03
- KD3 pad 2: VCC -> Net-(DD3-Pad2)
- KD4 pad 1: /LEDKD4 -> col04
- KD4 pad 2: VCC -> Net-(DD4-Pad2)
- KD5 pad 1: /LEDKD5 -> col05
- KD5 pad 2: VCC -> Net-(DD5-Pad2)
- KD6 pad 1: /LEDKD6 -> col06
- KD6 pad 2: VCC -> Net-(DD6-Pad2)
- KD7 pad 1: /LEDKD7 -> col07
- KD7 pad 2: VCC -> Net-(DD7-Pad2)
- KD8 pad 1: /LEDKD8 -> col08
- KD8 pad 2: VCC -> Net-(DD8-Pad2)
- KD9 pad 1: /LEDKD9 -> col09
- KD9 pad 2: VCC -> Net-(DD9-Pad2)
- KE0 pad 1: LEDR4 -> col00
- KE0 pad 2: VCC -> Net-(DE0-Pad2)
- KE1 pad 1: Net-(KE0-Pad3) -> col01
- KE1 pad 2: VCC -> Net-(DE1-Pad2)
- KE10 pad 1: Net-(KE10-Pad1) -> col10
- KE10 pad 2: VCC -> Net-(DE10-Pad2)
- KE11 pad 1: Net-(KE10-Pad3) -> col11
- KE11 pad 2: VCC -> Net-(DE11-Pad2)
- KE12 pad 1: Net-(KE11-Pad3) -> col12
- KE12 pad 2: VCC -> Net-(DE12-Pad2)
- KE13 pad 1: Net-(KD13-Pad3) -> col13
- KE13 pad 2: VCC -> Net-(DE13-Pad2)
- KE2 pad 1: Net-(KE1-Pad3) -> col02
- KE2 pad 2: VCC -> Net-(DE2-Pad2)
- KE3 pad 1: Net-(KE2-Pad3) -> col03
- KE3 pad 2: VCC -> Net-(DE3-Pad2)
- KE4 pad 1: Net-(KE3-Pad3) -> col04
- KE4 pad 2: VCC -> Net-(DE4-Pad2)
- KE5 pad 1: Net-(KE4-Pad3) -> col05
- KE5 pad 2: VCC -> Net-(DE5-Pad2)
- KE6 pad 1: Net-(KE5-Pad3) -> col06
- KE6 pad 2: VCC -> Net-(DE6-Pad2)
- KE7 pad 1: Net-(KE6-Pad3) -> col07
- KE7 pad 2: VCC -> Net-(DE7-Pad2)
- KE8 pad 1: Net-(KE7-Pad3) -> col08
- KE8 pad 2: VCC -> Net-(DE8-Pad2)
- KE9 pad 1: Net-(KE8-Pad3) -> col09
- KE9 pad 2: VCC -> Net-(DE9-Pad2)
- KF0 pad 1: /LEDKF0 -> col00
- KF0 pad 2: VCC -> Net-(DF0-Pad2)
- KF1 pad 1: /LEDKF1 -> col01
- KF1 pad 2: VCC -> Net-(DF1-Pad2)
- KF10 pad 1: /LEDKF10 -> col10
- KF10 pad 2: VCC -> Net-(DF10-Pad2)
- KF11 pad 1: /LEDKF11 -> col11
- KF11 pad 2: VCC -> Net-(DF11-Pad2)
- KF12 pad 1: /LEDKF12 -> col12
- KF12 pad 2: VCC -> Net-(DF12-Pad2)
- KF13 pad 1: Net-(KE13-Pad3) -> col13
- KF13 pad 2: VCC -> Net-(DF13-Pad2)
- KF2 pad 1: /LEDKF2 -> col02
- KF2 pad 2: VCC -> Net-(DF2-Pad2)
- KF3 pad 1: /LEDKF3 -> col03
- KF3 pad 2: VCC -> Net-(DF3-Pad2)
- KF4 pad 1: /LEDKF4 -> col04
- KF4 pad 2: VCC -> Net-(DF4-Pad2)
- KF5 pad 1: /LEDKF5 -> col05
- KF5 pad 2: VCC -> Net-(DF5-Pad2)
- KF6 pad 1: /LEDKF6 -> col06
- KF6 pad 2: VCC -> Net-(DF6-Pad2)
- KF7 pad 1: /LEDKF7 -> col07
- KF7 pad 2: VCC -> Net-(DF7-Pad2)
- KF8 pad 1: /LEDKF8 -> col08
- KF8 pad 2: VCC -> Net-(DF8-Pad2)
- KF9 pad 1: /LEDKF9 -> col09
- KF9 pad 2: VCC -> Net-(DF9-Pad2)
- U0 pad 1: SDA -> col13
- U0 pad 10: row02 -> col08
- U0 pad 11: row03 -> col07
- U0 pad 12: row04 -> col06
- U0 pad 13: GND -> col00
- U0 pad 14: row05 -> row00
- U0 pad 15: col00 -> row01
- U0 pad 16: col01 -> row02
- U0 pad 17: col02 -> row03
- U0 pad 18: GND -> row04
- U0 pad 19: col03 -> row05
- U0 pad 2: SCL -> col12
- U0 pad 20: col04 -> ENCB
- U0 pad 21: col12 -> VCC
- U0 pad 22: col11 -> RESET
- U0 pad 24: col10 -> ENCA
- U0 pad 25: col09 -> col05
- U0 pad 26: col08 -> col04
- U0 pad 27: col07 -> col03
- U0 pad 28: GND -> col02
- U0 pad 29: col06 -> col01
- U0 pad 4: LED -> GND
- U0 pad 5: ENCA -> SDA
- U0 pad 6: ENCB -> SCL
- U0 pad 7: row00 -> col11
- U0 pad 8: GND -> col10
- U0 pad 9: row01 -> col09
Routing:
- net VCC: track 2072.7 -> 55.7 mm, vias 15 -> 1
- net LEDR3: track 267.1 -> 0.00 mm, vias 2 -> 0
- net RESET: track 0.00 -> 59.3 mm
- net row04: track 438.0 -> 385.7 mm, vias 0 -> 1
- net col13: track 181.9 -> 142.5 mm, vias 6 -> 2
- net col08: track 285.7 -> 320.6 mm, vias 10 -> 1
- net Net-(KE11-Pad3): track 33.5 -> 0.00 mm, vias 2 -> 0
- net LED: track 33.0 -> 0.00 mm, vias 2 -> 0
- net row03: track 409.0 -> 378.2 mm, vias 0 -> 1
- net row00: track 404.3 -> 434.2 mm, vias 2 -> 0
- net SCL: track 21.3 -> 49.9 mm, vias 0 -> 1
- net Net-(KE0-Pad3): track 27.6 -> 0.00 mm
- net col10: track 254.4 -> 282.0 mm, vias 10 -> 1
- net Net-(KE10-Pad3): track 26.8 -> 0.00 mm
- net SDA: track 21.1 -> 47.9 mm, vias 0 -> 1
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Other:
- board size 334 x 143.3 mm -> 332 x 143 mm
- board text added: "Kanagawa rev 0.1 *prototype*"

Commit message: update pcb
Parts:
- LogoMiddle: footprint Pallas:Ciaanh_signature -> keyboard:Ciaanh_signature; moved to B.Cu
- moved MountBaseMiddleTop3 201.9 mm to (185.9, 127.2)
- moved MountBaseMiddleTop8 197.6 mm to (382.9, 205.2)
- moved MountBaseMiddleTop4 196.9 mm to (186.0, 210.0)
- moved MountBaseMiddleTop7 174.0 mm to (382.9, 83.2)
- moved MountBaseMiddleTop6 131.0 mm to (270.0, 205.0)
- moved MountBaseMiddleTop5 62.8 mm to (270.0, 83.2)
- moved LogoMiddle 49.3 mm to (356.9, 155.3), turned to 210 degrees

Commit message: edit kanagawa
Parts:
- removed LogoMiddle: LOGO, keyboard:Ciaanh_signature
- added LogoBase1: LOGO, layout-for-export:Great-wave, B.Cu at (222.9, 150.2)
- added LogoMiddle0: LOGO, keyboard:Ciaanh_signature_back, B.Cu at (372.2, 175.0)
- added LogoMiddle1: cc_logo, keyboard:cc, B.Cu at (383.0, 175.1)
- added LogoMiddle2: oshw_logo, keyboard:oshw, B.Cu at (382.7, 185.4)
- moved MountBaseMiddleTop3 4.57 mm to (190.4, 127.6)
Other:
- outline, holes or cut-outs redrawn
