File: Kanagawa/Kanagawa/Kanagawa.sch (KiCad schematic (older format))
At the start: 173 parts, among them J0 Conn_01x03, J1 Conn_01x04, SW99 Rotary_Encoder_Switch, U0 Pico

Commit message: Begin placing footprints
Parts:
- KA10, KA11, KA12, KA2, KA3, KA4, KA5, KA6, KA7, KA8, KA9, KB0, KB1, KB10, KB11, KB12, KB13, KB14, KB2, KB3, KB4, KB5, KB6, KB7, KB8, KB9, KC0, KC1, KC10, KC11, KC12, KC13, KC14, KC2, KC3, KC4, KC5, KC6, KC7, KC8, KC9, KD0, KD1, KD10, KD11, KD12, KD13, KD2, KD3, KD4, KD5, KD6, KD7, KD8, KD9, KE0, KE1, KE10, KE11, KE12, KE2, KE3, KE4, KE5, KE6, KE7, KE8, KE9, KF0, KF1, KF10, KF11, KF12, KF2, KF3, KF4, KF5, KF6, KF7, KF8, KF9: footprint (none) -> keyboard:SW_Cherry_MX_1.00u_SK6812MINI

Commit message: update footprint
Parts:
- KB13, KD12, KF4, KF5: footprint keyboard:SW_Cherry_MX_1.00u_SK6812MINI -> keyboard:SW_Cherry_MX_2.00u_SK6812MINI
- KC0, KC12: footprint keyboard:SW_Cherry_MX_1.00u_SK6812MINI -> keyboard:SW_Cherry_MX_1.50u_SK6812MINI
- KD0: footprint keyboard:SW_Cherry_MX_1.00u_SK6812MINI -> keyboard:SW_Cherry_MX_1.75u_SK6812MINI
- KD13, KF0, KF2, KF7, KF9: footprint keyboard:SW_Cherry_MX_1.00u_SK6812MINI -> keyboard:SW_Cherry_MX_1.25u_SK6812MINI
- KE0, KE11: footprint keyboard:SW_Cherry_MX_1.00u_SK6812MINI -> keyboard:SW_Cherry_MX_2.25u_SK6812MINI
- KE13: renamed from KB14; footprint keyboard:SW_Cherry_MX_1.00u_SK6812MINI -> keyboard:SW_Cherry_MX_1.25u_SK6812MINI
- KF13: renamed from KC14; footprint keyboard:SW_Cherry_MX_1.00u_SK6812MINI -> keyboard:SW_Cherry_MX_1.25u_SK6812MINI
- U0: footprint RPi_Pico:RPi_Pico_SMD_TH -> RP-Pico:RPi_Pico_SMD_TH
- renumbered DA14 to DA13, DB14 to DE13, DC14 to DF13
Connections:
- net col13 is gone; now on net SW99A: KB13.5, KC13.5, KD13.5, U0.32 (GPIO27_ADC1)
- net LEDR0: now also KB13.3 (DIN); no longer KE13.3 (DIN)
- net LEDR1: now also KC13.3 (DIN); no longer KF13.3 (DIN)
- net LEDR3: now also KE13.3 (DIN); no longer KE12.3 (DIN)
- net LEDR4: now also KF13.3 (DIN); no longer KF12.3 (DIN)
- net SW99A: no longer U0.34 (GPIO28_ADC2)
- net row01: no longer DE13.1 (K)
- net row02: no longer DF13.1 (K)
- net row04: now also DE13.1 (K)
- net row05: now also DF13.1 (K)
- net at KE13.1 (DOUT): now also KE12.3 (DIN); no longer KB13.3 (DIN)
- net at KF13.1 (DOUT): now also KF12.3 (DIN); no longer KC13.3 (DIN)
- no-connect marks 8 -> 9
Other:
- moved on the sheet: DA0, DA1, DA10, DA11, DA12, DA13, DA2, DA3, DA4, DA5, DA6, DA7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

Commit message: prepare pcb layout
Parts:
- KC12: footprint keyboard:SW_Cherry_MX_1.50u_SK6812MINI -> keyboard:SW_Cherry_MX_1.00u_SK6812MINI
- KC13: footprint keyboard:SW_Cherry_MX_1.00u_SK6812MINI -> keyboard:SW_Cherry_MX_1.50u_SK6812MINI
Changed lines of the file:
@@
 F 0 "KC12" H 19500 7345 50  0000 C CNN
 F 1 "KEY_SW" H 19500 7254 50  0000 C CNN
-F 2 "keyboard:SW_Cherry_MX_1.50u_SK6812MINI" H 19500 7090 50  0001 C CNN
+F 2 "keyboard:SW_Cherry_MX_1.00u_SK6812MINI" H 19500 7090 50  0001 C CNN
 F 3 "" H 19500 7090 50  0000 C CNN
 	1    19500 7090
@@
 F 0 "KC13" H 20940 7345 50  0000 C CNN
 F 1 "KEY_SW" H 20940 7254 50  0000 C CNN
-F 2 "keyboard:SW_Cherry_MX_1.00u_SK6812MINI" H 20940 7090 50  0001 C CNN
+F 2 "keyboard:SW_Cherry_MX_1.50u_SK6812MINI" H 20940 7090 50  0001 C CNN
 F 3 "" H 20940 7090 50  0000 C CNN
 	1    20940 7090

Commit message: update pcb
Parts:
- J1: footprint keyboard:conn_4pins -> keyboard:OLED_128x64_I2C
- U0: footprint RP-Pico:RPi_Pico_SMD_TH -> keyboard:RPi_Pico_TH
Changed lines of the file:
@@
 F 0 "U0" H 1650 3505 50  0000 C CNN
 F 1 "Pico" H 1650 3414 50  0000 C CNN
-F 2 "RP-Pico:RPi_Pico_SMD_TH" V 1650 2290 50  0001 C CNN
+F 2 "keyboard:RPi_Pico_TH" V 1650 2290 50  0001 C CNN
 F 3 "" H 1650 2290 50  0001 C CNN
 	1    1650 2290
@@
 F 0 "J1" H 4978 1275 50  0000 C CNN
 F 1 "Conn_01x04" H 4978 1366 50  0000 C CNN
-F 2 "keyboard:conn_4pins" H 5210 1300 50  0001 C CNN
+F 2 "keyboard:OLED_128x64_I2C" H 5210 1300 50  0001 C CNN
 F 3 "" H 5060 1700 50  0001 C CNN
 	1    5060 1700

Commit message: wip pcb
Connections:
- net LEDR2: now also KD12.3 (DIN); no longer KD13.3 (DIN)
- net LEDR3: now also KE12.3 (DIN); no longer KE13.3 (DIN)
- net LEDR4: now also KF12.3 (DIN); no longer KF13.3 (DIN)
- net at KB12.3 (DIN): no longer KB13.1 (DOUT)
- net at KD13.1 (DOUT): now also KE13.3 (DIN); no longer KD12.3 (DIN)
- net at KE13.1 (DOUT): now also KF13.3 (DIN); no longer KE12.3 (DIN)
- net at KF13.1 (DOUT): no longer KF12.3 (DIN)
- net LEDR5: now reaches KF0.1 (DOUT)
- net LEDR5: now also KD13.3 (DIN)
Changed lines of the file:
@@
 	20430 7240 20740 7240
-Wire Wire Line
-	19700 6410 20430 6410
-Wire Wire Line
-	20430 6410 20430 6310
-Wire Wire Line
-	20430 6310 20740 6310
 Wire Wire Line
 	18240 5480 18970 5480
@@
 Wire Wire Line
 	1880 9100 2060 9100
-Wire Wire Line
-	1880 10030 2060 10030
-NoConn ~ 1880 10030
 Text GLabel 21140 7340 2    50   Input ~ 0
 LEDR1
@@
 Connection ~ 16310 8950
 Connection ~ 15740 10370
-Text GLabel 21140 10130 2    50   Input ~ 0
+Text GLabel 19700 10130 2    50   Input ~ 0
 LEDR4
 $Comp
@@
 Wire Wire Line
 	18240 10130 18970 10130
-Wire Wire Line
-	19700 10130 20430 10130
 Wire Wire Line
 	16310 8950 16310 9880
@@
 Wire Wire Line
 	18970 9200 18970 9100
-Text GLabel 21140 9200 2    50   Input ~ 0
+Text GLabel 19700 9200 2    50   Input ~ 0
 LEDR3
 $Comp
@@
 Wire Wire Line
 	18970 9100 19300 9100
-Wire Wire Line
-	19700 9200 20430 9200
 Wire Wire Line
 	19200 8950 19200 9880
@@
 	0    -1   -1   0
 $EndComp
-Wire Wire Line
-	19700 8270 20430 8270
 $Comp
 L keyboard:KEY_SW_RGB KC13
@@
 Wire Wire Line
 	21490 8510 20050 8510
-Wire Wire Line
-	20430 8270 20430 8170
 Connection ~ 20640 7090
 $Comp
@@
 	-1   0    0    1
 $EndComp
-Text GLabel 21140 8270 2    50   Input ~ 0
+Text GLabel 19700 8270 2    50   Input ~ 0
 LEDR2
 Wire Wire Line
-	20430 8170 20740 8170
+	21490 8320 21490 8510
+Wire Wire Line
+	21240 8020 21490 8020
+$Comp
+L keyboard:GND #PWR0286
+U 1 1 6175EF70
+P 21270 8170
+F 0 "#PWR0286" H 21270 7920 50  0001 C CNN
+F 1 "GND" V 21275 8042 50  0000 R CNN
+F 2 "" H 21270 8170 50  0001 C CNN
+F 3 "" H 21270 8170 50  0001 C CNN
+	1    21270 8170
+	0    -1   -1   0
+$EndComp
+Wire Wire Line
+	21140 8170 21270 8170
+$Comp
+L keyboard:D DD13
+U 1 1 6175EF66
+P 21490 8170
+F 0 "DD13" V 21536 8091 50  0000 R CNN
+F 1 "D" V 21445 8091 50  0000 R CNN
+F 2 "keyboard:Diode_SMD_THT" H 21477 8004 50  0001 C CNN
+F 3 "" H 21490 8170 50  0001 C CNN
+	1    21490 8170
+	0    -1   -1   0
+$EndComp
+Wire Wire Line
+	21490 5530 21490 5720
+Wire Wire Line
+	21240 5230 21490 5230
+$Comp
+L keyboard:D DA13
+U 1 1 6175EFCD
+P 21490 5380
+F 0 "DA13" V 21536 5301 50  0000 R CNN
+F 1 "D" V 21445 5301 50  0000 R CNN
+F 2 "keyboard:Diode_SMD_THT" H 21477 5214 50  0001 C CNN
+F 3 "" H 21490 5380 50  0001 C CNN
+	1    21490 5380
+	0    -1   -1   0
+$EndComp
+Connection ~ 20050 9440
+Wire Wire Line
+	20640 8950 20640 9880
+Connection ~ 20640 8950
+Wire Wire Line
+	20050 10370 21490 10370
+Wire Wire Line
+	21490 10370 21490 10180
+Connection ~ 20050 10370
+Wire Wire Line
+	21490 9250 21490 9440
+Wire Wire Line
+	20050 9440 21490 9440
+NoConn ~ 2350 1940
+Wire Wire Line
+	19710 6410 20430 6410
+Wire Wire Line
+	20430 6410 20430 6310
+Wire Wire Line
+	20430 6310 20740 6310
+Wire Wire Line
+	20640 8020 20640 8950
 Wire Wire Line
 	20640 7090 20640 8020
+Connection ~ 20640 8020
 $Comp
 L keyboard:KEY_SW_RGB KD13
@@
 $EndComp
 Wire Wire Line
-	21490 8320 21490 8510
-Wire Wire Line
-	21240 8020 21490 8020
-$Comp
-L keyboard:GND #PWR0286
-U 1 1 6175EF70
-P 21270 8170
-F 0 "#PWR0286" H 21270 7920 50  0001 C CNN
-F 1 "GND" V 21275 8042 50  0000 R CNN
-F 2 "" H 21270 8170 50  0001 C CNN
-F 3 "" H 21270 8170 50  0001 C CNN
-	1    21270 8170
-	0    -1   -1   0
-$EndComp
-Wire Wire Line
-	21140 8170 21270 8170
-$Comp
-L keyboard:D DD13
-U 1 1 6175EF66
-P 21490 8170
-F 0 "DD13" V 21536 8091 50  0000 R CNN
-F 1 "D" V 21445 8091 50  0000 R CNN
-F 2 "keyboard:Diode_SMD_THT" H 21477 8004 50  0001 C CNN
-F 3 "" H 21490 8170 50  0001 C CNN
-	1    21490 8170
-	0    -1   -1   0
-$EndComp
-Wire Wire Line
-	21490 5530 21490 5720
-Wire Wire Line
-	21240 5230 21490 5230
-$Comp
-L keyboard:D DA13
-U 1 1 6175EFCD
-P 21490 5380
-F 0 "DA13" V 21536 5301 50  0000 R CNN
-F 1 "D" V 21445 5301 50  0000 R CNN
-F 2 "keyboard:Diode_SMD_THT" H 21477 5214 50  0001 C CNN
-F 3 "" H 21490 5380 50  0001 C CNN
-	1    21490 5380
-	0    -1   -1   0
-$EndComp
-Connection ~ 20050 9440
-Wire Wire Line
-	20640 8020 20640 8950
-Connection ~ 20640 8020
-Wire Wire Line
-	20640 8950 20640 9880
-Connection ~ 20640 8950
-Wire Wire Line
-	20050 10370 21490 10370
-Wire Wire Line
-	21490 10370 21490 10180
-Connection ~ 20050 10370
-Wire Wire Line
-	21490 9250 21490 9440
-Wire Wire Line
-	20050 9440 21490 9440
-Wire Wire Line
-	20430 9200 20430 9100
-Wire Wire Line
-	20430 9100 20740 9100
-Wire Wire Line
-	20430 10130 20430 10030
-Wire Wire Line
-	20430 10030 20740 10030
-NoConn ~ 2350 1940
+	21140 10130 21200 10130
+Wire Wire Line
+	21200 10130 21200 9550
+Wire Wire Line
+	21200 9550 20550 9550
+Wire Wire Line
+	20550 9550 20550 9100
+Wire Wire Line
+	20550 9100 20740 9100
+Wire Wire Line
+	21140 9200 21210 9200
+Wire Wire Line
+	21210 9200 21210 8600
+Wire Wire Line
+	21210 8600 20550 8600
+Wire Wire Line
+	20550 8600 20550 8170
+Wire Wire Line
+	20550 8170 20740 8170
+Text GLabel 2060 10030 0    50   Input ~ 0
+LEDR5
+Text GLabel 21140 8270 2    50   Input ~ 0
+LEDR5
+NoConn ~ 20740 10030
 $EndSCHEMATC

Commit message: wip routing
Connections:
- net col05: now also U0.31 (GPIO26_ADC0); no longer U0.21 (GPIO16)
- net col06: now also U0.29 (GPIO22); no longer U0.22 (GPIO17)
- net col07: now also U0.27 (GPIO21); no longer U0.24 (GPIO18)
- net col08: now also U0.26 (GPIO20); no longer U0.25 (GPIO19)
- net col09: now also U0.25 (GPIO19); no longer U0.26 (GPIO20)
- net col10: now also U0.24 (GPIO18); no longer U0.27 (GPIO21)
- net col11: now also U0.22 (GPIO17); no longer U0.29 (GPIO22)
- net col12: now also U0.21 (GPIO16); no longer U0.31 (GPIO26_ADC0)
- net at KB12.3 (DIN): now also KB13.1 (DOUT)
- net SW99A renamed col13
Changed lines of the file:
@@
 Text GLabel 950  3240 0    50   Input ~ 0
 col04
-Text GLabel 2350 3240 2    50   Input ~ 0
+Text GLabel 2350 2240 2    50   Input ~ 0
 col05
-Text GLabel 2350 3140 2    50   Input ~ 0
+Text GLabel 2350 2440 2    50   Input ~ 0
 col06
-Text GLabel 2350 2940 2    50   Input ~ 0
+Text GLabel 2350 2640 2    50   Input ~ 0
 col07
-Text GLabel 2350 2840 2    50   Input ~ 0
-col08
 Text GLabel 2350 2740 2    50   Input ~ 0
+col08
+Text GLabel 2350 2840 2    50   Input ~ 0
 col09
-Text GLabel 2350 2640 2    50   Input ~ 0
+Text GLabel 2350 2940 2    50   Input ~ 0
 col10
-Text GLabel 2350 2440 2    50   Input ~ 0
+Text GLabel 2350 3140 2    50   Input ~ 0
 col11
-Text GLabel 2350 2240 2    50   Input ~ 0
+Text GLabel 2350 3240 2    50   Input ~ 0
 col12
 Text GLabel 2350 2140 2    50   Input ~ 0
@@
 Text GLabel 7390 2390 0    50   Input ~ 0
 ENCB
-Text GLabel 7990 2190 2    50   Input ~ 0
-SW99A
-Text GLabel 7990 2390 2    50   Input ~ 0
-SW99B
 $Comp
 L keyboard:D DA0
@@
 	0    -1   -1   0
 $EndComp
-Wire Wire Line
-	9640 10030 9770 10030
 $Comp
 L keyboard:GND #PWR0146
 U 1 1 6140132C
-P 9770 10030
-F 0 "#PWR0146" H 9770 9780 50  0001 C CNN
-F 1 "GND" V 9775 9902 50  0000 R CNN
-F 2 "" H 9770 10030 50  0001 C CNN
-F 3 "" H 9770 10030 50  0001 C CNN
-	1    9770 10030
+P 9790 10030
+F 0 "#PWR0146" H 9790 9780 50  0001 C CNN
+F 1 "GND" V 9795 9902 50  0000 R CNN
+F 2 "" H 9790 10030 50  0001 C CNN
+F 3 "" H 9790 10030 50  0001 C CNN
+	1    9790 10030
 	0    -1   -1   0
 $EndComp
@@
 	-1   0    0    1
 $EndComp
-Text GLabel 20640 5090 2    50   Input ~ 0
-SW99A
-Text GLabel 21240 5230 0    50   Input ~ 0
-SW99B
 $Comp
 L keyboard:GND #PWR0262
@@
 SCL
 Wire Wire Line
-	20640 4770 20640 6160
+	20640 4770 20640 5090
 Wire Wire Line
 	2460 10130 3080 10130
@@
 	0    -1   -1   0
 $EndComp
-Wire Wire Line
-	19700 10030 19830 10030
 $Comp
 L keyboard:D DF12
@@
 NoConn ~ 2350 1940
 Wire Wire Line
-	19710 6410 20430 6410
-Wire Wire Line
-	20430 6410 20430 6310
-Wire Wire Line
-	20430 6310 20740 6310
-Wire Wire Line
 	20640 8020 20640 8950
 Wire Wire Line
@@
 LEDR5
 NoConn ~ 20740 10030
+Wire Wire Line
+	20770 5090 20640 5090
+Connection ~ 20640 5090
+Wire Wire Line
+	20640 5090 20640 6160
+Wire Wire Line
+	19700 6410 20430 6410
+Wire Wire Line
+	20740 6310 20430 6310
+Wire Wire Line
+	20430 6310 20430 6410
+Wire Wire Line
+	19700 10030 19830 10030
+Text Label 20770 5090 0    50   ~ 0
+SW99A
+Text Label 7990 2190 0    50   ~ 0
+SW99A
+Text Label 21240 5230 2    50   ~ 0
+SW99B
+Text Label 7990 2390 0    50   ~ 0
+SW99B
+Wire Wire Line
+	9640 10030 9790 10030
 $EndSCHEMATC

Commit message: rework routing
Connections:
- net LEDR0: now also KB0.3 (DIN); no longer KB13.3 (DIN)
- net LEDR1: now also KB13.1 (DOUT); no longer KB0.1 (DOUT)
- net LEDR2: now also KD0.3 (DIN); no longer KD12.3 (DIN)
- net LEDR3: now also KD12.1 (DOUT); no longer KD0.1 (DOUT)
- net LEDR4: now also KF0.3 (DIN); no longer KF12.3 (DIN)
- net LEDKB1: now reaches KB1.1 (DOUT)
- net LEDKB1: now also KB2.3 (DIN); no longer KB0.3 (DIN)
- net LEDKD1: now reaches KD1.1 (DOUT)
- net LEDKD1: now also KD2.3 (DIN); no longer KD0.3 (DIN)
- net LEDKB0: now reaches KB1.3 (DIN)
- net LEDKB0: now also KB0.1 (DOUT); no longer KB2.1 (DOUT)
- net LEDKD0: now reaches KD1.3 (DIN)
- net LEDKD0: now also KD0.1 (DOUT); no longer KD2.1 (DOUT)
- net LEDKF1: now reaches KF1.1 (DOUT)
- net LEDKF1: now also KF2.3 (DIN); no longer KF0.3 (DIN)
- net LEDKF0: now reaches KF1.3 (DIN)
- net LEDKF0: now also KF0.1 (DOUT); no longer KF2.1 (DOUT)
- net LEDKB3: now reaches KB3.1 (DOUT)
- net LEDKB3: now also KB4.3 (DIN); no longer KB2.3 (DIN)
- net LEDKD3: now reaches KD3.1 (DOUT)
- net LEDKD3: now also KD4.3 (DIN); no longer KD2.3 (DIN)
- net LEDKF3: now reaches KF3.1 (DOUT)
- net LEDKF3: now also KF4.3 (DIN); no longer KF2.3 (DIN)
- net LEDKB2: now reaches KB3.3 (DIN)
- net LEDKB2: now also KB2.1 (DOUT); no longer KB4.1 (DOUT)
- net LEDKD2: now reaches KD3.3 (DIN)
- net LEDKD2: now also KD2.1 (DOUT); no longer KD4.1 (DOUT)
- net LEDKF2: now reaches KF3.3 (DIN)
- net LEDKF2: now also KF2.1 (DOUT); no longer KF4.1 (DOUT)
- net LEDKB5: now reaches KB5.1 (DOUT)
- net LEDKB5: now also KB6.3 (DIN); no longer KB4.3 (DIN)
- net LEDKD5: now reaches KD5.1 (DOUT)
- net LEDKD5: now also KD6.3 (DIN); no longer KD4.3 (DIN)
- net LEDKF5: now reaches KF5.1 (DOUT)
- net LEDKF5: now also KF6.3 (DIN); no longer KF4.3 (DIN)
- net LEDKB4: now reaches KB5.3 (DIN)
- net LEDKB4: now also KB4.1 (DOUT); no longer KB6.1 (DOUT)
- net LEDKD4: now reaches KD5.3 (DIN)
- net LEDKD4: now also KD4.1 (DOUT); no longer KD6.1 (DOUT)
- net LEDKF4: now reaches KF5.3 (DIN)
- net LEDKF4: now also KF4.1 (DOUT); no longer KF6.1 (DOUT)
- net LEDKB7: now reaches KB7.1 (DOUT)
- net LEDKB7: now also KB8.3 (DIN); no longer KB6.3 (DIN)
- net LEDKD7: now reaches KD7.1 (DOUT)
- net LEDKD7: now also KD8.3 (DIN); no longer KD6.3 (DIN)
- net LEDKF7: now reaches KF7.1 (DOUT)
- net LEDKF7: now also KF8.3 (DIN); no longer KF6.3 (DIN)
- net LEDKB6: now reaches KB7.3 (DIN)
- net LEDKB6: now also KB6.1 (DOUT); no longer KB8.1 (DOUT)
- net LEDKD6: now reaches KD7.3 (DIN)
- net LEDKD6: now also KD6.1 (DOUT); no longer KD8.1 (DOUT)
- net LEDKF6: now reaches KF7.3 (DIN)
- net LEDKF6: now also KF6.1 (DOUT); no longer KF8.1 (DOUT)
- net LEDKB9: now reaches KB9.1 (DOUT)
- net LEDKB9: now also KB10.3 (DIN); no longer KB8.3 (DIN)
- net LEDKD9: now reaches KD9.1 (DOUT)
- net LEDKD9: now also KD10.3 (DIN); no longer KD8.3 (DIN)
- net LEDKF9: now reaches KF9.1 (DOUT)
- net LEDKF9: now also KF10.3 (DIN); no longer KF8.3 (DIN)
- net LEDKB10: now reaches KB10.1 (DOUT)
- net LEDKB10: now also KB11.3 (DIN); no longer KB9.3 (DIN)
- net LEDKD10: now reaches KD10.1 (DOUT)
- net LEDKD10: now also KD11.3 (DIN); no longer KD9.3 (DIN)
- net LEDKF10: now reaches KF10.1 (DOUT)
- net LEDKF10: now also KF11.3 (DIN); no longer KF9.3 (DIN)
- net LEDKB11: now reaches KB11.1 (DOUT)
- net LEDKB11: now also KB12.3 (DIN); no longer KB10.3 (DIN)
- net LEDKD11: now reaches KD11.1 (DOUT)
- net LEDKD11: now also KD12.3 (DIN); no longer KD10.3 (DIN)
- net LEDKF11: now reaches KF11.1 (DOUT)
- net LEDKF11: now also KF12.3 (DIN); no longer KF10.3 (DIN)
- net LEDKB12: now reaches KB12.1 (DOUT)
- net LEDKB12: now also KB13.3 (DIN); no longer KB11.3 (DIN)
- net LEDKF12: now reaches KF12.1 (DOUT)
- net LEDKF12: now also KF13.3 (DIN); no longer KF11.3 (DIN)
- net at KD13.1 (DOUT): no longer KE13.3 (DIN)
- net at KE13.1 (DOUT): now also KD13.3 (DIN); no longer KF13.3 (DIN)
- net at KF13.1 (DOUT): now also KE13.3 (DIN)
- removed net LEDR5: KD13.3 (DIN), KF0.1 (DOUT)
- new net LEDKB8: KB8.1 (DOUT), KB9.3 (DIN)
- new net LEDKD8: KD8.1 (DOUT), KD9.3 (DIN)
- new net LEDKF8: KF8.1 (DOUT), KF9.3 (DIN)

Commit message: Kanagawa routing
Parts:
- removed J0: Conn_01x03, keyboard:conn_3pins, symbol keyboard:Conn_01x03
- removed U0: Pico, keyboard:RPi_Pico_TH, symbol RP-Pico:Pico
- added MountBaseMiddleTop1, MountBaseMiddleTop2, MountBaseMiddleTop3, MountBaseMiddleTop4, MountBaseMiddleTop5, MountBaseMiddleTop6, MountBaseMiddleTop7, MountBaseMiddleTop8: MountingHole, keyboard:MountingHole_2.2mm_M2_Pad_Via, symbol keyboard:MountingHole
- added MountMiddle0: MountingHole USB breakout, keyboard:Keebio_USB-C_breakout_shadow, symbol keyboard:MountingHole
- added RSW0: SW_RST, keyboard:SW_RST, symbol keyboard:SW_RST
- added U0: Elite-C, keyboard:Elite-C-29pin-holes, symbol keyboard:Elite-C
- KA0, KA1, KA10, KA11, KA12, KA2, KA3, KA4, KA5, KA6, KA7, KA8, KA9, KB0, KB1, KB10, KB11, KB12, KB2, KB3, KB4, KB5, KB6, KB7, KB8, KB9, KC1, KC10, KC11, KC12, KC2, KC3, KC4, KC5, KC6, KC7, KC8, KC9, KD1, KD10, KD11, KD2, KD3, KD4, KD5, KD6, KD7, KD8, KD9, KE1, KE10, KE12, KE2, KE3, KE4, KE5, KE6, KE7, KE8, KE9, KF1, KF10, KF11, KF12, KF3, KF6, KF8: footprint keyboard:SW_Cherry_MX_1.00u_SK6812MINI -> keyboard:SW_Cherry_MX_1.00u_Hotswap; symbol keyboard:KEY_SW_RGB -> keyboard:KEY_SW
- KB13, KD12, KF4, KF5: footprint keyboard:SW_Cherry_MX_2.00u_SK6812MINI -> keyboard:SW_Cherry_MX_2.00u_Hotswap; symbol keyboard:KEY_SW_RGB -> keyboard:KEY_SW
- KC0, KC13: footprint keyboard:SW_Cherry_MX_1.50u_SK6812MINI -> keyboard:SW_Cherry_MX_1.50u_Hotswap; symbol keyboard:KEY_SW_RGB -> keyboard:KEY_SW
- KD0: footprint keyboard:SW_Cherry_MX_1.75u_SK6812MINI -> keyboard:SW_Cherry_MX_1.75u_Hotswap; symbol keyboard:KEY_SW_RGB -> keyboard:KEY_SW
- KD13, KE13, KF0, KF13, KF2, KF7, KF9: footprint keyboard:SW_Cherry_MX_1.25u_SK6812MINI -> keyboard:SW_Cherry_MX_1.25u_Hotswap; symbol keyboard:KEY_SW_RGB -> keyboard:KEY_SW
- KE0, KE11: footprint keyboard:SW_Cherry_MX_2.25u_SK6812MINI -> keyboard:SW_Cherry_MX_2.25u_Hotswap; symbol keyboard:KEY_SW_RGB -> keyboard:KEY_SW
Connections:
- net labels added: RESET
- net labels removed: LED, LEDKB0, LEDKB1, LEDKB10, LEDKB11, LEDKB12, LEDKB2, LEDKB3, LEDKB4, LEDKB5, LEDKB6, LEDKB7, LEDKB8, LEDKB9, LEDKD0, LEDKD1, LEDKD10, LEDKD11, LEDKD2, LEDKD3, LEDKD4, LEDKD5, LEDKD6, LEDKD7, LEDKD8, LEDKD9, LEDKF0, LEDKF1, LEDKF10, LEDKF11, LEDKF12, LEDKF2, LEDKF3, LEDKF4, LEDKF5, LEDKF6, LEDKF7, LEDKF8, LEDKF9, LEDR0, LEDR1, LEDR2, LEDR3, LEDR4
- wire segments 546 -> 344
- no-connect marks 9 -> 0
Other:
- moved on the sheet: J1, R1, R2, SW99
