File: Kanagawa/Kanagawa/generated_pcbs/middle.kicad_pcb (KiCad board)
At the start: 2 copper layers, 332 x 143 mm, 183 parts, among them J1 Conn_01x04, SW99 Rotary_Encoder_Switch, U0 Elite-C

Commit message: update pcb
Parts:
- moved MountBaseMiddleTop3 201.9 mm to (382.9, 83.2)
- moved MountBaseMiddleTop8 197.6 mm to (185.7, 217.2)
- moved MountBaseMiddleTop4 196.9 mm to (382.9, 205.2)
- moved MountBaseMiddleTop7 174.0 mm to (210.9, 109.2)
- moved MountBaseMiddleTop6 131.0 mm to (153.0, 146.0)
- moved MountBaseMiddleTop5 62.8 mm to (267.0, 146.0)
