File: Kanagawa/Kanagawa_RGB/Kanagawa.sch (KiCad schematic (older format))
At the start: 173 parts, among them J0 Conn_01x03, J1 Conn_01x04, SW99 Rotary_Encoder_Switch, U0 Pico

Commit message: Kanagawa routing
Parts:
- KA0, KA1, KA10, KA11, KA12, KA2, KA3, KA4, KA5, KA6, KA7, KA8, KA9, KB0, KB1, KB10, KB11, KB12, KB2, KB3, KB4, KB5, KB6, KB7, KB8, KB9, KC1, KC10, KC11, KC12, KC2, KC3, KC4, KC5, KC6, KC7, KC8, KC9, KD1, KD10, KD11, KD2, KD3, KD4, KD5, KD6, KD7, KD8, KD9, KE1, KE10, KE12, KE2, KE3, KE4, KE5, KE6, KE7, KE8, KE9, KF1, KF10, KF11, KF12, KF3, KF6, KF8: footprint keyboard:SW_Cherry_MX_1.00u_SK6812MINI -> keyboard:SW_Cherry_MX_1.00u_SK6812MINI_Hotswap
- KB13, KD12, KF4, KF5: footprint keyboard:SW_Cherry_MX_2.00u_SK6812MINI -> keyboard:SW_Cherry_MX_2.00u_SK6812MINI_Hotswap
- KC0, KC13: footprint keyboard:SW_Cherry_MX_1.50u_SK6812MINI -> keyboard:SW_Cherry_MX_1.50u_SK6812MINI_Hotswap
- KD0: footprint keyboard:SW_Cherry_MX_1.75u_SK6812MINI -> keyboard:SW_Cherry_MX_1.75u_SK6812MINI_Hotswap
- KD13, KE13, KF0, KF13, KF2, KF7, KF9: footprint keyboard:SW_Cherry_MX_1.25u_SK6812MINI -> keyboard:SW_Cherry_MX_1.25u_SK6812MINI_Hotswap
- KE0, KE11: footprint keyboard:SW_Cherry_MX_2.25u_SK6812MINI -> keyboard:SW_Cherry_MX_2.25u_SK6812MINI_Hotswap

Commit message: edit kanagawa
Parts:
- removed DA12, DA13, DB12, DB13, DC12, DC13, DD12, DD13, DE12, DE13, DF12, DF13: D, keyboard:Diode_SMD_THT, symbol keyboard:D
- removed J0: Conn_01x03, keyboard:conn_3pins, symbol keyboard:Conn_01x03
- removed KA12, KB12, KC12, KE12, KF12: KEY_SW, keyboard:SW_Cherry_MX_1.00u_SK6812MINI_Hotswap, symbol keyboard:KEY_SW_RGB
- removed KB13, KD12: KEY_SW, keyboard:SW_Cherry_MX_2.00u_SK6812MINI_Hotswap, symbol keyboard:KEY_SW_RGB
- removed KC13: KEY_SW, keyboard:SW_Cherry_MX_1.50u_SK6812MINI_Hotswap, symbol keyboard:KEY_SW_RGB
- removed KD13, KE13, KF13: KEY_SW, keyboard:SW_Cherry_MX_1.25u_SK6812MINI_Hotswap, symbol keyboard:KEY_SW_RGB
- removed U0: Pico, keyboard:RPi_Pico_TH, symbol RP-Pico:Pico
- added DG0, DG1, DG10, DG11, DG2, DG3, DG4, DG5, DG6, DG7, DG8, DG9: D, keyboard:Diode_SMD_THT, symbol keyboard:D
- added KG0, KG2, KG7, KG9: KEY_SW, keyboard:SW_Cherry_MX_1.25u_SK6812MINI_Hotswap, symbol keyboard:KEY_SW_RGB
- added KG1, KG10, KG3, KG6, KG8: KEY_SW, keyboard:SW_Cherry_MX_1.00u_SK6812MINI_Hotswap, symbol keyboard:KEY_SW_RGB
- added KG4, KG5: KEY_SW, keyboard:SW_Cherry_MX_2.00u_SK6812MINI_Hotswap, symbol keyboard:KEY_SW_RGB
- added MountBaseMiddleTop1, MountBaseMiddleTop2, MountBaseMiddleTop3, MountBaseMiddleTop4, MountBaseMiddleTop5, MountBaseMiddleTop6, MountBaseMiddleTop7, MountBaseMiddleTop8: MountingHole, keyboard:MountingHole_2.2mm_M2_Pad_Via, symbol keyboard:MountingHole
- added MountMiddle0: MountingHole USB breakout, keyboard:Keebio_USB-C_breakout_shadow, symbol keyboard:MountingHole
- added RSW0: SW_RST, keyboard:SW_RST, symbol keyboard:SW_RST
- added U0: Elite-C, keyboard:Elite-C-29pin-holes, symbol keyboard:Elite-C
Connections:
- net LEDKB11 is gone; now on net RGB-G9: KB11.1 (DOUT)
- net LEDKD11 is gone; now on net RGB-G9: KD11.1 (DOUT)
- net LEDKF11 is gone; now on net RGB-G9: KF11.1 (DOUT)
- net col13 is gone; now on net col11: SW99.S1
- net ENCA: now also U0.24 (B0)
- net ENCB: now also U0.20 (A3/PF4)
- net GND: now also KG0.4 (VDD), KG1.4 (VDD), KG10.4 (VDD), KG2.4 (VDD), KG3.4 (VDD), KG4.4 (VDD), KG5.4 (VDD), KG6.4 (VDD), KG7.4 (VDD), KG8.4 (VDD), KG9.4 (VDD), RSW0.2, U0.23 (GND), U0.3 (GND), U0.4 (GND)
- net SCL: now also U0.6 (3/PD0)
- net SDA: now also U0.5 (2/PD1)
- net SW99B: now also DG11.2 (A)
- net VCC: now also KG0.2 (VSS), KG1.2 (VSS), KG10.2 (VSS), KG2.2 (VSS), KG3.2 (VSS), KG4.2 (VSS), KG5.2 (VSS), KG6.2 (VSS), KG7.2 (VSS), KG8.2 (VSS), KG9.2 (VSS), U0.21 (VCC)
- net col00: now also KG0.5, U0.29 (F0)
- net col01: now also KG1.5, U0.28 (F1)
- net col02: now also KG2.5, U0.27 (C7)
- net col03: now also KG3.5, U0.26 (D5)
- net col04: now also KG4.5, U0.25 (B7)
- net col05: now also KG5.5, U0.12 (9/PB5)
- net col06: now also KG6.5, U0.11 (8/PB4)
- net col07: now also KG7.5, U0.10 (7/PE6)
- net col08: now also KG8.5, U0.9 (6/PD7)
- net col09: now also KG9.5, U0.8 (5/PC6)
- net col10: now also KG10.5, U0.7 (4/PD4)
- net col11: now also U0.2 (RX1/PD2)
- net row00: now also U0.13 (10/PB6)
- net row01: now also U0.14 (16/PB2)
- net row02: now also U0.15 (14/PB3)
- net row03: now also U0.16 (15/PB1)
- net row04: now also U0.17 (A0/PF7)
- net row05: now also DG0.1 (K), DG1.1 (K), DG10.1 (K), DG11.1 (K), DG2.1 (K), DG3.1 (K), DG4.1 (K), DG5.1 (K), DG6.1 (K), DG7.1 (K), DG8.1 (K), DG9.1 (K), U0.18 (A1/PF6)
- net RGB-G10: now reaches KA0.3 (DIN)
- net RGB-G10: now also KA1.3 (DIN), KA10.3 (DIN), KA11.3 (DIN), KA2.3 (DIN), KA3.3 (DIN), KA4.3 (DIN), KA5.3 (DIN), KA6.3 (DIN), KA7.3 (DIN), KA8.3 (DIN), KA9.3 (DIN), KB0.3 (DIN), KB1.3 (DIN), KB10.3 (DIN), KB11.3 (DIN), KB2.3 (DIN), KB3.3 (DIN), KB4.3 (DIN), KB5.3 (DIN), KB6.3 (DIN), KB7.3 (DIN), KB8.3 (DIN), KB9.3 (DIN), KC0.3 (DIN), KC1.3 (DIN), KC10.3 (DIN), KC11.3 (DIN), KC2.3 (DIN), KC3.3 (DIN), KC4.3 (DIN), KC5.3 (DIN), KC6.3 (DIN), KC7.3 (DIN), KC8.3 (DIN), KC9.3 (DIN), KD0.3 (DIN), KD1.3 (DIN), KD10.3 (DIN), KD11.3 (DIN), KD2.3 (DIN), KD3.3 (DIN), KD4.3 (DIN), KD5.3 (DIN), KD6.3 (DIN), KD7.3 (DIN), KD8.3 (DIN), KD9.3 (DIN), KE0.3 (DIN), KE1.3 (DIN), KE10.3 (DIN), KE11.3 (DIN), KE2.3 (DIN), KE3.3 (DIN), KE4.3 (DIN), KE5.3 (DIN), KE6.3 (DIN), KE7.3 (DIN), KE8.3 (DIN), KE9.3 (DIN), KF0.3 (DIN), KF1.3 (DIN), KF10.3 (DIN), KF11.3 (DIN), KF2.3 (DIN), KF3.3 (DIN), KF4.3 (DIN), KF5.3 (DIN), KF6.3 (DIN), KF7.3 (DIN), KF8.3 (DIN), KF9.3 (DIN), KG0.3 (DIN), KG1.3 (DIN), KG2.3 (DIN), KG3.3 (DIN), KG4.3 (DIN), KG5.3 (DIN), KG6.3 (DIN), KG7.3 (DIN), KG8.3 (DIN), KG9.3 (DIN); no longer KA1.1 (DOUT)
- net RGB-G9: now reaches KC1.1 (DOUT)
- net RGB-G9: now also KA0.1 (DOUT), KA1.1 (DOUT), KA10.1 (DOUT), KA11.1 (DOUT), KA2.1 (DOUT), KA3.1 (DOUT), KA4.1 (DOUT), KA5.1 (DOUT), KA6.1 (DOUT), KA7.1 (DOUT), KA8.1 (DOUT), KA9.1 (DOUT), KB0.1 (DOUT), KB1.1 (DOUT), KB10.1 (DOUT), KB2.1 (DOUT), KB3.1 (DOUT), KB4.1 (DOUT), KB5.1 (DOUT), KB6.1 (DOUT), KB7.1 (DOUT), KB8.1 (DOUT), KB9.1 (DOUT), KC0.1 (DOUT), KC10.1 (DOUT), KC11.1 (DOUT), KC2.1 (DOUT), KC3.1 (DOUT), KC4.1 (DOUT), KC5.1 (DOUT), KC6.1 (DOUT), KC7.1 (DOUT), KC8.1 (DOUT), KC9.1 (DOUT), KD0.1 (DOUT), KD1.1 (DOUT), KD10.1 (DOUT), KD2.1 (DOUT), KD3.1 (DOUT), KD4.1 (DOUT), KD5.1 (DOUT), KD6.1 (DOUT), KD7.1 (DOUT), KD8.1 (DOUT), KD9.1 (DOUT), KE0.1 (DOUT), KE1.1 (DOUT), KE10.1 (DOUT), KE11.1 (DOUT), KE2.1 (DOUT), KE3.1 (DOUT), KE4.1 (DOUT), KE5.1 (DOUT), KE6.1 (DOUT), KE7.1 (DOUT), KE8.1 (DOUT), KE9.1 (DOUT), KF0.1 (DOUT), KF1.1 (DOUT), KF10.1 (DOUT), KF2.1 (DOUT), KF3.1 (DOUT), KF4.1 (DOUT), KF5.1 (DOUT), KF6.1 (DOUT), KF7.1 (DOUT), KF8.1 (DOUT), KF9.1 (DOUT), KG0.1 (DOUT), KG1.1 (DOUT), KG2.1 (DOUT), KG3.1 (DOUT), KG4.1 (DOUT), KG5.1 (DOUT), KG6.1 (DOUT), KG7.1 (DOUT), KG8.1 (DOUT), KG9.1 (DOUT); no longer KC0.3 (DIN)
- removed net LEDKB0: KB0.1 (DOUT), KB1.3 (DIN)
- removed net LEDKB1: KB1.1 (DOUT), KB2.3 (DIN)
- removed net LEDKB10: KB10.1 (DOUT), KB11.3 (DIN)
- removed net LEDKB2: KB2.1 (DOUT), KB3.3 (DIN)
- removed net LEDKB3: KB3.1 (DOUT), KB4.3 (DIN)
- removed net LEDKB4: KB4.1 (DOUT), KB5.3 (DIN)
- removed net LEDKB5: KB5.1 (DOUT), KB6.3 (DIN)
- removed net LEDKB6: KB6.1 (DOUT), KB7.3 (DIN)
- removed net LEDKB7: KB7.1 (DOUT), KB8.3 (DIN)
- removed net LEDKB8: KB8.1 (DOUT), KB9.3 (DIN)
- removed net LEDKB9: KB10.3 (DIN), KB9.1 (DOUT)
- removed net LEDKD0: KD0.1 (DOUT), KD1.3 (DIN)
- removed net LEDKD1: KD1.1 (DOUT), KD2.3 (DIN)
- removed net LEDKD10: KD10.1 (DOUT), KD11.3 (DIN)
- removed net LEDKD2: KD2.1 (DOUT), KD3.3 (DIN)
- removed net LEDKD3: KD3.1 (DOUT), KD4.3 (DIN)
- removed net LEDKD4: KD4.1 (DOUT), KD5.3 (DIN)
- removed net LEDKD5: KD5.1 (DOUT), KD6.3 (DIN)
- removed net LEDKD6: KD6.1 (DOUT), KD7.3 (DIN)
- removed net LEDKD7: KD7.1 (DOUT), KD8.3 (DIN)
- removed net LEDKD8: KD8.1 (DOUT), KD9.3 (DIN)
- removed net LEDKD9: KD10.3 (DIN), KD9.1 (DOUT)
- removed net LEDKF0: KF0.1 (DOUT), KF1.3 (DIN)
- removed net LEDKF1: KF1.1 (DOUT), KF2.3 (DIN)
- removed net LEDKF10: KF10.1 (DOUT), KF11.3 (DIN)
- removed net LEDKF2: KF2.1 (DOUT), KF3.3 (DIN)
- removed net LEDKF3: KF3.1 (DOUT), KF4.3 (DIN)
- removed net LEDKF4: KF4.1 (DOUT), KF5.3 (DIN)
- removed net LEDKF5: KF5.1 (DOUT), KF6.3 (DIN)
- removed net LEDKF6: KF6.1 (DOUT), KF7.3 (DIN)
- removed net LEDKF7: KF7.1 (DOUT), KF8.3 (DIN)
- removed net LEDKF8: KF8.1 (DOUT), KF9.3 (DIN)
- removed net LEDKF9: KF10.3 (DIN), KF9.1 (DOUT)
- removed net LEDR0: KA0.1 (DOUT), KB0.3 (DIN)
- removed net LEDR2: KC0.1 (DOUT), KD0.3 (DIN)
- removed net LEDR4: KE0.1 (DOUT), KF0.3 (DIN)
- new net: DG0.2 (A), KG0.6
- new net: DG1.2 (A), KG1.6
- new net: DG2.2 (A), KG2.6
- new net: DG3.2 (A), KG3.6
- new net: DG4.2 (A), KG4.6
- new net: DG5.2 (A), KG5.6
- new net: DG6.2 (A), KG6.6
- new net: DG7.2 (A), KG7.6
- new net: DG8.2 (A), KG8.6
- new net: DG9.2 (A), KG9.6
- new net: DG10.2 (A), KG10.6
- new net RESET: RSW0.1, U0.22 (RST)
- new net RGB: KG10.3 (DIN), U0.1 (TX0/PD3)
- new net row06: U0.19 (A2/PF5)
- no-connect marks 9 -> 0
Other:
- moved on the sheet: J1, R1, R2, SW99
