File: Kanagawa/rev2/Kanagawa.kicad_pcb (KiCad board)
At the start: 2 copper layers, 332 x 143 mm, 186 parts, among them J1 Conn_01x04, SW99 Rotary_Encoder_Switch, U0 Elite-C

Commit message: edit rev2
Parts:
- moved MountBaseMiddleTop3 60.0 mm to (150.0, 83.2)
- moved MountBaseMiddleTop5 30.0 mm to (300.0, 83.2)
