File: Kanagawa/rev1/Kanagawa.kicad_pcb (KiCad board)
At the start: 2 copper layers, 330 x 144 mm, 184 parts, among them J1 Conn_01x04, SW99 Rotary_Encoder_Switch, U0 Elite-C

Commit message: change R D footprint
Parts:
- DA0, DA1, DA10, DA11, DA12, DA13, DA2, DA3, DA4, DA5, DA6, DA7, DA8, DA9, DB0, DB1, DB10, DB11, DB12, DB13, DB2, DB3, DB4, DB5, DB6, DB7, DB8, DB9, DC0, DC1, DC10, DC11, DC12, DC13, DC2, DC3, DC4, DC5, DC6, DC7, DC8, DC9, DD0, DD1, DD10, DD11, DD12, DD13, DD2, DD3, DD4, DD5, DD6, DD7, DD8, DD9, DE0, DE1, DE10, DE11, DE12, DE13, DE2, DE3, DE4, DE5, DE6, DE7, DE8, DE9, DF0, DF1, DF10, DF11, DF12, DF13, DF2, DF3, DF4, DF5, DF6, DF7, DF8, DF9: footprint keyboard:Diode_SMD_THT -> keyboard:Diode_THT
- R1, R2: footprint keyboard:Resistors_SMD_THT -> keyboard:Resistors_THT
- moved DA13 41.5 mm to (366.6, 103.2), turned to 0 degrees
- moved SW99 41.1 mm to (372.6, 113.5), turned to 90 degrees
- moved J1 21.1 mm to (333.6, 79.5)
- moved R1 10.1 mm to (369.8, 91.3), turned to 90 degrees
- moved R2 9.44 mm to (364.6, 91.5), turned to 90 degrees
- moved MountBaseMiddleTop1 1.00 mm to (61.0, 81.0)
- moved MountBaseMiddleTop2 1.00 mm to (61.0, 207.0)
- moved MountBaseMiddleTop5 1.00 mm to (380.0, 81.0)
- moved MountBaseMiddleTop6 1.00 mm to (379.0, 207.0)
Routing:
- net row05: track 431.7 -> 338.8 mm
- net row04: track 384.1 -> 335.8 mm
- net row01: track 366.7 -> 318.3 mm
- net row02: track 353.3 -> 305.0 mm
- net row03: track 367.3 -> 322.4 mm
- net ENCB: track 0.00 -> 20.5 mm
- net row00: track 380.0 -> 361.0 mm
- net col13: track 161.8 -> 146.9 mm
- net ENCA: track 0.00 -> 11.8 mm
- net Net-(DF13-Pad2): track 6.35 -> 2.75 mm
- net Net-(DF4-Pad2): track 15.5 -> 12.1 mm
- net Net-(DF3-Pad2): track 6.45 -> 2.99 mm
- net Net-(DF9-Pad2): track 6.45 -> 2.99 mm
- net Net-(DF8-Pad2): track 6.45 -> 2.99 mm
- net Net-(DF7-Pad2): track 6.45 -> 2.99 mm
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Other:
- board size 330 x 144 mm -> 328 x 144 mm

Commit message: rev1 routing done
Parts:
- moved R1 6.75 mm to (366.3, 97.1)
- moved R2 5.75 mm to (363.6, 97.1)
Routing:
- net VCC: track 0.09 -> 66.4 mm, vias 0 -> 1
- net SDA: track 12.9 -> 63.8 mm, vias 1 -> 2
- net SCL: track 18.0 -> 64.4 mm, vias 1 -> 2
- net row05: track 338.8 -> 384.9 mm
- net row04: track 335.8 -> 339.3 mm
- net col13: track 146.9 -> 145.1 mm

Commit message: edit pcb
Routing:
- net ENCA: vias 0 -> 1
- net VCC: vias 1 -> 0
Changed lines of the file:
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@@
     (thickness 1.6)
     (drawings 15)
-    (tracks 600)
+    (tracks 603)
     (zones 0)
     (modules 184)
@@
   (gr_line (start 384.89 207.232) (end 384.89 81.232) (layer Edge.Cuts) (width 0.05))
   (gr_line (start 56.89 81.232) (end 56.89 207.232) (layer Edge.Cuts) (width 0.05))
-  (segment (start 225.590355 204.851645) (end 244.1 199.892) (width 0.254) (layer F.Cu) (net 75))
   (segment (start 75.25 99.7) (end 103.85 99.7) (width 0.254) (layer F.Cu) (net 1) (status 30))
   (segment (start 103.85 99.7) (end 122.9 99.7) (width 0.254) (layer F.Cu) (net 1) (status 30))
@@
   (segment (start 343.25 175.27) (end 346.24 175.27) (width 0.254) (layer B.Cu) (net 73) (status 30))
   (segment (start 74.37 189.59) (end 77.36 189.59) (width 0.254) (layer B.Cu) (net 74) (status 30))
+  (segment (start 225.590355 204.851645) (end 244.1 199.892) (width 0.254) (layer F.Cu) (net 75))
   (segment (start 327.191 204.45) (end 365.29 204.45) (width 0.254) (layer F.Cu) (net 75) (status 30))
   (segment (start 179.93 213.97) (end 179.976488 213.923512) (width 0.254) (layer F.Cu) (net 75) (status 30))
@@
   (segment (start 362.29 194.25) (end 365.28 194.25) (width 0.254) (layer B.Cu) (net 87) (status 30))
   (segment (start 359.45 125.93) (end 359.358 125.93) (width 0.254) (layer F.Cu) (net 88) (status 30))
-  (segment (start 361.8 123.58) (end 361.8 117.542) (width 0.254) (layer B.Cu) (net 88))
-  (via (at 361.8 117.542) (size 0.8) (drill 0.4) (layers F.Cu B.Cu) (net 88))
-  (segment (start 359.45 125.93) (end 361.8 123.58) (width 0.254) (layer B.Cu) (net 88))
-  (segment (start 361.8 117.542) (end 361.8 104.352) (width 0.254) (layer F.Cu) (net 88))
-  (segment (start 361.8 104.352) (end 368.15 98.002) (width 0.254) (layer F.Cu) (net 88))
-  (segment (start 368.15 98.002) (end 368.15 93.092) (width 0.254) (layer F.Cu) (net 88))
-  (segment (start 368.15 93.092) (end 366.28 91.222) (width 0.254) (layer F.Cu) (net 88))
-  (segment (start 366.28 91.222) (end 366.28 86.952) (width 0.254) (layer F.Cu) (net 88))
   (segment (start 348.61 83.732) (end 345.83 80.952) (width 0.254) (layer F.Cu) (net 88))
   (segment (start 351.83 86.952) (end 348.61 83.732) (width 0.254) (layer F.Cu) (net 88))
   (segment (start 366.28 86.952) (end 351.83 86.952) (width 0.254) (layer F.Cu) (net 88))
+  (segment (start 368.15 93.092) (end 366.28 91.222) (width 0.254) (layer F.Cu) (net 88))
+  (segment (start 368.15 98.002) (end 368.15 93.092) (width 0.254) (layer F.Cu) (net 88))
+  (segment (start 361.8 104.352) (end 368.15 98.002) (width 0.254) (layer F.Cu) (net 88))
+  (segment (start 366.28 91.222) (end 366.28 86.952) (width 0.254) (layer F.Cu) (net 88))
+  (segment (start 361.8 123.58) (end 361.8 104.352) (width 0.254) (layer F.Cu) (net 88))
+  (segment (start 359.45 125.93) (end 361.8 123.58) (width 0.254) (layer F.Cu) (net 88))
   (segment (start 344.21 128.47) (end 345.9 126.78) (width 0.254) (layer F.Cu) (net 90) (status 10))
   (via (at 359.28 104.112) (size 0.8) (drill 0.4) (layers F.Cu B.Cu) (net 90))
@@
   (via (at 345.9 116.122) (size 0.8) (drill 0.4) (layers F.Cu B.Cu) (net 90))
   (segment (start 345.9 126.78) (end 345.9 116.122) (width 0.254) (layer F.Cu) (net 90))
-  (segment (start 345.9 116.122) (end 347.27 116.122) (width 0.254) (layer B.Cu) (net 90))
-  (segment (start 347.27 116.122) (end 359.28 104.112) (width 0.254) (layer B.Cu) (net 90))
   (segment (start 350.91 80.952) (end 366.28 96.322) (width 0.254) (layer B.Cu) (net 90))
   (segment (start 366.28 96.322) (end 366.28 97.112) (width 0.254) (layer B.Cu) (net 90))
+  (segment (start 345.9 116.122) (end 357.705 104.317) (width 0.254) (layer B.Cu) (net 90))
+  (segment (start 357.91 104.112) (end 357.705 104.317) (width 0.254) (layer B.Cu) (net 90))
+  (segment (start 359.28 104.112) (end 357.91 104.112) (width 0.254) (layer B.Cu) (net 90))
   (segment (start 346.68 128.54) (end 346.634 128.586) (width 0.254) (layer F.Cu) (net 91))
   (segment (start 346.68 114.292) (end 346.68 128.54) (width 0.254) (layer F.Cu) (net 91))
@@
   (segment (start 370.462 128.47) (end 375.15 123.782) (width 0.254) (layer F.Cu) (net 92))
   (segment (start 375.15 123.782) (end 375.15 120.962) (width 0.254) (layer F.Cu) (net 92) (status 20))
-  (segment (start 359.45 118.31) (end 367.498 118.31) (width 0.254) (layer F.Cu) (net 93) (status 10))
-  (segment (start 367.498 118.31) (end 370.15 120.962) (width 0.254) (layer F.Cu) (net 93) (status 20))
+  (via (at 364.8 118.312) (size 0.8) (drill 0.4) (layers F.Cu B.Cu) (net 93))
+  (segment (start 364.798 118.31) (end 364.8 118.312) (width 0.254) (layer B.Cu) (net 93))
+  (segment (start 359.45 118.31) (end 364.798 118.31) (width 0.254) (layer B.Cu) (net 93))
+  (segment (start 364.8 118.312) (end 367.5 118.312) (width 0.254) (layer F.Cu) (net 93))
+  (segment (start 367.5 118.312) (end 367.51 118.312) (width 0.254) (layer F.Cu) (net 93))
+  (segment (start 367.51 118.312) (end 370.17 120.972) (width 0.254) (layer F.Cu) (net 93))
   (segment (start 59.55 103.5) (end 59.55 103.07) (width 0.254) (layer B.Cu) (net 94))
   (segment (start 59.55 115.87) (end 59.55 103.5) (width 0.254) (layer B.Cu) (net 94) (status 10))

Commit message: edit pcb
Parts:
- KD13, KE13, KF13: footprint keyboard:SW_Cherry_MX_1.25u_Hotswap -> keyboard:SW_Cherry_MX_1.00u_Hotswap
- moved LogoBase1 8.00 mm to (214.9, 148.2)
- moved DE13 3.50 mm to (380.3, 164.9)
- moved DD13 3.48 mm to (380.3, 145.8)
- moved DF13 3.27 mm to (380.3, 184.0)
- moved MountBaseMiddleTop5 3.00 mm to (377.0, 81.0)
- moved MountBaseMiddleTop6 3.00 mm to (376.0, 207.0)
- moved LogoMiddle 2.83 mm to (374.9, 197.2)
- moved DA13 2.00 mm to (364.6, 103.2)
- moved J1 2.00 mm to (331.6, 79.5)
- moved R1 2.00 mm to (364.3, 97.1)
- moved R2 2.00 mm to (361.6, 97.1)
- moved RSW0 2.00 mm to (324.1, 78.2)
- moved SW99 2.00 mm to (370.6, 113.5)
- moved KD13 0.83 mm to (371.8, 137.5), turned to 270 degrees
- moved KE13 0.83 mm to (371.8, 156.6), turned to 270 degrees
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Routing:
- net ENCB: track 20.5 -> 9.45 mm
- net col13: track 145.1 -> 155.0 mm
- net Net-(DF13-Pad2): track 2.75 -> 9.79 mm
- net Net-(DD13-Pad2): track 2.76 -> 9.79 mm
- net Net-(DE13-Pad2): track 2.78 -> 9.79 mm
- net ENCA: track 11.8 -> 9.82 mm
- net SDA: track 63.8 -> 62.2 mm
- net row05: track 384.9 -> 386.1 mm
- net row00: track 361.0 -> 362.1 mm
- net row04: track 339.3 -> 340.3 mm
- net SCL: track 64.4 -> 63.5 mm
- net VCC: track 66.4 -> 65.6 mm
- net row03: track 322.4 -> 323.2 mm
Other:
- board size 328 x 144 mm -> 325 x 143 mm
