File: Kanagawa/rev1/Kanagawa.kicad_pcb (KiCad board)
At the start: 2 copper layers, 325 x 143 mm, 184 parts, among them J1 Conn_01x04, SW99 Rotary_Encoder_Switch, U0 Elite-C

Commit message: rework rev1 from fusion layout
Parts:
- added MountBaseMiddleTop3: MountingHole, keyboard:MountingHole_2.2mm_M2_Pad_Via, F.Cu at (125.9, 81.2)
- added MountBaseMiddleTop4: MountingHole, keyboard:MountingHole_2.2mm_M2_Pad_Via, F.Cu at (125.9, 207.2)
- LogoBase1: footprint layout-for-export:Great-wave -> keyboard:hokusai
- RSW0: value SW_RST -> SW_Push
- moved KD12 23.5 mm to (299.8, 147.3)
- moved KE0 23.4 mm to (56.9, 166.4)
- moved KF4 21.6 mm to (147.4, 190.8)
- moved KB13 21.3 mm to (304.5, 109.2)
- moved KF5 21.1 mm to (186.5, 200.6)
- moved KE11 19.2 mm to (290.3, 166.4)
- moved KD0 19.1 mm to (56.9, 147.3)
- moved KC13 17.2 mm to (314.1, 128.3)
- moved KC0 17.1 mm to (56.9, 128.3)
- moved KF2 15.2 mm to (99.8, 185.4)
- moved KF0 15.2 mm to (56.9, 185.4)
- moved KD13 13.7 mm to (381.9, 128.3)
- moved KE13 13.6 mm to (381.9, 147.3)
- moved KF13 13.6 mm to (381.9, 166.4)
- moved KA0 13.6 mm to (56.9, 85.1)
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- renumbered MountBaseMiddleTop3 to MountBaseMiddleTop5, MountBaseMiddleTop4 to MountBaseMiddleTop6, MountBaseMiddleTop5 to MountBaseMiddleTop7, MountBaseMiddleTop6 to MountBaseMiddleTop8
Routing:
- net ENCB: track 9.45 -> 19.6 mm
- net Net-(DD12-Pad2): track 14.4 -> 12.4 mm
- net row03: track 323.2 -> 321.7 mm
- net col13: track 155.0 -> 156.2 mm
- net col10: track 276.4 -> 277.4 mm
- net col04: track 370.9 -> 371.8 mm
- net col03: track 602.9 -> 603.8 mm
- net row05: track 386.1 -> 386.9 mm
- net RESET: track 67.6 -> 68.5 mm
- net col07: track 324.4 -> 325.2 mm
- net col02: track 411.3 -> 411.9 mm
- net col12: track 208.1 -> 207.6 mm
- net col09: track 283.7 -> 284.2 mm
- net Net-(DE11-Pad2): track 3.28 -> 2.78 mm

Commit message: review board
Routing:
- net col03: track 603.8 -> 390.8 mm
- net col06: track 346.4 -> 356.4 mm
- net col07: track 325.2 -> 334.5 mm
- net col08: track 303.8 -> 312.3 mm
- net col05: track 366.8 -> 373.4 mm
- net col09: track 284.2 -> 290.4 mm
- net col02: track 411.9 -> 415.6 mm
- net col01: track 441.3 -> 437.8 mm
- net col12: track 207.6 -> 209.7 mm
- net col10: track 277.4 -> 275.3 mm
- net col11: track 249.7 -> 251.4 mm
- net col04: track 371.8 -> 372.9 mm
- net col00: track 447.7 -> 446.8 mm
- net row05: vias 1 -> 2

Commit message: review board edges
Other:
- board size 325 x 143 mm -> 325 x 144.9 mm

Commit message: review PCB
Parts:
- moved RSW0 5.00 mm to (319.1, 78.2)
Routing:
- net RESET: track 68.5 -> 70.6 mm
Other:
- board size 325 x 144.9 mm -> 325 x 143 mm
Changed lines of the file:
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@@
   (general
     (thickness 1.6)
-    (drawings 737)
+    (drawings 738)
     (tracks 699)
     (zones 0)
@@
   )
   (module keyboard:SW_RST (layer F.Cu)
-    (at 324.05 78.182)
+    (at 319.05 78.182)
     (fp_text reference RSW0 (at 0 -1.27) (layer Dwgs.User) hide
       (effects (font (size 1 1) (thickness 0.15)))
@@
       (xy 2.996029 1.227264) (xy 3.044593 1.230575) (xy 3.095505 1.230604) (xy 3.146737 1.227413)) (layer B.Mask) (width 0.01))
   )
-  (gr_line (start 315.048447 75.232) (end 323.048447 75.232) (layer Edge.Cuts) (width 0.05))
+  (dimension 143 (width 0.15) (layer Dwgs.User)
+    (gr_text "143,000 mm" (at 41.59 147.732 90) (layer Dwgs.User)
+      (effects (font (size 1 1) (thickness 0.15)))
+    )
+    (feature1 (pts (xy 184.89 76.232) (xy 42.303579 76.232)))
+    (feature2 (pts (xy 184.89 219.232) (xy 42.303579 219.232)))
+    (crossbar (pts (xy 42.89 219.232) (xy 42.89 76.232)))
+    (arrow1a (pts (xy 42.89 76.232) (xy 43.476421 77.358504)))
+    (arrow1b (pts (xy 42.89 76.232) (xy 42.303579 77.358504)))
+    (arrow2a (pts (xy 42.89 219.232) (xy 43.476421 218.105496)))
+    (arrow2b (pts (xy 42.89 219.232) (xy 42.303579 218.105496)))
+  )
+  (dimension 136 (width 0.15) (layer Dwgs.User)
+    (gr_text "136,000 mm" (at 47.59 144.232 270) (layer Dwgs.User)
+      (effects (font (size 1 1) (thickness 0.15)))
+    )
+    (feature1 (pts (xy 61.89 212.232) (xy 48.303579 212.232)))
+    (feature2 (pts (xy 61.89 76.232) (xy 48.303579 76.232)))
+    (crossbar (pts (xy 48.89 76.232) (xy 48.89 212.232)))
+    (arrow1a (pts (xy 48.89 212.232) (xy 48.303579 211.105496)))
+    (arrow1b (pts (xy 48.89 212.232) (xy 49.476421 211.105496)))
+    (arrow2a (pts (xy 48.89 76.232) (xy 48.303579 77.358504)))
+    (arrow2b (pts (xy 48.89 76.232) (xy 49.476421 77.358504)))
+  )
+  (dimension 325.000001 (width 0.15) (layer Dwgs.User)
+    (gr_text "325,000 mm" (at 219.389999 62.932 1.762947022e-07) (layer Dwgs.User)
+      (effects (font (size 1 1) (thickness 0.15)))
+    )
+    (feature1 (pts (xy 56.889999 81.232001) (xy 56.889999 63.64558)))
+    (feature2 (pts (xy 381.89 81.232) (xy 381.89 63.645579)))
+    (crossbar (pts (xy 381.89 64.232) (xy 56.889999 64.232001)))
+    (arrow1a (pts (xy 56.889999 64.232001) (xy 58.016503 63.64558)))
+    (arrow1b (pts (xy 56.889999 64.232001) (xy 58.016503 64.818422)))
+    (arrow2a (pts (xy 381.89 64.232) (xy 380.763496 63.645579)))
+    (arrow2b (pts (xy 381.89 64.232) (xy 380.763496 64.818421)))
+  )
+  (gr_line (start 315.048447 75.232) (end 323.048447 75.232) (layer Dwgs.User) (width 0.05))
   (gr_circle (center 125.89 81.232) (end 126.99 81.232) (layer Edge.Cuts) (width 0.05))
   (gr_circle (center 229.7994 79.8039) (end 231.3994 79.8039) (layer Edge.Cuts) (width 0.05))
   (gr_circle (center 376.89 81.232001) (end 377.99 81.232001) (layer Edge.Cuts) (width 0.05))
   (gr_circle (center 244.89 81.232) (end 245.99 81.232) (layer Edge.Cuts) (width 0.05))
-  (gr_line (start 216.2697 74.3039) (end 225.4697 74.3039) (layer Edge.Cuts) (width 0.05))
   (gr_circle (center 61.89 81.232) (end 62.99 81.232) (layer Edge.Cuts) (width 0.05))
-  (gr_line (start 61.89 76.232) (end 236.7994 76.232001) (layer Edge.Cuts) (width 0.05))
   (gr_circle (center 376.89 207.232149) (end 377.99 207.232149) (layer Edge.Cuts) (width 0.05))
   (gr_circle (center 244.89 207.232) (end 245.99 207.232) (layer Edge.Cuts) (width 0.05))
@@
   (gr_circle (center 211.94 79.8039) (end 213.54 79.8039) (layer Edge.Cuts) (width 0.05))
   (gr_line (start 196.489483 219.232) (end 222.613839 212.232) (layer Edge.Cuts) (width 0.05))
-  (gr_line (start 376.851402 212.232) (end 236.7994 212.232) (layer Edge.Cuts) (width 0.05))
+  (gr_line (start 376.89 212.232) (end 236.7994 212.232) (layer Edge.Cuts) (width 0.05))
   (gr_arc (start 61.89 81.232001) (end 61.89 76.232) (angle -90) (layer Edge.Cuts) (width 0.05))
   (gr_line (start 61.89 212.232) (end 148.053656 212.232) (layer Edge.Cuts) (width 0.05))
@@
   (segment (start 316.589999 119.212001) (end 316.589999 125.791999) (width 0.254) (layer B.Cu) (net 110))
   (segment (start 316.589999 116.183999) (end 316.589999 119.212001) (width 0.254) (layer B.Cu) (net 110))
-  (segment (start 324.98 81.612) (end 321.55 78.182) (width 0.254) (layer F.Cu) (net 111) (status 20))
   (segment (start 329.41399 100.81599) (end 324.98 96.382) (width 0.254) (layer F.Cu) (net 111))
   (segment (start 342.394914 100.81599) (end 329.41399 100.81599) (width 0.254) (layer F.Cu) (net 111))
@@
   (segment (start 359.45 123.39) (end 354.37203 118.31203) (width 0.254) (layer F.Cu) (net 111))
   (segment (start 354.37203 118.31203) (end 354.37203 112.793106) (width 0.254) (layer F.Cu) (net 111))
-  (segment (start 324.98 96.382) (end 324.98 81.612) (width 0.254) (layer F.Cu) (net 111))
+  (segment (start 324.98 96.382) (end 324.98 86.602) (width 0.254) (layer F.Cu) (net 111))
+  (segment (start 324.98 86.602) (end 316.56 78.182) (width 0.254) (layer F.Cu) (net 111))
   (zone (net 89) (net_name GND) (layer B.Cu) (hatch edge 0.508)
     (connect_pads (clearance 0.508))
