File: Kanagawa/rev1/Kanagawa.sch (KiCad schematic (older format))
At the start: 182 parts, among them J1 Conn_01x04, SW99 Rotary_Encoder_Switch, U0 Elite-C

Commit message: clean revisions
Parts:
- removed MountBaseMiddleTop7, MountBaseMiddleTop8: MountingHole, keyboard:MountingHole_2.2mm_M2_Pad_Via, symbol keyboard:MountingHole
- KD12: footprint keyboard:SW_Cherry_MX_2.00u_Hotswap -> keyboard:SW_Cherry_MX_2.25u_Hotswap
- KE11: footprint keyboard:SW_Cherry_MX_2.25u_Hotswap -> keyboard:SW_Cherry_MX_1.75u_Hotswap
- KF7, KF9: footprint keyboard:SW_Cherry_MX_1.25u_Hotswap -> keyboard:SW_Cherry_MX_1.00u_Hotswap
Changed lines of the file:
@@
 F 0 "KF7" H 12330 10135 50  0000 C CNN
 F 1 "KEY_SW" H 12330 10044 50  0000 C CNN
-F 2 "keyboard:SW_Cherry_MX_1.25u_Hotswap" H 12330 9880 50  0001 C CNN
+F 2 "keyboard:SW_Cherry_MX_1.00u_Hotswap" H 12330 9880 50  0001 C CNN
 F 3 "" H 12330 9880 50  0000 C CNN
 	1    12330 9880
@@
 F 0 "KF9" H 15190 10135 50  0000 C CNN
 F 1 "KEY_SW" H 15190 10044 50  0000 C CNN
-F 2 "keyboard:SW_Cherry_MX_1.25u_Hotswap" H 15190 9880 50  0001 C CNN
+F 2 "keyboard:SW_Cherry_MX_1.00u_Hotswap" H 15190 9880 50  0001 C CNN
 F 3 "" H 15190 9880 50  0000 C CNN
 	1    15190 9880
@@
 F 0 "KE11" H 18040 9205 50  0000 C CNN
 F 1 "KEY_SW" H 18040 9114 50  0000 C CNN
-F 2 "keyboard:SW_Cherry_MX_2.25u_Hotswap" H 18040 8950 50  0001 C CNN
+F 2 "keyboard:SW_Cherry_MX_1.75u_Hotswap" H 18040 8950 50  0001 C CNN
 F 3 "" H 18040 8950 50  0000 C CNN
 	1    18040 8950
@@
 F 0 "KD12" H 19500 8275 50  0000 C CNN
 F 1 "KEY_SW" H 19500 8184 50  0000 C CNN
-F 2 "keyboard:SW_Cherry_MX_2.00u_Hotswap" H 19500 8020 50  0001 C CNN
+F 2 "keyboard:SW_Cherry_MX_2.25u_Hotswap" H 19500 8020 50  0001 C CNN
 F 3 "" H 19500 8020 50  0000 C CNN
 	1    19500 8020
@@
 	1    0    0    -1
 $EndComp
-$Comp
-L keyboard:MountingHole MountBaseMiddleTop7
-U 1 1 615C07FA
-P 9560 820
-F 0 "MountBaseMiddleTop7" H 9660 866 50  0000 L CNN
-F 1 "MountingHole" H 9660 775 50  0000 L CNN
-F 2 "keyboard:MountingHole_2.2mm_M2_Pad_Via" H 9910 670 50  0001 C CNN
-F 3 "" H 9560 820 50  0001 C CNN
-	1    9560 820
-	1    0    0    -1
-$EndComp
-$Comp
-L keyboard:MountingHole MountBaseMiddleTop8
-U 1 1 615C0800
-P 9560 990
-F 0 "MountBaseMiddleTop8" H 9660 1036 50  0000 L CNN
-F 1 "MountingHole" H 9660 945 50  0000 L CNN
-F 2 "keyboard:MountingHole_2.2mm_M2_Pad_Via" H 9910 840 50  0001 C CNN
-F 3 "" H 9560 990 50  0001 C CNN
-	1    9560 990
-	1    0    0    -1
-$EndComp

Commit message: reviewe kanagawa rev1
Parts:
- J1: footprint keyboard:OLED_128x64_I2C -> keyboard:OLED_128x64_I2C_cutout
Changed lines of the file:
@@
 F 0 "J1" H 3508 1205 50  0000 C CNN
 F 1 "Conn_01x04" H 3508 1296 50  0000 C CNN
-F 2 "keyboard:OLED_128x64_I2C" H 3740 1230 50  0001 C CNN
+F 2 "keyboard:OLED_128x64_I2C_cutout" H 3740 1230 50  0001 C CNN
 F 3 "" H 3590 1630 50  0001 C CNN
 	1    3590 1630

Commit message: edit pcb
Parts:
- DA0, DA1, DA10, DA11, DA12, DA13, DA2, DA3, DA4, DA5, DA6, DA7, DA8, DA9, DB0, DB1, DB10, DB11, DB12, DB13, DB2, DB3, DB4, DB5, DB6, DB7, DB8, DB9, DC0, DC1, DC10, DC11, DC12, DC13, DC2, DC3, DC4, DC5, DC6, DC7, DC8, DC9, DD0, DD1, DD10, DD11, DD12, DD13, DD2, DD3, DD4, DD5, DD6, DD7, DD8, DD9, DE0, DE1, DE10, DE11, DE12, DE13, DE2, DE3, DE4, DE5, DE6, DE7, DE8, DE9, DF0, DF1, DF10, DF11, DF12, DF13, DF2, DF3, DF4, DF5, DF6, DF7, DF8, DF9: footprint keyboard:Diode_SMD_THT -> keyboard:Diode_THT
- KD13, KE13, KF13: footprint keyboard:SW_Cherry_MX_1.25u_Hotswap -> keyboard:SW_Cherry_MX_1.00u_Hotswap
- R1, R2: footprint keyboard:Resistors_SMD_THT -> keyboard:Resistors_THT
