File: Kanagawa/rev1_rgb/Kanagawa.sch (KiCad schematic (older format))
At the start: 180 parts, among them J1 Conn_01x04, SW99 Rotary_Encoder_Switch, U0 Elite-C

Commit message: Add new case stl
Parts:
- added MountBaseMiddleTop7, MountBaseMiddleTop8: MountingHole, keyboard:MountingHole_2.2mm_M2_Pad_Via, symbol keyboard:MountingHole
- DA0, DA1, DA10, DA11, DA12, DA13, DA2, DA3, DA4, DA5, DA6, DA7, DA8, DA9, DB0, DB1, DB10, DB11, DB12, DB13, DB2, DB3, DB4, DB5, DB6, DB7, DB8, DB9, DC0, DC1, DC10, DC11, DC12, DC13, DC2, DC3, DC4, DC5, DC6, DC7, DC8, DC9, DD0, DD1, DD10, DD11, DD12, DD13, DD2, DD3, DD4, DD5, DD6, DD7, DD8, DD9, DE0, DE1, DE10, DE11, DE12, DE13, DE2, DE3, DE4, DE5, DE6, DE7, DE8, DE9, DF0, DF1, DF10, DF11, DF12, DF13, DF2, DF3, DF4, DF5, DF6, DF7, DF8, DF9: footprint keyboard:Diode_SMD_THT -> keyboard:Diode_THT
- J1: footprint keyboard:OLED_128x64_I2C -> keyboard:OLED_128x64_I2C_cutout
- KD13, KE13, KF13, KF7, KF9: footprint keyboard:SW_Cherry_MX_1.25u_SK6812MINI-E_Hotswap -> keyboard:SW_Cherry_MX_1.00u_SK6812MINI-E_Hotswap
- KE11: footprint keyboard:SW_Cherry_MX_2.25u_SK6812MINI-E_Hotswap -> keyboard:SW_Cherry_MX_1.75u_SK6812MINI-E_Hotswap
Connections:
- net OUT_A0 is gone; now on net IN_B0: KA0.3 (DOUT)
- net OUT_A1 is gone; now on net IN_A0: KA1.3 (DOUT)
- net OUT_A10 is gone; now on net IN_A9: KA10.3 (DOUT)
- net OUT_A11 is gone; now on net IN_A10: KA11.3 (DOUT)
- net OUT_A2 is gone; now on net IN_A1: KA2.3 (DOUT)
- net OUT_A3 is gone; now on net IN_A2: KA3.3 (DOUT)
- net OUT_A4 is gone; now on net IN_A3: KA4.3 (DOUT)
- net OUT_A5 is gone; now on net IN_A4: KA5.3 (DOUT)
- net OUT_A6 is gone; now on net IN_A5: KA6.3 (DOUT)
- net OUT_A7 is gone; now on net IN_A6: KA7.3 (DOUT)
- net OUT_A8 is gone; now on net IN_A7: KA8.3 (DOUT)
- net OUT_A9 is gone; now on net IN_A8: KA9.3 (DOUT)
- net OUT_B0 is gone; now on net IN_B1: KB0.3 (DOUT)
- net OUT_B1 is gone; now on net IN_B2: KB1.3 (DOUT)
- net OUT_B10 is gone; now on net IN_B11: KB10.3 (DOUT)
- net OUT_B2 is gone; now on net IN_B3: KB2.3 (DOUT)
- net OUT_B3 is gone; now on net IN_B4: KB3.3 (DOUT)
- net OUT_B4 is gone; now on net IN_B5: KB4.3 (DOUT)
- net OUT_B5 is gone; now on net IN_B6: KB5.3 (DOUT)
- net OUT_B6 is gone; now on net IN_B7: KB6.3 (DOUT)
- net OUT_B7 is gone; now on net IN_B8: KB7.3 (DOUT)
- net OUT_B8 is gone; now on net IN_B9: KB8.3 (DOUT)
- net OUT_B9 is gone; now on net IN_B10: KB9.3 (DOUT)
- net OUT_C1 is gone; now on net IN_C0: KC1.3 (DOUT)
- net OUT_C10 is gone; now on net IN_C9: KC10.3 (DOUT)
- net OUT_C11 is gone; now on net IN_C10: KC11.3 (DOUT)
- net OUT_C2 is gone; now on net IN_C1: KC2.3 (DOUT)
- net OUT_C3 is gone; now on net IN_C2: KC3.3 (DOUT)
- net OUT_C4 is gone; now on net IN_C3: KC4.3 (DOUT)
- net OUT_C5 is gone; now on net IN_C4: KC5.3 (DOUT)
- net OUT_C6 is gone; now on net IN_C5: KC6.3 (DOUT)
- net OUT_C7 is gone; now on net IN_C6: KC7.3 (DOUT)
- net OUT_C8 is gone; now on net IN_C7: KC8.3 (DOUT)
- net OUT_C9 is gone; now on net IN_C8: KC9.3 (DOUT)
- net IN_A11: now also KA12.3 (DOUT)
- net IN_C11: now also KC12.3 (DOUT)
- net RGB: now also KA12.5 (DIN)
- net col00: now also KD13.1; no longer KA12.1
- net col01: now also KE13.1; no longer KB12.1
- net col02: now also KF13.1; no longer KB13.1
- net col03: now also KE12.1; no longer KC12.1
- net col04: now also KF12.1; no longer KC13.1
- net col06: now also KC12.1; no longer KE12.1
- net col07: now also KC13.1; no longer KF12.1
- net col08: now also KB12.1; no longer KF13.1
- net col09: now also KB13.1; no longer KE13.1
- net col10: now also KA12.1, U0.1 (TX0/PD3); no longer KD13.1, U0.2 (RX1/PD2)
- net col11: now also U0.2 (RX1/PD2); no longer U0.1 (TX0/PD3)
- removed net IN: KA12.5 (DIN), KB12.5 (DIN), KB13.5 (DIN), KC12.5 (DIN), KC13.5 (DIN), KD0.5 (DIN), KD1.5 (DIN), KD10.5 (DIN), KD11.5 (DIN), KD12.5 (DIN), KD13.5 (DIN), KD2.5 (DIN), KD3.5 (DIN), KD4.5 (DIN), KD5.5 (DIN), KD6.5 (DIN), KD7.5 (DIN), KD8.5 (DIN), KD9.5 (DIN), KE0.5 (DIN), KE1.5 (DIN), KE10.5 (DIN), KE11.5 (DIN), KE12.5 (DIN), KE13.5 (DIN), KE2.5 (DIN), KE3.5 (DIN), KE4.5 (DIN), KE5.5 (DIN), KE6.5 (DIN), KE7.5 (DIN), KE8.5 (DIN), KE9.5 (DIN), KF0.5 (DIN), KF1.5 (DIN), KF10.5 (DIN), KF11.5 (DIN), KF12.5 (DIN), KF13.5 (DIN), KF2.5 (DIN), KF3.5 (DIN), KF4.5 (DIN), KF5.5 (DIN), KF6.5 (DIN), KF7.5 (DIN), KF8.5 (DIN), KF9.5 (DIN)
- removed net OUT: KA12.3 (DOUT), KB12.3 (DOUT), KB13.3 (DOUT), KC12.3 (DOUT), KC13.3 (DOUT), KD0.3 (DOUT), KD1.3 (DOUT), KD10.3 (DOUT), KD11.3 (DOUT), KD12.3 (DOUT), KD13.3 (DOUT), KD2.3 (DOUT), KD3.3 (DOUT), KD4.3 (DOUT), KD5.3 (DOUT), KD6.3 (DOUT), KD7.3 (DOUT), KD8.3 (DOUT), KD9.3 (DOUT), KE0.3 (DOUT), KE1.3 (DOUT), KE10.3 (DOUT), KE11.3 (DOUT), KE12.3 (DOUT), KE13.3 (DOUT), KE2.3 (DOUT), KE3.3 (DOUT), KE4.3 (DOUT), KE5.3 (DOUT), KE6.3 (DOUT), KE7.3 (DOUT), KE8.3 (DOUT), KE9.3 (DOUT), KF0.3 (DOUT), KF1.3 (DOUT), KF10.3 (DOUT), KF11.3 (DOUT), KF12.3 (DOUT), KF13.3 (DOUT), KF2.3 (DOUT), KF3.3 (DOUT), KF4.3 (DOUT), KF5.3 (DOUT), KF6.3 (DOUT), KF7.3 (DOUT), KF8.3 (DOUT), KF9.3 (DOUT)
- net OUT_B11 renamed IN_B12
- net IN_B12: now also KB12.5 (DIN)
- net OUT_C0 renamed IN_D0
- net IN_D0: now also KD0.5 (DIN)
- new net IN_B13: KB12.3 (DOUT), KB13.5 (DIN)
- new net IN_C12: KC12.5 (DIN), KC13.3 (DOUT)
- new net IN_C13: KB13.3 (DOUT), KC13.5 (DIN)
- new net IN_D1: KD0.3 (DOUT), KD1.5 (DIN)
- new net IN_D10: KD10.5 (DIN), KD9.3 (DOUT)
- new net IN_D11: KD10.3 (DOUT), KD11.5 (DIN)
- new net IN_D12: KD11.3 (DOUT), KD12.5 (DIN)
- new net IN_D13: KD13.5 (DIN), KE13.3 (DOUT)
- new net IN_D2: KD1.3 (DOUT), KD2.5 (DIN)
- new net IN_D3: KD2.3 (DOUT), KD3.5 (DIN)
- new net IN_D4: KD3.3 (DOUT), KD4.5 (DIN)
- new net IN_D5: KD4.3 (DOUT), KD5.5 (DIN)
- new net IN_D6: KD5.3 (DOUT), KD6.5 (DIN)
- new net IN_D7: KD6.3 (DOUT), KD7.5 (DIN)
- new net IN_D8: KD7.3 (DOUT), KD8.5 (DIN)
- new net IN_D9: KD8.3 (DOUT), KD9.5 (DIN)
- new net IN_E0: KE0.5 (DIN), KE1.3 (DOUT)
- new net IN_E1: KE1.5 (DIN), KE2.3 (DOUT)
- new net IN_E10: KE10.5 (DIN), KE11.3 (DOUT)
- new net IN_E11: KD12.3 (DOUT), KE11.5 (DIN)
- new net IN_E12: KE12.5 (DIN), KF11.3 (DOUT)
- new net IN_E13: KE13.5 (DIN), KF13.3 (DOUT)
- new net IN_E2: KE2.5 (DIN), KE3.3 (DOUT)
- new net IN_E3: KE3.5 (DIN), KE4.3 (DOUT)
- new net IN_E4: KE4.5 (DIN), KE5.3 (DOUT)
- new net IN_E5: KE5.5 (DIN), KE6.3 (DOUT)
- new net IN_E6: KE6.5 (DIN), KE7.3 (DOUT)
- new net IN_E7: KE7.5 (DIN), KE8.3 (DOUT)
- new net IN_E8: KE8.5 (DIN), KE9.3 (DOUT)
- new net IN_E9: KE10.3 (DOUT), KE9.5 (DIN)
- new net IN_F0: KE0.3 (DOUT), KF0.5 (DIN)
- new net IN_F1: KF0.3 (DOUT), KF1.5 (DIN)
- new net IN_F10: KF10.5 (DIN), KF9.3 (DOUT)
- new net IN_F11: KF10.3 (DOUT), KF11.5 (DIN)
- new net IN_F12: KE12.3 (DOUT), KF12.5 (DIN)
- new net IN_F13: KF12.3 (DOUT), KF13.5 (DIN)
- new net IN_F2: KF1.3 (DOUT), KF2.5 (DIN)
- new net IN_F3: KF2.3 (DOUT), KF3.5 (DIN)
- new net IN_F4: KF3.3 (DOUT), KF4.5 (DIN)
- new net IN_F5: KF4.3 (DOUT), KF5.5 (DIN)
- new net IN_F6: KF5.3 (DOUT), KF6.5 (DIN)
- new net IN_F7: KF6.3 (DOUT), KF7.5 (DIN)
- new net IN_F8: KF7.3 (DOUT), KF8.5 (DIN)
- new net IN_F9: KF8.3 (DOUT), KF9.5 (DIN)
- new net OUT_D13: KD13.3 (DOUT)
- no-connect marks 0 -> 1
Other:
- moved on the sheet: DA12, DB12, DB13, DC12, DC13, DD13, DE12, DE13, DF12, DF13, J1, KA12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
