File: Kanagawa/rev1_rgb/Rotary_Encoder/Kanagawa_rgb_encoder.kicad_pcb (KiCad board)
At the start: 2 copper layers, 18 x 17 mm, 2 parts, among them J1 Conn_01x05

Commit message: edit kanagawa rgb
Other:
- outline, holes or cut-outs redrawn
Changed lines of the file:
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@@
     )
   )
+  (gr_line (start 55.89 86.712) (end 75.89 86.712) (layer "Dwgs.User") (width 0.1))
   (gr_arc (start 72.890001 76.231999) (mid 74.304215 76.817785) (end 74.89 78.232) (layer "Edge.Cuts") (width 0.05))
+  (gr_line (start 69.89 86.912) (end 61.89 86.912) (layer "Edge.Cuts") (width 0.05))
+  (gr_line (start 61.89 86.912) (end 61.89 84.912) (layer "Edge.Cuts") (width 0.05))
   (gr_arc (start 58.890001 93.231999) (mid 57.475787 92.646214) (end 56.89 91.232) (layer "Edge.Cuts") (width 0.05))
   (gr_line (start 74.89 78.232) (end 74.89 91.232) (layer "Edge.Cuts") (width 0.05))
+  (gr_line (start 61.89 84.912) (end 69.89 84.912) (layer "Edge.Cuts") (width 0.05))
   (gr_line (start 58.89 76.232) (end 72.890001 76.231999) (layer "Edge.Cuts") (width 0.05))
   (gr_line (start 72.890001 93.232001) (end 58.89 93.232) (layer "Edge.Cuts") (width 0.05))
@@
   (gr_arc (start 56.89 78.232) (mid 57.475786 76.817786) (end 58.89 76.232) (layer "Edge.Cuts") (width 0.05))
   (gr_arc (start 74.89 91.232) (mid 74.304215 92.646214) (end 72.890001 93.232001) (layer "Edge.Cuts") (width 0.05))
+  (gr_line (start 69.89 84.912) (end 69.89 86.912) (layer "Edge.Cuts") (width 0.05))
+  (gr_line (start 56.64 86.712) (end 56.64 85.112) (layer "Margin") (width 0.05))
+  (gr_line (start 56.64 82.012) (end 56.64 80.412) (layer "Margin") (width 0.05))
+  (gr_line (start 55.39 80.412) (end 56.64 80.412) (layer "Margin") (width 0.05))
+  (gr_line (start 75.14 82.012) (end 75.14 80.412) (layer "Margin") (width 0.05))
+  (gr_line (start 61.89 86.912) (end 69.89 86.912) (layer "Margin") (width 0.05))
+  (gr_line (start 69.89 86.912) (end 69.89 84.912) (layer "Margin") (width 0.05))
+  (gr_line (start 56.89 93.212) (end 74.89 93.212) (layer "Margin") (width 0.05))
+  (gr_line (start 75.14 85.112) (end 76.39 85.112) (layer "Margin") (width 0.05))
+  (gr_line (start 75.14 86.712) (end 76.39 86.712) (layer "Margin") (width 0.05))
+  (gr_line (start 74.89 93.212) (end 74.89 76.212) (layer "Margin") (width 0.05))
+  (gr_line (start 75.14 80.412) (end 76.39 80.412) (layer "Margin") (width 0.05))
+  (gr_line (start 55.39 82.012) (end 56.64 82.012) (layer "Margin") (width 0.05))
+  (gr_line (start 61.89 84.912) (end 61.89 86.912) (layer "Margin") (width 0.05))
+  (gr_line (start 56.89 76.212) (end 56.89 93.212) (layer "Margin") (width 0.05))
+  (gr_line (start 75.14 86.712) (end 75.14 85.112) (layer "Margin") (width 0.05))
+  (gr_line (start 56.64 86.712) (end 55.39 86.712) (layer "Margin") (width 0.05))
+  (gr_line (start 74.89 76.212) (end 56.89 76.212) (layer "Margin") (width 0.05))
+  (gr_line (start 69.89 84.912) (end 61.89 84.912) (layer "Margin") (width 0.05))
+  (gr_line (start 76.39 82.012) (end 75.14 82.012) (layer "Margin") (width 0.05))
+  (gr_line (start 55.39 85.112) (end 56.64 85.112) (layer "Margin") (width 0.05))
   (gr_text "S1\n" (at 68.42 92.872) (layer "F.SilkS")
     (effects (font (size 0.5 0.5) (thickness 0.1)))
@@
     (effects (font (size 0.5 0.5) (thickness 0.1)))
   )
-  (segment (start 58.39 83.332) (end 60.8 85.742) (width 0.25) (layer "F.Cu") (net 1))
-  (segment (start 60.8 85.742) (end 60.8 91.412) (width 0.25) (layer "F.Cu") (net 1))
-  (segment (start 58.39 80.832) (end 63.34 85.782) (width 0.25) (layer "F.Cu") (net 2))
-  (segment (start 63.34 85.782) (end 63.34 91.412) (width 0.25) (layer "F.Cu") (net 2))
+  (dimension (type aligned) (layer "Dwgs.User")
+    (pts (xy 56.89 78.232) (xy 74.89 78.232))
+    (height -5.97)
+    (gr_text "18,0000 mm" (at 65.89 71.112) (layer "Dwgs.User")
+      (effects (font (size 1 1) (thickness 0.15)))
+    )
+    (format (units 3) (units_format 1) (precision 4))
+    (style (thickness 0.1) (arrow_length 1.27) (text_position_mode 0) (extension_height 0.58642) (extension_offset 0.5) keep_text_aligned)
+  )
+  (dimension (type aligned) (layer "Dwgs.User")
+    (pts (xy 58.89 76.232) (xy 58.89 93.232))
+    (height 6.01)
+    (gr_text "17,0000 mm" (at 51.73 84.732 90) (layer "Dwgs.User")
+      (effects (font (size 1 1) (thickness 0.15)))
+    )
+    (format (units 3) (units_format 1) (precision 4))
+    (style (thickness 0.1) (arrow_length 1.27) (text_position_mode 0) (extension_height 0.58642) (extension_offset 0.5) keep_text_aligned)
+  )
+  (segment (start 60 89.162) (end 60 85.602) (width 0.25) (layer "F.Cu") (net 1))
+  (segment (start 60.815 91.412) (end 60.815 89.977) (width 0.25) (layer "F.Cu") (net 1))
+  (segment (start 60.44 89.602) (end 60 89.162) (width 0.25) (layer "F.Cu") (net 1))
+  (segment (start 60 85.602) (end 60 84.942) (width 0.25) (layer "F.Cu") (net 1))
+  (segment (start 60.815 89.977) (end 60.44 89.602) (width 0.25) (layer "F.Cu") (net 1))
+  (segment (start 60 84.942) (end 58.39 83.332) (width 0.25) (layer "F.Cu") (net 1))
+  (segment (start 60.44952 86.502) (end 60.44952 82.89152) (width 0.25) (layer "F.Cu") (net 2))
+  (segment (start 63.355 91.412) (end 60.44952 88.50652) (width 0.25) (layer "F.Cu") (net 2))
+  (segment (start 60.44952 88.50652) (end 60.44952 86.502) (width 0.25) (layer "F.Cu") (net 2))
+  (segment (start 60.44952 82.89152) (end 58.39 80.832) (width 0.25) (layer "F.Cu") (net 2))
   (segment (start 59.6 92.812) (end 58.95 92.162) (width 0.25) (layer "B.Cu") (net 3))
   (segment (start 65.88 91.412) (end 64.48 92.812) (width 0.25) (layer "B.Cu") (net 3))
@@
   (segment (start 68.42 91.412) (end 72.89 86.942) (width 0.25) (layer "B.Cu") (net 4))
   (segment (start 72.89 86.942) (end 72.89 85.832) (width 0.25) (layer "B.Cu") (net 4))
-  (segment (start 72.89 80.832) (end 70.96 82.762) (width 0.25) (layer "F.Cu") (net 5))
-  (segment (start 70.96 82.762) (end 70.96 91.412) (width 0.25) (layer "F.Cu") (net 5))
+  (segment (start 70.975 82.747) (end 72.89 80.832) (width 0.25) (layer "F.Cu") (net 5))
+  (segment (start 70.975 91.412) (end 70.975 82.747) (width 0.25) (layer "F.Cu") (net 5))
+  (group "" (id a790683a-069b-4421-8438-777be1d18cf0)
+    (members
+      101afe42-5ef3-4b70-8f0a-b0d5217abdbd
+      11940ca7-8823-438b-afda-02830975f06f
+      195ce8f5-74a9-4f0c-a43b-b99ac0cb690a
+      2535776b-bd58-4223-8268-a2161b7d7d29
+      33ba7e7a-c777-4635-9a0d-28eb2c0c7247
+      38eefd17-cc22-4d50-addc-10c507c0d11a
+      414c79b4-a110-435e-9ad1-f66f45e52958
+      42991e70-cf87-4d06-bcb3-aed0ee3fbdaa
+      6abf4fea-b973-4fef-88fb-bfd229dc0701
+      70f0fed5-5501-4676-aa5f-74c1d0957760
+      8247d3e5-1187-4085-bc20-52202af71d13
+      936e9618-81e2-4923-9896-3f8ee7dde9c4
+      96d7e503-19bd-45c0-975f-6efc723a7dd3
+      aab24421-830f-4a74-a6cf-38f35075e2be
+      b8c39d2e-c86c-48fd-81f9-45d26be85412
+      e41872d6-dd23-4520-b16d-c9059845a942
+      e7d256be-aa65-4de5-9abd-350eebce835c
+      e9d70a2f-e816-4618-b0b6-1f308f4d3e29
+      f1e292bc-b765-4b92-aa0f-b7d09020651b
+      fa524a96-486b-4148-8215-fdeb63421ea5
+    )
+  )
 )
