File: Kanagawa/rev2_rgb/ANSI/Kanagawa_rgb_ansi.kicad_sch (KiCad schematic)
At the start: 185 parts, among them J1 Oled128x32, J3 OledJump2, J4 OledJump1, J5 RGB_Out, J6 RGB_Selector_Pin, J7 RGB_Selector_Matrix, J8 Conn_01x05, U1 Pico

Commit message: rework rev2 kanagawa
Parts:
- removed J3: OledJump2, keyboard:Jumper_3pins, symbol keyboard:Conn_01x03
- removed J4: OledJump1, keyboard:Jumper_3pins, symbol keyboard:Conn_01x03
- added J2: Conn_01x05, keyboard:PinHeader_1x05_P2.54mm_Vertical, symbol keyboard:Conn_01x05
- added MountBase2: MountingHole USB breakout, keyboard:MountingHole_3.2mm_M2_Pad_Via, symbol keyboard:MountingHole
- added MountBaseMiddleTop7, MountBaseMiddleTop8: MountingHole, keyboard:MountingHole_3.2mm_M2_Pad_Via, symbol keyboard:MountingHole
- added SWA13: Rotary_Encoder_Switch, keyboard:RotaryEncoder_Alps_EC11E-Switch_Vertical_H20mm, symbol keyboard:Rotary_Encoder_Switch
- KA0, KA1, KA10, KA11, KA12, KA2, KA3, KA4, KA5, KA6, KA7, KA8, KA9, KB0, KB1, KB10, KB11, KB12, KB2, KB3, KB4, KB5, KB6, KB7, KB8, KB9, KC1, KC10, KC11, KC12, KC2, KC3, KC4, KC5, KC6, KC7, KC8, KC9, KD1, KD10, KD11, KD13, KD2, KD3, KD4, KD5, KD6, KD7, KD8, KD9, KE1, KE10, KE12, KE13, KE2, KE3, KE4, KE5, KE6, KE7, KE8, KE9, KF1, KF10, KF11, KF12, KF13, KF3, KF6, KF7, KF8, KF9: footprint keyboard:SW_Cherry_MX_1.00u_SK6812MINI -> keyboard:SW_Cherry_MX_1.00u_SK6812MINI-E_Hotswap
- KB13, KF4, KF5: footprint keyboard:SW_Cherry_MX_1.00u_SK6812MINI -> keyboard:SW_Cherry_MX_2.00u_SK6812MINI-E_Hotswap
- KC0: footprint keyboard:SW_Cherry_MX_1.00u_SK6812MINI -> keyboard:SW_Cherry_MX_1.50u_SK6812MINI-E_Hotswap
- KD0, KE11: footprint keyboard:SW_Cherry_MX_1.00u_SK6812MINI -> keyboard:SW_Cherry_MX_1.75u_SK6812MINI-E_Hotswap
- KE0: footprint keyboard:SW_Cherry_MX_1.00u_SK6812MINI -> keyboard:SW_Cherry_MX_2.25u_SK6812MINI-E_Hotswap
- KF0, KF2: footprint keyboard:SW_Cherry_MX_1.00u_SK6812MINI -> keyboard:SW_Cherry_MX_1.25u_SK6812MINI-E_Hotswap
- MountBase1: renamed from MountMiddle0; footprint keyboard:Keebio_USB-C_breakout_shadow -> keyboard:MountingHole_3.2mm_M2_Pad_Via
- renumbered J8 to J3
Connections:
- net OledPin1 is gone; now on net GND: J1.1 (Pin_1)
- net OledPin2 is gone; now on net VCC: J1.2 (Pin_2)
- net ENCA: now also J3.3 (Pin_3); no longer J3.2 (Pin_2)
- net ENCB: now also J3.2 (Pin_2); no longer J3.3 (Pin_3)
- net IN_D13: now also KE0.4 (DOUT); no longer KE13.4 (DOUT)
- net IN_E12: now also KF12.4 (DOUT); no longer KF11.4 (DOUT)
- net IN_E13: now also KD13.4 (DOUT); no longer KF13.4 (DOUT)
- net IN_F0: now also KF1.4 (DOUT); no longer KE0.4 (DOUT)
- net IN_F1: now also KF2.4 (DOUT); no longer KF0.4 (DOUT)
- net IN_F10: now also KF11.4 (DOUT); no longer KF9.4 (DOUT)
- net IN_F11: now also KE12.4 (DOUT); no longer KF10.4 (DOUT)
- net IN_F12: now also KF13.4 (DOUT); no longer KE12.4 (DOUT)
- net IN_F13: now also KE13.4 (DOUT); no longer KF12.4 (DOUT)
- net IN_F2: now also KF3.4 (DOUT); no longer KF1.4 (DOUT)
- net IN_F3: now also KF4.4 (DOUT); no longer KF2.4 (DOUT)
- net IN_F4: now also KF5.4 (DOUT); no longer KF3.4 (DOUT)
- net IN_F5: now also KF6.4 (DOUT); no longer KF4.4 (DOUT)
- net IN_F6: now also KF7.4 (DOUT); no longer KF5.4 (DOUT)
- net IN_F7: now also KF8.4 (DOUT); no longer KF6.4 (DOUT)
- net IN_F8: now also KF9.4 (DOUT); no longer KF7.4 (DOUT)
- net IN_F9: now also KF10.4 (DOUT); no longer KF8.4 (DOUT)
- net RGB_Out: now also KF0.4 (DOUT); no longer KD13.4 (DOUT)
- new net A: J2.3 (Pin_3), SWA13.A
- new net B: J2.2 (Pin_2), SWA13.B
- new net G: J2.1 (Pin_1), SWA13.C
- new net S1: J2.4 (Pin_4), SWA13.S1
- new net S2: J2.5 (Pin_5), SWA13.S2
Other:
- moved on the sheet: J3, J5, J6, J7, MountBase1

Commit message: add stamp version
Connections:
- net G is gone; now on net GND: J2.1 (Pin_1), SWA13.C
Changed lines of the file:
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@@
     (effects (font (size 1.27 1.27)) (justify right bottom))
   )
-  (label "G" (at 30.353 121.92 180)
+  (label "GND" (at 30.353 121.92 180)
     (effects (font (size 1.27 1.27)) (justify right bottom))
   )
@@
     (effects (font (size 1.27 1.27)) (justify left bottom))
   )
-  (label "G" (at 50.165 104.648 0)
-    (effects (font (size 1.27 1.27)) (justify left bottom))
-  )
+  (label "GND" (at 50.165 104.648 0)
+    (effects (font (size 1.27 1.27)) (justify left bottom))
+  )

Commit message: edit stamp version
Parts:
- removed J6: RGB_Selector_Pin, keyboard:Jumper_3pins, symbol keyboard:Conn_01x03
- removed J7: RGB_Selector_Matrix, keyboard:Jumper_2pins, symbol keyboard:Conn_01x02
- renumbered J5 to J4
Connections:
- net RGB is gone; now on net RGB_Matrix: U1.34 (GPIO28_ADC2)
- net RGB_Pin is gone; now on net RGB_Out: J4.1 (Pin_1)
Other:
- moved on the sheet: J1, J4, SWA13
