File: Kanagawa/rev2_rgb/ANSI_stamp/Kanagawa_rgb_ansi_stamp.kicad_sch (KiCad schematic)
At the start: 184 parts, among them J1 Oled128x32, J2 Conn_01x05, J3 Conn_01x05, U0 RP2040_Stamp

Commit message: edit stamp version
Parts:
- removed F0: 500mA, keyboard:polyfuse_5.1mm, symbol Device:Polyfuse_Small
- added J4: Conn_01x03, keyboard:conn_3pins, symbol keyboard:Conn_01x03
Connections:
- net +5V: now also JUSB1.A4 (VBUS), JUSB1.A9 (VBUS), JUSB1.B4 (VBUS), JUSB1.B9 (VBUS)
- net ENCA: now also U0.4 (GPIO3); no longer U0.2 (GPIO1)
- net ENCB: now also U0.5 (GPIO4); no longer U0.3 (GPIO2)
- net GND: now also J4.3 (Pin_3)
- net RGB_Matrix: now also U0.25 (GPIO24); no longer U0.15 (GPIO14)
- net RGB_Out: now also J4.1 (Pin_1)
- net SCL: now also U0.16 (GPIO15); no longer U0.14 (GPIO13)
- net SDA: now also U0.15 (GPIO14); no longer U0.13 (GPIO12)
- net VCC: now also J4.2 (Pin_2)
- net col05: now also U0.24 (GPIO23); no longer U0.25 (GPIO24)
- net col06: now also U0.23 (GPIO22); no longer U0.24 (GPIO23)
- net col07: now also U0.22 (GPIO21); no longer U0.23 (GPIO22)
- net col08: now also U0.21 (GPIO20); no longer U0.22 (GPIO21)
- net col09: now also U0.20 (GPIO19); no longer U0.21 (GPIO20)
- net col10: now also U0.19 (GPIO18); no longer U0.20 (GPIO19)
- net col11: now also U0.18 (GPIO17); no longer U0.19 (GPIO18)
- net col12: now also U0.17 (GPIO16); no longer U0.18 (GPIO17)
- net col13: now also U0.3 (GPIO2); no longer U0.17 (GPIO16)
- net row00: now also U0.14 (GPIO13); no longer U0.9 (GPIO8)
- net row01: now also U0.13 (GPIO12); no longer U0.8 (GPIO7)
- net row02: now also U0.12 (GPIO11); no longer U0.7 (GPIO6)
- net row03: now also U0.9 (GPIO8); no longer U0.6 (GPIO5)
- net row04: now also U0.10 (GPIO9); no longer U0.5 (GPIO4)
- net row05: now also U0.11 (GPIO10); no longer U0.4 (GPIO3)
- no-connect marks 7 -> 12
Other:
- moved on the sheet: JUSB1

Commit message: edit kanagawa
Parts:
- removed MountBaseMiddleTop1, MountBaseMiddleTop2, MountBaseMiddleTop3, MountBaseMiddleTop4, MountBaseMiddleTop5, MountBaseMiddleTop6, MountBaseMiddleTop7, MountBaseMiddleTop8: MountingHole, keyboard:MountingHole_3.2mm_M2_Pad_Via, symbol keyboard:MountingHole
- added J5: Conn_01x02, Connector_JST:JST_PH_S2B-PH-SM4-TB_1x02-1MP_P2.00mm_Horizontal, symbol keyboard:Conn_01x02
- added J6: I2C, keyboard:PinHeader_1x04_P2.54mm_Vertical, symbol keyboard:Conn_01x04
- KF4, KF5: footprint keyboard:SW_Cherry_MX_2.00u_SK6812MINI-E_Hotswap -> keyboard:SW_Cherry_MX_2.00u_SK6812MINI-E_Hotswap_Reversed
Connections:
- net GND: now also J5.2 (Pin_2), J6.1 (Pin_1)
- net SCL: now also U0.27 (GPIO26), J6.3 (Pin_3); no longer U0.16 (GPIO15)
- net SDA: now also U0.26 (GPIO25), J6.4 (Pin_4); no longer U0.15 (GPIO14)
- net VCC: now also J6.2 (Pin_2)
- net col03: now also U0.24 (GPIO23); no longer U0.27 (GPIO26)
- net col04: now also U0.23 (GPIO22); no longer U0.26 (GPIO25)
- net col05: now also U0.22 (GPIO21); no longer U0.24 (GPIO23)
- net col06: now also U0.21 (GPIO20); no longer U0.23 (GPIO22)
- net col07: now also U0.20 (GPIO19); no longer U0.22 (GPIO21)
- net col08: now also U0.19 (GPIO18); no longer U0.21 (GPIO20)
- net col09: now also U0.18 (GPIO17); no longer U0.20 (GPIO19)
- net col10: now also U0.17 (GPIO16); no longer U0.19 (GPIO18)
- net col11: now also U0.16 (GPIO15); no longer U0.18 (GPIO17)
- net col12: now also U0.15 (GPIO14); no longer U0.17 (GPIO16)
- net VBAT: now reaches U0.32 (VBAT)
- net VBAT: now also J5.1 (Pin_1)
- no-connect marks 12 -> 11
