File: Kanagawa/rev2_rgb/ANSI_Pico/Kanagawa_rgb_ansi_pico.kicad_sch (KiCad schematic)
At the start: 176 parts, among them J1 Oled128x32, J2 Conn_01x05, J3 Conn_01x05, J4 Conn_01x03, U0 Pico

Commit message: update pcb
Parts:
- added RSW1: SW_RST, keyboard:SW_RST, symbol keyboard:SW_RST
- U0: symbol keyboard:Pico -> keyboard:Pi Pico; Height (none) -> 1; Manufacturer_Name (none) -> RASPBERRY-PI; Manufacturer_Part_Number (none) -> PICO
Connections:
- net D+: now also U0.TP3 (USB_DP)
- net D-: now also U0.TP2 (USB_DM)
- net ENCA: now also U0.4 (GP2); no longer U0.5 (GPIO3)
- net ENCB: now also U0.5 (GP3); no longer U0.4 (GPIO2)
- net GND: now also U0.TP1 (GND_10), RSW1.2
- new net BOOTSEL: RSW1.1, U0.TP6 (BOOTSEL)
- no-connect marks 11 -> 13
Other:
- moved on the sheet: JUSB2, RSW0
