File: Kanagawa/rev2_rgb H/ISO_Pico/generated_pcbs/base.kicad_pcb (KiCad board)
At the start: 2 copper layers, 335.2 x 145.9 mm, 8 parts

Commit message: adjust kanagawa rev2 pcbs
Parts:
- moved MountBaseTop1 3.00 mm to (47.0, 192.0)
- moved MountBaseTop3 3.00 mm to (115.8, 192.0)
- moved MountBaseTop5 3.00 mm to (239.3, 192.0)
- moved MountBaseTop7 3.00 mm to (376.2, 192.0)
Other:
- outline, holes or cut-outs redrawn
Changed lines of the file:
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@@
   )
   (footprint "keyboard:MountingHole_2.2mm_M2_Pad_Via" (layer "F.Cu")
-    (at 376.225 188.97)
+    (at 376.225 191.97)
     (descr "Mounting Hole 2.2mm, M2")
     (tags "mounting hole 2.2mm m2")
@@
   )
   (footprint "keyboard:MountingHole_2.2mm_M2_Pad_Via" (layer "F.Cu")
-    (at 115.831016 188.97)
+    (at 115.831016 191.97)
     (descr "Mounting Hole 2.2mm, M2")
     (tags "mounting hole 2.2mm m2")
@@
   )
   (footprint "keyboard:MountingHole_2.2mm_M2_Pad_Via" (layer "F.Cu")
-    (at 47 188.97)
+    (at 47 191.97)
     (descr "Mounting Hole 2.2mm, M2")
     (tags "mounting hole 2.2mm m2")
@@
   )
   (footprint "keyboard:MountingHole_2.2mm_M2_Pad_Via" (layer "F.Cu")
-    (at 239.343984 188.97)
+    (at 239.343984 191.97)
     (descr "Mounting Hole 2.2mm, M2")
     (tags "mounting hole 2.2mm m2")
@@
     (pad "1" thru_hole circle (at -1.65 0) (size 0.7 0.7) (drill 0.4) (layers *.Cu *.Mask))
   )
+  (gr_line (start 379.225 57.57) (end 379.225 191.97) (layer "Edge.Cuts") (width 0.05))
+  (gr_arc (start 44 57.57) (mid 44.87868 55.44868) (end 47 54.57) (layer "Edge.Cuts") (width 0.05))
+  (gr_line (start 44 191.97) (end 44 57.57) (layer "Edge.Cuts") (width 0.05))
   (gr_line (start 170.75857 200.469915) (end 184.41643 200.469915) (layer "Edge.Cuts") (width 0.05))
-  (gr_line (start 139.036457 191.97) (end 170.75857 200.469915) (layer "Edge.Cuts") (width 0.05))
-  (gr_line (start 44 188.97) (end 44 57.57) (layer "Edge.Cuts") (width 0.05))
-  (gr_line (start 379.225 57.57) (end 379.225 188.97) (layer "Edge.Cuts") (width 0.05))
-  (gr_arc (start 47 191.97) (mid 44.87868 191.09132) (end 44 188.97) (layer "Edge.Cuts") (width 0.05))
+  (gr_arc (start 47 194.97) (mid 44.87868 194.09132) (end 44 191.97) (layer "Edge.Cuts") (width 0.05))
+  (gr_arc (start 376.225 54.57) (mid 378.34632 55.44868) (end 379.225 57.57) (layer "Edge.Cuts") (width 0.05))
   (gr_line (start 47 54.57) (end 376.225 54.57) (layer "Edge.Cuts") (width 0.05))
-  (gr_line (start 139.036457 191.97) (end 47 191.97) (layer "Edge.Cuts") (width 0.05))
-  (gr_line (start 216.138543 191.97) (end 376.225 191.97) (layer "Edge.Cuts") (width 0.05))
-  (gr_arc (start 376.225 54.57) (mid 378.34632 55.44868) (end 379.225 57.57) (layer "Edge.Cuts") (width 0.05))
-  (gr_arc (start 44 57.57) (mid 44.87868 55.44868) (end 47 54.57) (layer "Edge.Cuts") (width 0.05))
-  (gr_line (start 184.41643 200.469915) (end 216.138543 191.97) (layer "Edge.Cuts") (width 0.05))
-  (gr_arc (start 379.225 188.97) (mid 378.34632 191.09132) (end 376.225 191.97) (layer "Edge.Cuts") (width 0.05))
+  (gr_line (start 184.41643 200.469915) (end 204.942391 194.97) (layer "Edge.Cuts") (width 0.05))
+  (gr_line (start 204.942391 194.97) (end 376.225 194.97) (layer "Edge.Cuts") (width 0.05))
+  (gr_line (start 150.232609 194.97) (end 47 194.97) (layer "Edge.Cuts") (width 0.05))
+  (gr_line (start 150.232609 194.97) (end 170.75857 200.469915) (layer "Edge.Cuts") (width 0.05))
+  (gr_arc (start 379.225 191.97) (mid 378.34632 194.09132) (end 376.225 194.97) (layer "Edge.Cuts") (width 0.05))
   (zone (net 1) (net_name "GND") (layer "F.Cu") (hatch edge 0.508)
     (connect_pads (clearance 0.508))
