File: Kanagawa/rev2_rgb H/ISO_Pico/generated_pcbs/top.kicad_pcb (KiCad board)
At the start: 2 copper layers, 335.2 x 145.9 mm, 16 parts

Commit message: iso H
Other:
- outline, holes or cut-outs redrawn

Commit message: adjust kanagawa rev2 pcbs
Parts:
- moved MountBaseTop1 3.00 mm to (47.0, 192.0)
- moved MountBaseTop3 3.00 mm to (115.8, 192.0)
- moved MountBaseTop5 3.00 mm to (239.3, 192.0)
- moved MountBaseTop7 3.00 mm to (376.2, 192.0)
Other:
- outline, holes or cut-outs redrawn
