File: Kanagawa/rev2_rgb H/ANSI_Pico/generated_pcbs/top.kicad_pcb (KiCad board)
At the start: 2 copper layers, 335.2 x 145.9 mm, 16 parts

Commit message: iso H
Parts:
- added G***: LOGO, keyboard:Wave, F.Cu at (301.3, 87.2)
- added G***: LOGO, keyboard:Wave, F.Cu at (211.9, 87.2)
- added G***: LOGO, keyboard:Wave, F.Cu at (74.4, 87.2)
- added G***: LOGO, keyboard:Wave, F.Cu at (266.9, 83.1)
- added G***: LOGO, keyboard:Wave, F.Cu at (53.8, 83.1)
- added G***: LOGO, keyboard:Wave, F.Cu at (148.5, 165.8)
- added G***: LOGO, keyboard:Wave, F.Cu at (335.6, 87.2)
- added G***: LOGO, keyboard:Wave, F.Cu at (205.0, 87.2)
- added G***: LOGO, keyboard:Wave, F.Cu at (170.6, 87.2)
- added G***: LOGO, keyboard:Wave, F.Cu at (67.6, 83.1)
- added G***: LOGO, keyboard:Wave, F.Cu at (67.6, 87.2)
- added G***: LOGO, keyboard:Wave, F.Cu at (196.6, 178.2)
- added G***: LOGO, keyboard:Wave, F.Cu at (189.7, 165.8)
- added G***: LOGO, keyboard:Wave, F.Cu at (184.4, 87.2)
- added G***: LOGO, keyboard:Wave, F.Cu at (196.6, 174.1)
- added G***: LOGO, keyboard:Wave, F.Cu at (101.9, 87.2)
- added G***: LOGO, keyboard:Wave, F.Cu at (60.7, 83.1)
- added G***: LOGO, keyboard:Wave, F.Cu at (169.1, 169.9)
- added G***: LOGO, keyboard:Wave, F.Cu at (230.9, 165.8)
- added G***: LOGO, keyboard:Wave, F.Cu at (162.2, 169.9)
- added G***: LOGO, keyboard:Wave, F.Cu at (321.9, 83.1)
- added G***: LOGO, keyboard:Wave, F.Cu at (210.3, 169.9)
- added G***: LOGO, keyboard:Wave, F.Cu at (143.1, 87.2)
- added G***: LOGO, keyboard:Wave, F.Cu at (260.0, 83.1)
- added G***: LOGO, keyboard:Wave, F.Cu at (155.4, 169.9)
- added G***: LOGO, keyboard:Wave, F.Cu at (127.9, 165.8)
- added G***: LOGO, keyboard:Wave, F.Cu at (239.4, 83.1)
- added G***: LOGO, keyboard:Wave, F.Cu at (122.5, 83.1)
- added G***: LOGO, keyboard:Wave, F.Cu at (176.0, 174.1)
- added G***: LOGO, keyboard:Wave, F.Cu at (232.5, 87.2)
- added G***: LOGO, keyboard:Wave, F.Cu at (182.8, 174.1)
- added G***: LOGO, keyboard:Wave, F.Cu at (163.8, 83.1)
- added G***: LOGO, keyboard:Wave, F.Cu at (217.2, 170.0)
- added G***: LOGO, keyboard:Wave, F.Cu at (150.0, 83.1)
- added G***: LOGO, keyboard:Wave, F.Cu at (121.0, 165.8)
- added G***: LOGO, keyboard:Wave, F.Cu at (182.8, 169.9)
- added G***: LOGO, keyboard:Wave, F.Cu at (196.6, 169.9)
- added G***: LOGO, keyboard:Wave, F.Cu at (169.1, 178.2)
- added G***: LOGO, keyboard:Wave, F.Cu at (148.5, 169.9)
- added G***: LOGO, keyboard:Wave, F.Cu at (150.0, 87.2)
- added G***: LOGO, keyboard:Wave, F.Cu at (176.0, 169.9)
- added G***: LOGO, keyboard:Wave, F.Cu at (225.6, 83.1)
- added G***: LOGO, keyboard:Wave, F.Cu at (129.4, 87.2)
- added G***: LOGO, keyboard:Wave, F.Cu at (260.0, 87.2)
- added G***: LOGO, keyboard:Wave, F.Cu at (301.3, 83.1)
- added G***: LOGO, keyboard:Wave, F.Cu at (169.1, 165.8)
- added G***: LOGO, keyboard:Wave, F.Cu at (162.2, 178.2)
- added G***: LOGO, keyboard:Wave, F.Cu at (184.4, 83.1)
- added G***: LOGO, keyboard:Wave, F.Cu at (280.6, 87.2)
- added G***: LOGO, keyboard:Wave, F.Cu at (95.0, 87.2)
- added G***: LOGO, keyboard:Wave, F.Cu at (246.2, 87.2)
- added G***: LOGO, keyboard:Wave, F.Cu at (47.0, 83.1)
- added G***: LOGO, keyboard:Wave, F.Cu at (136.3, 83.1)
- added G***: LOGO, keyboard:Wave, F.Cu at (155.3, 165.8)
- added G***: LOGO, keyboard:Wave, F.Cu at (328.7, 83.1)
- added G***: LOGO, keyboard:Wave, F.Cu at (315.0, 87.2)
- added G***: LOGO, keyboard:Wave, F.Cu at (342.5, 83.1)
- added G***: LOGO, keyboard:Wave, F.Cu at (203.4, 174.1)
- added G***: LOGO, keyboard:Wave, F.Cu at (163.8, 87.2)
- added G***: LOGO, keyboard:Wave, F.Cu at (210.3, 165.8)
- added G***: LOGO, keyboard:Wave, F.Cu at (203.4, 165.8)
- added G***: LOGO, keyboard:Wave, F.Cu at (47.0, 87.2)
- added G***: LOGO, keyboard:Wave, F.Cu at (191.3, 87.2)
- added G***: LOGO, keyboard:Wave, F.Cu at (232.5, 83.1)
- added G***: LOGO, keyboard:Wave, F.Cu at (129.4, 83.1)
- added G***: LOGO, keyboard:Wave, F.Cu at (266.9, 87.2)
- added G***: LOGO, keyboard:Wave, F.Cu at (328.7, 87.2)
- added G***: LOGO, keyboard:Wave, F.Cu at (218.8, 83.1)
- added G***: LOGO, keyboard:Wave, F.Cu at (81.3, 87.2)
- added G***: LOGO, keyboard:Wave, F.Cu at (155.4, 174.1)
- added G***: LOGO, keyboard:Wave, F.Cu at (169.1, 174.1)
- added G***: LOGO, keyboard:Wave, F.Cu at (53.8, 87.2)
- added G***: LOGO, keyboard:Wave, F.Cu at (315.0, 83.1)
- added G***: LOGO, keyboard:Wave, F.Cu at (218.7, 87.2)
- added G***: LOGO, keyboard:Wave, F.Cu at (170.7, 83.1)
- added G***: LOGO, keyboard:Wave, F.Cu at (101.9, 83.1)
- added G***: LOGO, keyboard:Wave, F.Cu at (253.1, 83.1)
- added G***: LOGO, keyboard:Wave, F.Cu at (287.5, 87.2)
- added G***: LOGO, keyboard:Wave, F.Cu at (294.4, 83.1)
- added G***: LOGO, keyboard:Wave, F.Cu at (141.6, 169.9)
- added G***: LOGO, keyboard:Wave2, F.Cu at (234.6, 165.8)
- added G***: LOGO, keyboard:Wave, F.Cu at (273.7, 87.2)
- added G***: LOGO, keyboard:Wave, F.Cu at (189.7, 178.2)
- added G***: LOGO, keyboard:Wave, F.Cu at (342.5, 87.2)
- added G***: LOGO, keyboard:Wave, F.Cu at (74.4, 83.1)
- added G***: LOGO, keyboard:Wave, F.Cu at (287.5, 83.1)
- added G***: LOGO, keyboard:Wave, F.Cu at (134.7, 165.8)
- added G***: LOGO, keyboard:Wave, F.Cu at (177.5, 83.1)
- added G***: LOGO, keyboard:Wave, F.Cu at (308.1, 87.2)
- added G***: LOGO, keyboard:Wave, F.Cu at (156.9, 87.2)
- added G***: LOGO, keyboard:Wave, F.Cu at (134.7, 170.0)
- added G***: LOGO, keyboard:Wave, F.Cu at (224.0, 169.9)
- added G***: LOGO, keyboard:Wave, F.Cu at (81.3, 83.1)
- added G***: LOGO, keyboard:Wave, F.Cu at (162.2, 165.8)
- added G***: LOGO, keyboard:Wave, F.Cu at (88.2, 87.2)
- added G***: LOGO, keyboard:Wave, F.Cu at (141.6, 165.8)
- added G***: LOGO, keyboard:Wave, F.Cu at (196.6, 165.8)
- added G***: LOGO, keyboard:Wave, F.Cu at (321.9, 87.2)
- added G***: LOGO, keyboard:Wave, F.Cu at (148.5, 174.1)
- added G***: LOGO, keyboard:Wave, F.Cu at (280.6, 83.1)
- added G***: LOGO, keyboard:Wave, F.Cu at (143.2, 83.1)
- added G***: LOGO, keyboard:Wave, F.Cu at (198.1, 83.1)
- added G***: LOGO, keyboard:Wave, F.Cu at (108.8, 83.1)
- added G***: LOGO, keyboard:Wave, F.Cu at (122.5, 87.2)
- added G***: LOGO, keyboard:Wave, F.Cu at (203.4, 169.9)
- added G***: LOGO, keyboard:Wave, F.Cu at (211.9, 83.1)
- added G***: LOGO, keyboard:Wave, F.Cu at (273.7, 83.1)
- added G***: LOGO, keyboard:Wave, F.Cu at (239.4, 87.2)
- added G***: LOGO, keyboard:Wave, F.Cu at (88.2, 83.1)
- added G***: LOGO, keyboard:Wave, F.Cu at (189.7, 169.9)
- added G***: LOGO, keyboard:Wave, F.Cu at (217.2, 165.8)
- added G***: LOGO, keyboard:Wave, F.Cu at (115.7, 83.1)
- added G***: LOGO, keyboard:Wave, F.Cu at (198.1, 87.2)
- added G***: LOGO, keyboard:Wave, F.Cu at (189.7, 174.1)
- added G***: LOGO, keyboard:Wave, F.Cu at (191.3, 83.1)
- added G***: LOGO, keyboard:Wave, F.Cu at (108.8, 87.2)
- added G***: LOGO, keyboard:Wave, F.Cu at (156.9, 83.1)
- added G***: LOGO, keyboard:Wave, F.Cu at (253.1, 87.2)
- added G***: LOGO, keyboard:Wave, F.Cu at (182.8, 178.2)
- added G***: LOGO, keyboard:Wave, F.Cu at (60.7, 87.2)
- added G***: LOGO, keyboard:Wave, F.Cu at (205.0, 83.1)
- added G***: LOGO, keyboard:Wave, F.Cu at (294.4, 87.2)
- added G***: LOGO, keyboard:Wave, F.Cu at (335.6, 83.1)
- added G***: LOGO, keyboard:Wave, F.Cu at (175.9, 178.2)
- added G***: LOGO, keyboard:Wave, F.Cu at (95.0, 83.1)
- added G***: LOGO, keyboard:Wave, F.Cu at (224.0, 165.8)
- added G***: LOGO, keyboard:Wave, F.Cu at (308.1, 83.1)
- added G***: LOGO, keyboard:Wave, F.Cu at (175.9, 165.8)
- added G***: LOGO, keyboard:Wave, F.Cu at (177.5, 87.2)
- added G***: LOGO, keyboard:Wave, F.Cu at (162.2, 174.1)
- added G***: LOGO, keyboard:Wave, F.Cu at (182.8, 165.8)
- added G***: LOGO, keyboard:Wave, F.Cu at (225.6, 87.2)
- added G***: LOGO, keyboard:Wave, F.Cu at (246.3, 83.1)
- added G***: LOGO, keyboard:Wave, F.Cu at (136.3, 87.2)
- added G***: LOGO, keyboard:Wave, F.Cu at (115.7, 87.2)

Commit message: adjust kanagawa rev2 pcbs
Parts:
- removed G*** (x134): LOGO, keyboard:Wave
- removed G***: LOGO, keyboard:Wave2
- moved MountBaseTop1 3.00 mm to (47.0, 192.0)
- moved MountBaseTop3 3.00 mm to (115.8, 192.0)
- moved MountBaseTop5 3.00 mm to (239.3, 192.0)
- moved MountBaseTop7 3.00 mm to (376.2, 192.0)
Other:
- outline, holes or cut-outs redrawn

Commit message: edit Kanagawa PCB
Parts:
- MountBaseTop1, MountBaseTop2, MountBaseTop3, MountBaseTop4, MountBaseTop5, MountBaseTop6, MountBaseTop7, MountBaseTop8: footprint keyboard:MountingHole_2.2mm_M2_Pad_Via -> Keyboard:MountingHole_2.2mm_M2_Pad_Via
- MountTopMiddle1, MountTopMiddle2, MountTopMiddle3, MountTopMiddle4, MountTopMiddle5, MountTopMiddle6, MountTopMiddle7, MountTopMiddle8: footprint keyboard:MountingHole_2.2mm_M2_Pad -> Keyboard:MountingHole_2.2mm_M2_Pad
Other:
- board text added: "JLCJLCJLCJLC"
