File: Kanagawa/rev2_rgb H/ANSI_Pico/Kanagawa_rgb_ansi_pico.kicad_sch (KiCad schematic)
At the start: 175 parts, among them J1 Oled128x32, J4 Conn_01x03, U0 Pico

Commit message: edit Kanagawa PCB
Parts:
- DA0, DA1, DA10, DA11, DA12, DA13, DA2, DA3, DA4, DA5, DA6, DA7, DA8, DA9, DB0, DB1, DB10, DB11, DB12, DB13, DB2, DB3, DB4, DB5, DB6, DB7, DB8, DB9, DC0, DC1, DC10, DC11, DC12, DC13, DC2, DC3, DC4, DC5, DC6, DC7, DC8, DC9, DD0, DD1, DD10, DD11, DD12, DD13, DD2, DD3, DD4, DD5, DD6, DD7, DD8, DD9, DE0, DE1, DE10, DE11, DE12, DE13, DE2, DE3, DE4, DE5, DE6, DE7, DE8, DE9, DF0, DF1, DF10, DF11, DF12, DF13, DF2, DF3, DF4, DF5, DF6, DF7, DF8, DF9: footprint keyboard:Diode_THT -> Keyboard:Diode_THT; symbol keyboard:D -> Keyboard:D
- J1: footprint keyboard:OLED_128x32_I2C -> Keyboard:OLED_128x32_I2C; symbol keyboard:Conn_01x04 -> Keyboard:Conn_01x04
- J4: footprint keyboard:conn_3pins -> Keyboard:conn_3pins; symbol keyboard:Conn_01x03 -> Keyboard:Conn_01x03
- JUSB1: footprint keyboard:GCT_USB4085-GF-A_REVA4 -> Keyboard:GCT_USB4085-GF-A_REVA4; symbol keyboard:USB4085-GF-A_REVA4 -> Keyboard:USB4085-GF-A_REVA4
- JUSB2: footprint keyboard:conn_4pins -> Keyboard:conn_4pins; symbol keyboard:Conn_01x04 -> Keyboard:Conn_01x04
- KA0, KA1, KA10, KA11, KA12, KA2, KA3, KA4, KA5, KA6, KA7, KA8, KA9, KB0, KB1, KB10, KB11, KB12, KB2, KB3, KB4, KB5, KB6, KB7, KB8, KB9, KC1, KC10, KC11, KC12, KC2, KC3, KC4, KC5, KC6, KC7, KC8, KC9, KD1, KD10, KD11, KD13, KD2, KD3, KD4, KD5, KD6, KD7, KD8, KD9, KE1, KE10, KE12, KE13, KE2, KE3, KE4, KE5, KE6, KE7, KE8, KE9, KF1, KF10, KF11, KF12, KF13, KF3, KF6, KF7, KF8, KF9: footprint keyboard:SW_Cherry_MX_1.00u_SK6812MINI-E_Hotswap -> Keyboard:SW_Cherry_MX_1.00u_SK6812MINI-E_Hotswap; symbol keyboard:KEY_SW_RGB -> Keyboard:KEY_SW_RGB
- KB13: footprint keyboard:SW_Cherry_MX_2.00u_SK6812MINI-E_Hotswap -> Keyboard:SW_Cherry_MX_2.00u_SK6812MINI-E_Hotswap; symbol keyboard:KEY_SW_RGB -> Keyboard:KEY_SW_RGB
- KC0, KC13: footprint keyboard:SW_Cherry_MX_1.50u_SK6812MINI-E_Hotswap -> Keyboard:SW_Cherry_MX_1.50u_SK6812MINI-E_Hotswap; symbol keyboard:KEY_SW_RGB -> Keyboard:KEY_SW_RGB
- KD0, KE11: footprint keyboard:SW_Cherry_MX_1.75u_SK6812MINI-E_Hotswap -> Keyboard:SW_Cherry_MX_1.75u_SK6812MINI-E_Hotswap; symbol keyboard:KEY_SW_RGB -> Keyboard:KEY_SW_RGB
- KD12, KE0: footprint keyboard:SW_Cherry_MX_2.25u_SK6812MINI-E_Hotswap -> Keyboard:SW_Cherry_MX_2.25u_SK6812MINI-E_Hotswap; symbol keyboard:KEY_SW_RGB -> Keyboard:KEY_SW_RGB
- KF0, KF2: footprint keyboard:SW_Cherry_MX_1.25u_SK6812MINI-E_Hotswap -> Keyboard:SW_Cherry_MX_1.25u_SK6812MINI-E_Hotswap; symbol keyboard:KEY_SW_RGB -> Keyboard:KEY_SW_RGB
- KF4, KF5: footprint keyboard:SW_Cherry_MX_2.00u_SK6812MINI-E_Hotswap_Reversed -> Keyboard:SW_Cherry_MX_2.00u_SK6812MINI-E_Hotswap_Reversed; symbol keyboard:KEY_SW_RGB -> Keyboard:KEY_SW_RGB
- RSW0, RSW1: footprint keyboard:SW_RST -> Keyboard:SW_RST; symbol keyboard:SW_RST -> Keyboard:SW_RST
- SWA13: footprint keyboard:RotaryEncoder_EC11-Switch_Horizontal_H15mm -> Keyboard:RotaryEncoder_EC11-Switch_Horizontal_H15mm; symbol keyboard:Rotary_Encoder_Switch -> Keyboard:Rotary_Encoder_Switch
- U0: footprint keyboard:RPi_Pico_TH -> Keyboard:RPi_Pico_TH; symbol keyboard:Pi Pico -> Keyboard:Pi Pico

Commit message: edit Kanagawa PCB
Parts:
- removed JUSB2: USB Breakout, Keyboard:conn_4pins, symbol Keyboard:Conn_01x04
- added R1, R2: 5.1k, Keyboard:Resistors_THT, symbol Keyboard:R
Connections:
- net GND: now also R1.1, R2.1
- net at JUSB1.A5 (CC1): now also R2.2
- net at JUSB1.B5 (CC2): now also R1.2
- no-connect marks 13 -> 11
Other:
- moved on the sheet: JUSB1
