File: Kanagawa/rev2_rgb H/One_Pico/Kanagawa_rgb_pico.kicad_sch (KiCad schematic)
At the start: 182 parts, among them J1 Oled128x32, J4 Conn_01x03, U0 Pico

Commit message: edit Kanagawa PCB
Parts:
- added J2: ANSI RGB Jumper, Keyboard:SolderJumper, symbol Keyboard:Conn_01x02
- added R1, R2: 5.1k, Keyboard:Resistors_THT, symbol Keyboard:R
Connections:
- net GND: now also R1.1, R2.1
- net IN_E0: now also J2.1 (Pin_1)
- net IN_E1: now also J2.2 (Pin_2)
- net at JUSB1.A5 (CC1): now also R1.2
- net at JUSB1.B5 (CC2): now also R2.2
- no-connect marks 13 -> 11
Other:
- moved on the sheet: JUSB1, U0
