File: Kanagawa/rev2_rgb H/One_Pico/generated_pcbs/top.kicad_pcb (KiCad board)
At the start: 2 copper layers, 335.2 x 145.9 mm, 16 parts

Commit message: edit Kanagawa PCB
Parts:
- removed the MountTopMiddle7 at (339.5, 170.5)
- moved MountTopMiddle7 35.6 mm to (370.5, 105.7)
- moved MountTopMiddle5 25.0 mm to (310.1, 158.9)
- renumbered MountTopMiddle8 to MountTopMiddle7
Routing:
- net GND: vias 1 -> 0
Other:
- outline, holes or cut-outs redrawn

Commit message: Update rev2.1
Parts:
- moved MountTopMiddle1 16.8 mm to (51.4, 160.3)
- moved MountBaseTop1 2.00 mm to (45.0, 192.0)
- moved MountBaseTop2 2.00 mm to (45.0, 57.6)
- moved MountBaseTop7 2.00 mm to (378.2, 192.0)
- moved MountBaseTop8 2.00 mm to (378.2, 57.6)
- moved MountBaseTop3 0.16 mm to (115.7, 192.0)
- moved MountBaseTop4 0.16 mm to (115.7, 57.6)
- moved MountBaseTop5 0.16 mm to (239.5, 192.0)
- moved MountBaseTop6 0.16 mm to (239.5, 57.6)
Other:
- board size 335.2 x 145.9 mm -> 339.2 x 147.4 mm
