File: Kanagawa/rev1/generated_pcbs/base.kicad_pcb (KiCad board)
At the start: 2 copper layers, 330 x 142 mm, 8 parts

Commit message: edit arc for edge cut in script
Parts:
- removed MountBaseMiddleTop7: MountingHole, keyboard:MountingHole_2.2mm_M2_Pad_Via
- moved MountBaseMiddleTop1 2.40 mm to (60.0, 81.0)
- moved MountBaseMiddleTop5 2.23 mm to (381.0, 81.0)
- moved MountBaseMiddleTop3 2.00 mm to (244.9, 81.2)
- moved MountBaseMiddleTop2 0.92 mm to (60.0, 207.0)
- moved MountBaseMiddleTop4 0.92 mm to (244.0, 207.0)
- moved MountBaseMiddleTop6 0.92 mm to (380.0, 207.0)
Other:
- board size 330 x 142 mm -> 330 x 144 mm

Commit message: rework rev1 from fusion layout
Parts:
- added MountBaseMiddleTop3: MountingHole, keyboard:MountingHole_2.2mm_M2_Pad_Via, F.Cu at (125.9, 81.2)
- added MountBaseMiddleTop4: MountingHole, keyboard:MountingHole_2.2mm_M2_Pad_Via, F.Cu at (125.9, 207.2)
- LogoBase1: footprint layout-for-export:Great-wave -> keyboard:hokusai
- moved MountBaseMiddleTop7 4.12 mm to (376.9, 81.2)
- moved LogoBase1 4.09 mm to (219.3, 146.2)
- moved MountBaseMiddleTop8 3.12 mm to (376.9, 207.2)
- moved MountBaseMiddleTop1 1.90 mm to (61.9, 81.2)
- moved MountBaseMiddleTop2 1.90 mm to (61.9, 207.2)
- moved MountBaseMiddleTop6 0.92 mm to (244.9, 207.2)
- renumbered MountBaseMiddleTop3 to MountBaseMiddleTop5, MountBaseMiddleTop4 to MountBaseMiddleTop6, MountBaseMiddleTop5 to MountBaseMiddleTop7, MountBaseMiddleTop6 to MountBaseMiddleTop8
Other:
- board size 330 x 144 mm -> 325 x 143 mm

Commit message: generate kanagawa gerber
Other:
- outline, holes or cut-outs redrawn

Commit message: re route pcbs
Other:
- outline, holes or cut-outs redrawn
- net class Default removed

Commit message: release 1.0
Parts:
- moved LogoBase1 3.01 mm to (219.5, 149.2)
