File: Pallas/generated_pcbs/base.kicad_pcb (KiCad board)
At the start: 2 copper layers, 467.5 x 140 mm, 18 parts

Commit message: Fix issue with label design by
Changed lines of the file:
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@@
-(kicad_pcb (version 20171130) (host pcbnew "(5.1.6)-1")
+(kicad_pcb (version 20171130) (host pcbnew 5.1.6-c6e7f7d~86~ubuntu20.04.1)
   (general
     (thickness 1.6)
@@
       (drillshape 0)
       (scaleselection 1)
-      (outputdirectory "gerber/base/"))
+      (outputdirectory "pallas/"))
   )
   (net 0 "")
@@
       (xy -2.511352 -3.707233) (xy -2.125299 -3.941597) (xy -1.71799 -4.135869) (xy -1.29263 -4.288478)
       (xy -0.852427 -4.397857) (xy -0.400584 -4.462436) (xy 0.059691 -4.480646) (xy 0.525194 -4.450919)) (layer F.SilkS) (width 0.01))
-    (fp_text user Ciaanh (at -13 4 270) (layer B.SilkS)
+    (fp_text user Ciaanh (at -13 4 285) (layer B.SilkS)
       (effects (font (size 1 1) (thickness 0.15) italic) (justify mirror))
     )
-    (fp_text user "Designed by" (at -13 2 270) (layer B.SilkS)
+    (fp_text user "Designed by" (at -13 2 285) (layer B.SilkS)
       (effects (font (size 1 1) (thickness 0.15) italic) (justify mirror))
     )
-    (fp_text user Ciaanh (at -13 4 90) (layer F.SilkS)
+    (fp_text user Ciaanh (at -13 4 105) (layer F.SilkS)
       (effects (font (size 1 1) (thickness 0.15) italic))
     )
-    (fp_text user "Designed by" (at -13 2 90) (layer F.SilkS)
+    (fp_text user "Designed by" (at -13 2 105) (layer F.SilkS)
       (effects (font (size 1 1) (thickness 0.15) italic))
     )
