File: Pallas/generated_pcbs/middle.kicad_pcb (KiCad board)
At the start: 2 copper layers, 467.5 x 140 mm, 259 parts, among them J1 OLED, J2 RGB_LED, Q1 IRLML6344TRPbF, SW00 SW_PUSH, SW01 SW_PUSH, SW010 SW_PUSH, SW011 SW_PUSH, SW012 SW_PUSH, SW013 SW_PUSH, SW014 SW_PUSH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

Commit message: review
Routing:
- net GND: vias 3 -> 99

Commit message: fix mosfet footprint
Routing:
- net GND: vias 99 -> 13
