File: Wonderland/Board/Wonderland.kicad_sch (KiCad schematic)
At the start: 176 parts, among them J1 Conn_01x03, J2 Conn_01x02, J4 Conn_01x03, U1 RP2040_Stamp

Commit message: edit wonderland routes
Parts:
- added MountTopMiddle1, MountTopMiddle2, MountTopMiddle3, MountTopMiddle4, MountTopMiddle5, MountTopMiddle6: MountingHole, Keyboard:MountingHole_2.2mm_M2_Pad, symbol Keyboard:MountingHole
Connections:
- net col00: now also U1.10 (GPIO9); no longer U1.7 (GPIO6)
- net col01: now also U1.9 (GPIO8); no longer U1.6 (GPIO5)
- net col02: now also U1.8 (GPIO7); no longer U1.5 (GPIO4)
- net col03: now also U1.7 (GPIO6); no longer U1.4 (GPIO3)
- net col04: now also U1.6 (GPIO5); no longer U1.3 (GPIO2)
- net col05: now also U1.5 (GPIO4); no longer U1.2 (GPIO1)
- net col06: now also U1.4 (GPIO3); no longer U1.1 (GPIO0)
- net row00: now also U1.1 (GPIO0); no longer U1.11 (GPIO10)
- net row01: now also U1.2 (GPIO1); no longer U1.12 (GPIO11)
- net row02: now also U1.3 (GPIO2); no longer U1.13 (GPIO12)
