File: Wonderland/rp2040-guide/Wonderland.kicad_sch (KiCad schematic)
At the start: 218 parts, among them J1 USB_C_Receptacle_USB2.0, J2 SWD, J3 Conn_01x11, J4 Conn_01x11, J5 Conn_01x11, J6 Conn_01x03, J7 Conn_01x03, J8 Conn_01x02, SW1 SW_Push, U1 W25Q128JVS, U2 USBLC6-2SC6, U3 RP2040, U4 XC6206PxxxMR-Regulator_Linear, U5 RP2040_Stamp, Y1 12MHz

Commit message: add rp2040 minimal & review test board with hardware specs
Parts:
- removed J1: USB_C_Receptacle_USB2.0, Connector_USB:USB_C_Receptacle_HRO_TYPE-C-31-M-12, symbol Connector:USB_C_Receptacle_USB2.0
- removed R8, R9: 5.1k, Keyboard:Resistors_THT, symbol Keyboard:R
- removed SW1: SW_Push, Connector_PinSocket_2.54mm:PinSocket_1x02_P2.54mm_Vertical, symbol Switch:SW_Push
- removed U5: RP2040_Stamp, Keyboard:RP2040_Stamp_THT, symbol Keyboard:RP2040_Stamp
- U3: footprint Sleep-Lib:RP2040-QFN-56 -> RP2040_minimal:RP2040-QFN-56; symbol Sleep-lib:RP2040 -> MCU_RaspberryPi_RP2040:RP2040
Connections:
- net BOOTSEL is gone; now on net GND: RSW1.1
- net D+ is gone; now on net D_USB_P: JUSB1.A6 (DP1), JUSB1.B6 (DP2)
- net D- is gone; now on net D_USB_N: JUSB1.A7 (DN1), JUSB1.B7 (DN2)
- net RESET is gone; now on net ~{RESET}: RSW2.1
- net +5V: no longer JUSB1.A4 (VBUS), JUSB1.A9 (VBUS), JUSB1.B4 (VBUS), JUSB1.B9 (VBUS)
- net CC1: now also JUSB1.A5 (CC1), R3.2; no longer R3.1
- net CC2: now also JUSB1.B5 (CC2), R4.2; no longer R4.1
- net ENCA: now also U3.34 (GPIO22)
- net ENCB: now also U3.32 (GPIO21)
- net GND: now also R3.1, R4.1; no longer R3.2, R4.2, RSW1.2
- net RGB_Matrix: now also U3.35 (GPIO23); no longer U3.37 (GPIO25)
- net VBUS: now also JUSB1.A4 (VBUS), JUSB1.A9 (VBUS), JUSB1.B4 (VBUS), JUSB1.B9 (VBUS)
- net col00: now also U3.2 (GPIO0)
- net col01: now also U3.3 (GPIO1)
- net col02: now also U3.4 (GPIO2)
- net col03: now also U3.5 (GPIO3)
- net col04: now also U3.6 (GPIO4)
- net col05: now also U3.7 (GPIO5)
- net col06: now also U3.8 (GPIO6)
- net col07: now also U3.9 (GPIO7); no longer U3.36 (GPIO24)
- net col08: now also U3.11 (GPIO8); no longer U3.35 (GPIO23)
- net col09: now also U3.12 (GPIO9); no longer U3.34 (GPIO22)
- net col10: now also U3.13 (GPIO10); no longer U3.32 (GPIO21)
- net col11: now also U3.14 (GPIO11); no longer U3.31 (GPIO20)
- net col12: now also U3.15 (GPIO12); no longer U3.30 (GPIO19)
- net col13: now also U3.16 (GPIO13); no longer U3.29 (GPIO18)
- net row00: now also U3.18 (GPIO15)
- net row01: now also U3.27 (GPIO16)
- net row02: now also U3.28 (GPIO17)
- net row03: now also U3.29 (GPIO18)
- net row04: now also U3.30 (GPIO19)
- net row05: now also U3.31 (GPIO20)
- net ~{USB_BOOT}: now also RSW1.2
- no-connect marks 14 -> 9
Other:
- note added: "Crystal oscillator"
- note added: "Make sure C4 is close to pin 45"
- note added: "Make sure C8 is close to pin 44"
- note added: "Make sure R5 & R6 are close to MCU"
- note added: "Power supply & data"
- note removed: "Crystal"
- note removed: "MOUNTINGHOLES (REMOVED)"
- note removed: "Maybe add something on shield?"
- note removed: "USB"
- moved on the sheet: C1, C10, C11, C12, C13, C14, C15, C16, C17, C4, C5, C6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

Commit message: edit full pcb
Parts:
- removed J2: SWD, Connector_PinSocket_2.54mm:PinSocket_1x05_P2.54mm_Vertical, symbol Connector_Generic:Conn_01x05
- removed J3, J4, J5: Conn_01x11, Connector_PinSocket_2.54mm:PinSocket_1x11_P2.54mm_Vertical, symbol Connector_Generic:Conn_01x11
- renumbered DA1 to DA0, DA2 to DA1, DA11 to DA10, DA12 to DA11, DA13 to DA12, DA14 to DA13, DA3 to DA2, DA4 to DA3, DA5 to DA4, DA6 to DA5, DA7 to DA6, DA8 to DA7, DA9 to DA8, DA10 to DA9, DB1 to DB0, DB2 to DB1, DB11 to DB10, DB12 to DB11, DB13 to DB12, DB14 to DB13, DB3 to DB2, DB4 to DB3, DB5 to DB4, DB6 to DB5, DB7 to DB6, DB8 to DB7, DB9 to DB8, DB10 to DB9, DC1 to DC0, DC2 to DC1, DC11 to DC10, DC12 to DC11, DC13 to DC12, DC14 to DC13, DC3 to DC2, DC4 to DC3, DC5 to DC4, DC6 to DC5, DC7 to DC6, DC8 to DC7, DC9 to DC8, DC10 to DC9, DD1 to DD0, DD2 to DD1, DD11 to DD10, DD12 to DD11, DD13 to DD12, DD14 to DD13, DD3 to DD2, DD4 to DD3, DD5 to DD4, DD6 to DD5, DD7 to DD6, DD8 to DD7, DD9 to DD8, DD10 to DD9, DE1 to DE0, DE2 to DE1, DE11 to DE10, DE12 to DE11, DE13 to DE12, DE14 to DE13, DE3 to DE2, DE4 to DE3, DE5 to DE4, DE6 to DE5, DE7 to DE6, DE8 to DE7, DE9 to DE8, DE10 to DE9, DF1 to DF0, DF2 to DF1, DF11 to DF10, DF12 to DF11, DF13 to DF12, DF14 to DF13, DF3 to DF2, DF4 to DF3, DF5 to DF4, DF6 to DF5, DF7 to DF6, DF8 to DF7, DF9 to DF8, DF10 to DF9, KA1 to KA0, KA2 to KA1, KB1 to KB0, KB2 to KB1, KC1 to KC0, KC2 to KC1, KD1 to KD0, KD2 to KD1, KE1 to KE0, KE2 to KE1, KF1 to KF0, KF2 to KF1
Connections:
- net OUT_D0 is gone; now on net IN_E13: KD0.4 (DOUT)
- net XTAL_O is gone; now on net GND: C3.2, R7.1, Y1.1
- net VCC renamed +3.3V
Other:
- note added: "Key matrix"
- note added: "MCU"
- note added: "Make sure R1 is close to the flash chip"
- note added: "Mounting holes"
- note added: "RGB matrix"
- moved on the sheet: C1, C10, C11, C12, C13, C14, C15, C16, C17, C2, C3, C4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

Commit message: review schematics wonderland
Parts:
- DA0, DA1, DA10, DA11, DA12, DA13, DA2, DA3, DA4, DA5, DA6, DA7, DA8, DA9, DB0, DB1, DB10, DB11, DB12, DB13, DB2, DB3, DB4, DB5, DB6, DB7, DB8, DB9, DC0, DC1, DC10, DC11, DC12, DC13, DC2, DC3, DC4, DC5, DC6, DC7, DC8, DC9, DD0, DD1, DD10, DD11, DD12, DD13, DD2, DD3, DD4, DD5, DD6, DD7, DD8, DD9, DE0, DE1, DE10, DE11, DE12, DE13, DE2, DE3, DE4, DE5, DE6, DE7, DE8, DE9, DF0, DF1, DF10, DF11, DF12, DF13, DF2, DF3, DF4, DF5, DF6, DF7, DF8, DF9: value D -> 1N4148; footprint Keyboard:Diode_THT -> Diode_SMD:D_SOD-123
- KA0, KA1, KB0, KB1, KC0, KC1, KD0, KD1, KE0, KE1, KF0, KF1: value KEY_SW -> CPG151101S11-1
- KA10: renamed from KA11; value KEY_SW -> CPG151101S11-1
- KA11: renamed from KA12; value KEY_SW -> CPG151101S11-1
- KA12: renamed from KA13; value KEY_SW -> CPG151101S11-1
- KA13: renamed from KA14; value KEY_SW -> CPG151101S11-1
- KA2: renamed from KA3; value KEY_SW -> CPG151101S11-1
- KA3: renamed from KA4; value KEY_SW -> CPG151101S11-1
- KA4: renamed from KA5; value KEY_SW -> CPG151101S11-1
- KA5: renamed from KA6; value KEY_SW -> CPG151101S11-1
- KA6: renamed from KA7; value KEY_SW -> CPG151101S11-1
- KA7: renamed from KA8; value KEY_SW -> CPG151101S11-1
- KA8: renamed from KA9; value KEY_SW -> CPG151101S11-1
- KA9: renamed from KA10; value KEY_SW -> CPG151101S11-1
- KB10: renamed from KB11; value KEY_SW -> CPG151101S11-1
- KB11: renamed from KB12; value KEY_SW -> CPG151101S11-1
- KB12: renamed from KB13; value KEY_SW -> CPG151101S11-1
- KB13: renamed from KB14; value KEY_SW -> CPG151101S11-1
- KB2: renamed from KB3; value KEY_SW -> CPG151101S11-1
- KB3: renamed from KB4; value KEY_SW -> CPG151101S11-1
- KB4: renamed from KB5; value KEY_SW -> CPG151101S11-1
- KB5: renamed from KB6; value KEY_SW -> CPG151101S11-1
- KB6: renamed from KB7; value KEY_SW -> CPG151101S11-1
- KB7: renamed from KB8; value KEY_SW -> CPG151101S11-1
- KB8: renamed from KB9; value KEY_SW -> CPG151101S11-1
- KB9: renamed from KB10; value KEY_SW -> CPG151101S11-1
- KC10: renamed from KC11; value KEY_SW -> CPG151101S11-1
- KC11: renamed from KC12; value KEY_SW -> CPG151101S11-1
- KC12: renamed from KC13; value KEY_SW -> CPG151101S11-1
- KC13: renamed from KC14; value KEY_SW -> CPG151101S11-1
- KC2: renamed from KC3; value KEY_SW -> CPG151101S11-1
- KC3: renamed from KC4; value KEY_SW -> CPG151101S11-1
- KC4: renamed from KC5; value KEY_SW -> CPG151101S11-1
- KC5: renamed from KC6; value KEY_SW -> CPG151101S11-1
- KC6: renamed from KC7; value KEY_SW -> CPG151101S11-1
- KC7: renamed from KC8; value KEY_SW -> CPG151101S11-1
- KC8: renamed from KC9; value KEY_SW -> CPG151101S11-1
- KC9: renamed from KC10; value KEY_SW -> CPG151101S11-1
- KD10: renamed from KD11; value KEY_SW -> CPG151101S11-1
- KD11: renamed from KD12; value KEY_SW -> CPG151101S11-1
- KD12: renamed from KD13; value KEY_SW -> CPG151101S11-1
- KD13: renamed from KD14; value KEY_SW -> CPG151101S11-1
- KD2: renamed from KD3; value KEY_SW -> CPG151101S11-1
- KD3: renamed from KD4; value KEY_SW -> CPG151101S11-1
- KD4: renamed from KD5; value KEY_SW -> CPG151101S11-1
- KD5: renamed from KD6; value KEY_SW -> CPG151101S11-1
- KD6: renamed from KD7; value KEY_SW -> CPG151101S11-1
- KD7: renamed from KD8; value KEY_SW -> CPG151101S11-1
- KD8: renamed from KD9; value KEY_SW -> CPG151101S11-1
- KD9: renamed from KD10; value KEY_SW -> CPG151101S11-1
- KE10: renamed from KE11; value KEY_SW -> CPG151101S11-1
- KE11: renamed from KE12; value KEY_SW -> CPG151101S11-1
- KE12: renamed from KE13; value KEY_SW -> CPG151101S11-1
- KE13: renamed from KE14; value KEY_SW -> CPG151101S11-1
- KE2: renamed from KE3; value KEY_SW -> CPG151101S11-1
- KE3: renamed from KE4; value KEY_SW -> CPG151101S11-1
- KE4: renamed from KE5; value KEY_SW -> CPG151101S11-1
- KE5: renamed from KE6; value KEY_SW -> CPG151101S11-1
- KE6: renamed from KE7; value KEY_SW -> CPG151101S11-1
- KE7: renamed from KE8; value KEY_SW -> CPG151101S11-1
- KE8: renamed from KE9; value KEY_SW -> CPG151101S11-1
- KE9: renamed from KE10; value KEY_SW -> CPG151101S11-1
- KF10: renamed from KF11; value KEY_SW -> CPG151101S11-1
- KF11: renamed from KF12; value KEY_SW -> CPG151101S11-1
- KF12: renamed from KF13; value KEY_SW -> CPG151101S11-1
- KF2: renamed from KF3; value KEY_SW -> CPG151101S11-1
- KF3: renamed from KF4; value KEY_SW -> CPG151101S11-1
- KF4: renamed from KF5; value KEY_SW -> CPG151101S11-1
- KF5: renamed from KF6; value KEY_SW -> CPG151101S11-1
- KF6: renamed from KF7; value KEY_SW -> CPG151101S11-1
- KF7: renamed from KF8; value KEY_SW -> CPG151101S11-1
- KF8: renamed from KF9; value KEY_SW -> CPG151101S11-1
- KF9: renamed from KF10; value KEY_SW -> CPG151101S11-1
- U1: LCSC C131025 -> (none)
- U3: LCSC C2040 -> (none)
- U4: symbol kicad-keyboard-parts:XC6206PxxxMR-Regulator_Linear -> Keyboard:XC6206PxxxMR-Regulator_Linear
- renumbered J7 to J1, J8 to J2, J6 to J3
Connections:
- net SWCLK: no longer names the net of U3.24 (SWCLK)
- net SWD: no longer names the net of U3.25 (SWD)
- no-connect marks 9 -> 11
Other:
- moved on the sheet: C1, DA0, DA1, DA10, DA11, DA12, DA13, DA2, DA3, DA4, DA5, DA6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
