File: Wonderland/Board-integrated/generated_pcbs/plate.kicad_pcb (KiCad board)
At the start: 2 copper layers, 341 x 140.6 mm, 6 parts

Commit message: generated PCB
Other:
- outline, holes or cut-outs redrawn
