File: Wonderland/Board-integrated/generated_pcbs/plate.kicad_pcb (KiCad board)
At the start: 2 copper layers, 341 x 140.6 mm, 6 parts

Commit message: generated PCB
Other:
- board size 341 x 140.6 mm -> 339 x 146.6 mm

Commit message: update wonderland
Other:
- board size 339 x 146.6 mm -> 339 x 143.1 mm
